File: 02.0_top_plate/ori_top_plate.kicad_pcb (KiCad board)
At the start: 2 copper layers, 252.4 x 82.2 mm, 65 parts, among them U1 HOLE, U10 HOLE, U11 HOLE, U12 HOLE, U13 HOLE, U14 HOLE, U15 HOLE, U16 HOLE, U17 HOLE, U18 HOLE, U19 HOLE, U2 HOLE, U20 HOLE, U21 HOLE, U22 HOLE, U23 HOLE, U24 HOLE, U25 HOLE, U26 HOLE, U27 HOLE, U28 HOLE, U29 HOLE, U3 HOLE, U30 HOLE, U31 HOLE, U32 HOLE, U33 HOLE, U34 HOLE, U35 HOLE, U36 HOLE, U37 HOLE, U38 HOLE, U39 HOLE, U4 HOLE, U40 HOLE, U41 HOLE, U42 HOLE, U43 HOLE, U44 HOLE, U45 HOLE, U46 HOLE, U47 HOLE, U48 HOLE, U49 HOLE, U5 HOLE, U53 HOLE, U57 HOLE, U6 HOLE, U61 HOLE, U7 HOLE, U8 HOLE, U9 HOLE

Commit message: modify top plate
Parts:
- added H12: MountingHole, MountingHole:MountingHole_2.2mm_M2, F.Cu at (165.5, 59.5)
- added H13: MountingHole, MountingHole:MountingHole_2.2mm_M2, F.Cu at (298.9, 59.5)
- added H14: MountingHole, MountingHole:MountingHole_2.2mm_M2, F.Cu at (165.5, 97.6)
- added H15: MountingHole, MountingHole:MountingHole_2.2mm_M2, F.Cu at (298.9, 97.6)
- added H16: MountingHole, MountingHole:MountingHole_2.2mm_M2, F.Cu at (222.7, 59.5)
- added H17: MountingHole, MountingHole:MountingHole_2.2mm_M2, F.Cu at (356.0, 59.5)
- added H18: MountingHole, MountingHole:MountingHole_2.2mm_M2, F.Cu at (222.7, 97.6)
- added H19: MountingHole, MountingHole:MountingHole_2.2mm_M2, F.Cu at (356.0, 97.6)
- added H20: MountingHole, MountingHole:MountingHole_2.2mm_M2, F.Cu at (379.8, 59.5)
- added H21: MountingHole, MountingHole:MountingHole_2.2mm_M2, F.Cu at (379.8, 97.6)
Changed lines of the file:
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@@
     (tracks 4)
     (zones 0)
-    (modules 65)
+    (modules 75)
     (nets 5)
   )
@@
     (uvia_drill 0.2)
   )
+  (module MountingHole:MountingHole_2.2mm_M2 (layer F.Cu)
+    (at 379.835826 97.618904)
+    (descr "Mounting Hole 2.2mm, no annular, M2")
+    (tags "mounting hole 2.2mm no annular m2")
+    (attr virtual)
+    (fp_text reference H21 (at 0 -3.2) (layer Dwgs.User)
+      (effects (font (size 1 1) (thickness 0.15)))
+    )
+    (fp_text value MountingHole (at 0 3.2) (layer F.Fab)
+      (effects (font (size 1 1) (thickness 0.15)))
+    )
+    (fp_text user %R (at 0.3 0) (layer F.Fab)
+      (effects (font (size 1 1) (thickness 0.15)))
+    )
+    (fp_circle (center 0 0) (end 2.45 0) (layer F.CrtYd) (width 0.05))
+    (fp_circle (center 0 0) (end 2.2 0) (layer Cmts.User) (width 0.15))
+    (pad 1 np_thru_hole circle (at 0 0) (size 2.2 2.2) (drill 2.2) (layers *.Cu *.Mask))
+  )
+  (module MountingHole:MountingHole_2.2mm_M2 (layer F.Cu)
+    (at 379.835826 59.518936)
+    (descr "Mounting Hole 2.2mm, no annular, M2")
+    (tags "mounting hole 2.2mm no annular m2")
+    (attr virtual)
+    (fp_text reference H20 (at 0 -3.2) (layer Dwgs.User)
+      (effects (font (size 1 1) (thickness 0.15)))
+    )
+    (fp_text value MountingHole (at 0 3.2) (layer F.Fab)
+      (effects (font (size 1 1) (thickness 0.15)))
+    )
+    (fp_text user %R (at 0.3 0) (layer F.Fab)
+      (effects (font (size 1 1) (thickness 0.15)))
+    )
+    (fp_circle (center 0 0) (end 2.45 0) (layer F.CrtYd) (width 0.05))
+    (fp_circle (center 0 0) (end 2.2 0) (layer Cmts.User) (width 0.15))
+    (pad 1 np_thru_hole circle (at 0 0) (size 2.2 2.2) (drill 2.2) (layers *.Cu *.Mask))
+  )
+  (module MountingHole:MountingHole_2.2mm_M2 (layer F.Cu)
+    (at 356.023346 97.618904)
+    (descr "Mounting Hole 2.2mm, no annular, M2")
+    (tags "mounting hole 2.2mm no annular m2")
+    (attr virtual)
+    (fp_text reference H19 (at 0 -3.2) (layer Dwgs.User)
+      (effects (font (size 1 1) (thickness 0.15)))
+    )
+    (fp_text value MountingHole (at 0 3.2) (layer F.Fab)
+      (effects (font (size 1 1) (thickness 0.15)))
+    )
+    (fp_text user %R (at 0.3 0) (layer F.Fab)
+      (effects (font (size 1 1) (thickness 0.15)))
+    )
+    (fp_circle (center 0 0) (end 2.45 0) (layer F.CrtYd) (width 0.05))
+    (fp_circle (center 0 0) (end 2.2 0) (layer Cmts.User) (width 0.15))
+    (pad 1 np_thru_hole circle (at 0 0) (size 2.2 2.2) (drill 2.2) (layers *.Cu *.Mask))
+  )
+  (module MountingHole:MountingHole_2.2mm_M2 (layer F.Cu)
+    (at 222.673458 97.618904)
+    (descr "Mounting Hole 2.2mm, no annular, M2")
+    (tags "mounting hole 2.2mm no annular m2")
+    (attr virtual)
+    (fp_text reference H18 (at 0 -3.2) (layer Dwgs.User)
+      (effects (font (size 1 1) (thickness 0.15)))
+    )
+    (fp_text value MountingHole (at 0 3.2) (layer F.Fab)
+      (effects (font (size 1 1) (thickness 0.15)))
+    )
+    (fp_text user %R (at 0.3 0) (layer F.Fab)
+      (effects (font (size 1 1) (thickness 0.15)))
+    )
+    (fp_circle (center 0 0) (end 2.45 0) (layer F.CrtYd) (width 0.05))
+    (fp_circle (center 0 0) (end 2.2 0) (layer Cmts.User) (width 0.15))
+    (pad 1 np_thru_hole circle (at 0 0) (size 2.2 2.2) (drill 2.2) (layers *.Cu *.Mask))
+  )
+  (module MountingHole:MountingHole_2.2mm_M2 (layer F.Cu)
+    (at 356.023346 59.518936)
+    (descr "Mounting Hole 2.2mm, no annular, M2")
+    (tags "mounting hole 2.2mm no annular m2")
+    (attr virtual)
+    (fp_text reference H17 (at 0 -3.2) (layer Dwgs.User)
+      (effects (font (size 1 1) (thickness 0.15)))
+    )
+    (fp_text value MountingHole (at 0 3.2) (layer F.Fab)
+      (effects (font (size 1 1) (thickness 0.15)))
+    )
+    (fp_text user %R (at 0.3 0) (layer F.Fab)
+      (effects (font (size 1 1) (thickness 0.15)))
+    )
+    (fp_circle (center 0 0) (end 2.45 0) (layer F.CrtYd) (width 0.05))
+    (fp_circle (center 0 0) (end 2.2 0) (layer Cmts.User) (width 0.15))
+    (pad 1 np_thru_hole circle (at 0 0) (size 2.2 2.2) (drill 2.2) (layers *.Cu *.Mask))
+  )
+  (module MountingHole:MountingHole_2.2mm_M2 (layer F.Cu)
+    (at 222.673458 59.518936)
+    (descr "Mounting Hole 2.2mm, no annular, M2")
+    (tags "mounting hole 2.2mm no annular m2")
+    (attr virtual)
+    (fp_text reference H16 (at 0 -3.2) (layer Dwgs.User)
+      (effects (font (size 1 1) (thickness 0.15)))
+    )
+    (fp_text value MountingHole (at 0 3.2) (layer F.Fab)
+      (effects (font (size 1 1) (thickness 0.15)))
+    )
+    (fp_text user %R (at 0.3 0) (layer F.Fab)
+      (effects (font (size 1 1) (thickness 0.15)))
+    )
+    (fp_circle (center 0 0) (end 2.45 0) (layer F.CrtYd) (width 0.05))
+    (fp_circle (center 0 0) (end 2.2 0) (layer Cmts.User) (width 0.15))
+    (pad 1 np_thru_hole circle (at 0 0) (size 2.2 2.2) (drill 2.2) (layers *.Cu *.Mask))
+  )
+  (module MountingHole:MountingHole_2.2mm_M2 (layer F.Cu)
+    (at 298.873394 97.618904)
+    (descr "Mounting Hole 2.2mm, no annular, M2")
+    (tags "mounting hole 2.2mm no annular m2")
+    (attr virtual)
+    (fp_text reference H15 (at 0 -3.2) (layer Dwgs.User)
+      (effects (font (size 1 1) (thickness 0.15)))
+    )
+    (fp_text value MountingHole (at 0 3.2) (layer F.Fab)
+      (effects (font (size 1 1) (thickness 0.15)))
+    )
+    (fp_text user %R (at 0.3 0) (layer F.Fab)
+      (effects (font (size 1 1) (thickness 0.15)))
+    )
+    (fp_circle (center 0 0) (end 2.45 0) (layer F.CrtYd) (width 0.05))
+    (fp_circle (center 0 0) (end 2.2 0) (layer Cmts.User) (width 0.15))
+    (pad 1 np_thru_hole circle (at 0 0) (size 2.2 2.2) (drill 2.2) (layers *.Cu *.Mask))
+  )
+  (module MountingHole:MountingHole_2.2mm_M2 (layer F.Cu)
+    (at 165.523506 97.618904)
+    (descr "Mounting Hole 2.2mm, no annular, M2")
+    (tags "mounting hole 2.2mm no annular m2")
+    (attr virtual)
+    (fp_text reference H14 (at 0 -3.2) (layer Dwgs.User)
+      (effects (font (size 1 1) (thickness 0.15)))
+    )
+    (fp_text value MountingHole (at 0 3.2) (layer F.Fab)
+      (effects (font (size 1 1) (thickness 0.15)))
+    )
+    (fp_text user %R (at 0.3 0) (layer F.Fab)
+      (effects (font (size 1 1) (thickness 0.15)))
+    )
+    (fp_circle (center 0 0) (end 2.45 0) (layer F.CrtYd) (width 0.05))
+    (fp_circle (center 0 0) (end 2.2 0) (layer Cmts.User) (width 0.15))
+    (pad 1 np_thru_hole circle (at 0 0) (size 2.2 2.2) (drill 2.2) (layers *.Cu *.Mask))
+  )
+  (module MountingHole:MountingHole_2.2mm_M2 (layer F.Cu)
+    (at 298.873394 59.518936)
+    (descr "Mounting Hole 2.2mm, no annular, M2")
+    (tags "mounting hole 2.2mm no annular m2")
+    (attr virtual)
+    (fp_text reference H13 (at 0 -3.2) (layer Dwgs.User)
+      (effects (font (size 1 1) (thickness 0.15)))
+    )
+    (fp_text value MountingHole (at 0 3.2) (layer F.Fab)
+      (effects (font (size 1 1) (thickness 0.15)))
+    )
+    (fp_text user %R (at 0.3 0) (layer F.Fab)
+      (effects (font (size 1 1) (thickness 0.15)))
+    )
+    (fp_circle (center 0 0) (end 2.45 0) (layer F.CrtYd) (width 0.05))
+    (fp_circle (center 0 0) (end 2.2 0) (layer Cmts.User) (width 0.15))
+    (pad 1 np_thru_hole circle (at 0 0) (size 2.2 2.2) (drill 2.2) (layers *.Cu *.Mask))
+  )
+  (module MountingHole:MountingHole_2.2mm_M2 (layer F.Cu)
+    (at 165.523506 59.518936)
+    (descr "Mounting Hole 2.2mm, no annular, M2")
+    (tags "mounting hole 2.2mm no annular m2")
+    (attr virtual)
+    (fp_text reference H12 (at 0 -3.2) (layer Dwgs.User)
+      (effects (font (size 1 1) (thickness 0.15)))
+    )
+    (fp_text value MountingHole (at 0 3.2) (layer F.Fab)
+      (effects (font (size 1 1) (thickness 0.15)))
+    )
+    (fp_text user %R (at 0.3 0) (layer F.Fab)
+      (effects (font (size 1 1) (thickness 0.15)))
+    )
+    (fp_circle (center 0 0) (end 2.45 0) (layer F.CrtYd) (width 0.05))
+    (fp_circle (center 0 0) (end 2.2 0) (layer Cmts.User) (width 0.15))
+    (pad 1 np_thru_hole circle (at 0 0) (size 2.2 2.2) (drill 2.2) (layers *.Cu *.Mask))
+  )
   (module acheron_Hardware:MouseBite_IPC7351 (layer F.Cu)
     (at 375.04845 97.631692 90)
@@
   )
   (module Keeb_footprints:MX100_slot (layer F.Cu)
-    (at 389.33601 107.1567)
+    (at 389.360818 107.143896)
     (fp_text reference U61 (at 0.0127 1.8288) (layer Dwgs.User)
       (effects (font (size 1 1) (thickness 0.15)))
