File: 01.1_non-snap-off/01_ori/ori.kicad_pcb (KiCad board)
At the start: 2 copper layers, 250 x 76.5 mm, 141 parts, among them J1 TYPE-C-31-M12_13, J2 AVR-ISP-6_mod, K1 KEYSW, K10 KEYSW, K11 KEYSW, K12 KEYSW, K13 KEYSW, K14 KEYSW, K15 KEYSW, K16 KEYSW, K17 KEYSW, K18 KEYSW, K19 KEYSW, K2 KEYSW, K20 KEYSW, K21 KEYSW, K22 KEYSW, K23 KEYSW, K24 KEYSW, K25 KEYSW, K26 KEYSW, K27 KEYSW, K28 KEYSW, K29 KEYSW, K3 KEYSW, K30 KEYSW, K31 KEYSW, K32 KEYSW, K33 KEYSW, K34 KEYSW, K35 KEYSW, K36 KEYSW, K37 KEYSW, K38 KEYSW, K39 KEYSW, K4 KEYSW, K40 KEYSW, K41 KEYSW, K42 KEYSW, K43 KEYSW, K44 KEYSW, K45 KEYSW, K46 KEYSW, K47 KEYSW, K48 KEYSW, K49 KEYSW, K5 KEYSW, K50 KEYSW, K51 KEYSW, K52 KEYSW, K6 KEYSW, K7 KEYSW, K8 KEYSW, K9 KEYSW, SW1 SW_PUSH, SW2 Rotary_Encoder_Switch, U1 ATMEGA32U4, U3 USBLC6-2SC6, Y1 16MHz

Commit message: update column names
Connections:
- J2 pad 3: col0 -> col11
- J2 pad 4: col11 -> col10
- J2 pad 5: col10 -> col9
- K1 pad 1: col1 -> col0
- K10 pad 1: col10 -> col9
- K11 pad 1: col11 -> col10
- K12 pad 1: col0 -> col11
- K13 pad 1: col1 -> col0
- K14 pad 1: col2 -> col1
- K15 pad 1: col3 -> col2
- K16 pad 1: col4 -> col3
- K17 pad 1: col5 -> col4
- K18 pad 1: col6 -> col5
- K19 pad 1: col7 -> col6
- K2 pad 1: col2 -> col1
- K20 pad 1: col8 -> col7
- K21 pad 1: col9 -> col8
- K22 pad 1: col10 -> col9
- K23 pad 1: col11 -> col10
- K24 pad 1: col0 -> col11
- K25 pad 1: col1 -> col0
- K26 pad 1: col2 -> col1
- K27 pad 1: col3 -> col2
- K28 pad 1: col4 -> col3
- K29 pad 1: col5 -> col4
- K3 pad 1: col3 -> col2
- K30 pad 1: col6 -> col5
- K31 pad 1: col7 -> col6
- K32 pad 1: col8 -> col7
- K33 pad 1: col9 -> col8
- K34 pad 1: col10 -> col9
- K35 pad 1: col11 -> col10
- K36 pad 1: col0 -> col11
- K37 pad 1: col1 -> col0
- K38 pad 1: col2 -> col1
- K39 pad 1: col3 -> col2
- K4 pad 1: col4 -> col3
- K40 pad 1: col4 -> col3
- K41 pad 1: col5 -> col4
- K42 pad 1: col6 -> col5
- K43 pad 1: col7 -> col6
- K44 pad 1: col8 -> col7
- K45 pad 1: col9 -> col8
- K46 pad 1: col10 -> col9
- K47 pad 1: col11 -> col10
- K48 pad 1: col0 -> col11
- K5 pad 1: col5 -> col4
- K6 pad 1: col6 -> col5
- K7 pad 1: col7 -> col6
- K8 pad 1: col8 -> col7
- K9 pad 1: col9 -> col8
- U1 pad 1: col8 -> col7
- U1 pad 10: col11 -> col10
- U1 pad 11: col0 -> col11
- U1 pad 12: col3 -> col2
- U1 pad 22: col2 -> col1
- U1 pad 27: col1 -> col0
- U1 pad 38: col4 -> col3
- U1 pad 39: col5 -> col4
- U1 pad 40: col6 -> col5
- U1 pad 41: col7 -> col6
- U1 pad 8: col9 -> col8
- U1 pad 9: col10 -> col9
Routing:
- net col0: track 358.5 -> 83.0 mm, vias 2 -> 1
- net col9: track 173.1 -> 266.1 mm, vias 1 -> 2
- net col11: track 310.7 -> 358.5 mm
- net col10: track 266.1 -> 310.7 mm
- net col2: track 103.3 -> 63.2 mm, vias 0 -> 3
- net col3: track 63.2 -> 100.1 mm
- net col1: track 83.0 -> 103.3 mm, vias 1 -> 0
- net col4: track 100.1 -> 118.5 mm
- net col5: track 118.5 -> 136.7 mm
- net col6: track 136.7 -> 154.7 mm
- net col8: track 158.3 -> 173.1 mm, vias 3 -> 1
- net col7: track 154.7 -> 158.3 mm

Commit message: moved mounting holes
Parts:
- removed H17, H18: MountingHole, random-keyboard-parts:plate_hole_4mm_tht
- moved H14 14.3 mm to (167.8, 102.8)
- moved H15 14.3 mm to (167.8, 64.7)
- moved H16 9.52 mm to (239.3, 64.7)
- moved H13 9.52 mm to (239.3, 102.8)
Other:
- outline, holes or cut-outs redrawn
- board text added: "Ori Rev 1.1"
- board text added: "Ori Rev. 1.1 2021.09.03"
- board text removed: "Ori Rev 1.0"
- board text removed: "Ori Rev. 1.0 2021.08.22"
