File: 01.1_non-snap-off/03_bottom_plate/ori_bottom_plate.kicad_pcb (KiCad board)
At the start: 2 copper layers, 252.4 x 82.2 mm, 62 parts, among them U1 HOLE, U10 HOLE, U11 HOLE, U12 HOLE, U13 HOLE, U14 HOLE, U15 HOLE, U16 HOLE, U17 HOLE, U18 HOLE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

Commit message: moved mounting holes
Parts:
- moved H5 44.1 mm to (312.0, 39.9)
- moved H6 44.1 mm to (312.0, 117.3)
- moved H3 27.4 mm to (233.4, 39.9)
- moved H4 27.4 mm to (233.4, 117.3)
- moved H1 9.52 mm to (156.0, 39.9)
- moved H2 9.52 mm to (156.0, 117.3)
Other:
- outline, holes or cut-outs redrawn
