File: 01_ori/ori.sch (KiCad schematic (older format))
At the start: 131 parts, among them J1 TYPE-C-31-M12_13, J2 AVR-ISP-6_mod, K1 KEYSW, K10 KEYSW, K11 KEYSW, K12 KEYSW, K13 KEYSW, K14 KEYSW, K15 KEYSW, K16 KEYSW, K17 KEYSW, K18 KEYSW, K19 KEYSW, K2 KEYSW, K20 KEYSW, K21 KEYSW, K22 KEYSW, K23 KEYSW, K24 KEYSW, K25 KEYSW, K26 KEYSW, K27 KEYSW, K28 KEYSW, K29 KEYSW, K3 KEYSW, K30 KEYSW, K31 KEYSW, K32 KEYSW, K33 KEYSW, K34 KEYSW, K35 KEYSW, K36 KEYSW, K37 KEYSW, K38 KEYSW, K39 KEYSW, K4 KEYSW, K40 KEYSW, K41 KEYSW, K42 KEYSW, K43 KEYSW, K44 KEYSW, K45 KEYSW, K46 KEYSW, K47 KEYSW, K48 KEYSW, K49 KEYSW, K5 KEYSW, K50 KEYSW, K51 KEYSW, K52 KEYSW, K6 KEYSW, K7 KEYSW, K8 KEYSW, K9 KEYSW, SW1 SW_PUSH, SW2 Rotary_Encoder_Switch, U1 ATMEGA32U4, U3 USBLC6-2SC6, Y1 16MHz

Commit message: new ESD protection
Parts:
- removed C7: 4.7nF, Capacitor_SMD:C_0805_2012Metric_Pad1.15x1.40mm_HandSolder, symbol Device:C_Small
- removed CESD1: .1uF, Capacitor_SMD:C_0805_2012Metric_Pad1.15x1.40mm_HandSolder, symbol Device:C_Small
- removed R5: 1M, Resistor_SMD:R_0805_2012Metric_Pad1.15x1.40mm_HandSolder, symbol Device:R_Small
- removed U3: USBLC6-2SC6, acheron_Components:SOT-23-6, symbol Ori-rescue:Power_Protection_USBLC6-2SC6-shark-cache
- added R? (x2): 22, Resistor_SMD:R_0805_2012Metric_Pad1.15x1.40mm_HandSolder, symbol Device:R
- added U? (x2): PRTR5V0U2X, symbol keyboard_parts:PRTR5V0U2X
Connections:
- net D+: now also R?.1
- net D-: now also R?.1
- net DBUS+: now also R3.2, U?.2 (I01); no longer J1.A6 (D+), J1.B6 (D+)
- net DBUS-: now also R2.2, U?.3 (I02); no longer J1.A7 (D-), J1.B7 (D-)
- net GND: now also J1.S (SHIELD), U?.1 (GND), U?.1 (GND)
- net VBUS: now also U?.4 (VCC), U?.4 (VCC)
- new net: J1.A6 (D+), J1.B6 (D+), R?.2, U?.2 (I01)
- new net: J1.A7 (D-), J1.B7 (D-), R?.2, U?.3 (I02)
Other:
- moved on the sheet: R2, R3
Changed lines of the file:
@@
 	1    0    0    -1
 $EndComp
-Wire Wire Line
-	2750 6550 2750 6600
-Wire Wire Line
-	2750 6850 2750 6900
-Wire Wire Line
-	2800 6600 2750 6600
-Connection ~ 2750 6600
-Wire Wire Line
-	2750 6600 2750 6650
-Wire Wire Line
-	2800 6900 2750 6900
-Connection ~ 2750 6900
-Wire Wire Line
-	2750 6900 2750 6950
 Connection ~ 4750 5800
 Text GLabel 5300 6800 0    50   Input ~ 0
@@
 Text GLabel 5300 6900 0    50   Input ~ 0
 XTAL2
-Text GLabel 2800 6900 2    50   BiDi ~ 0
+Text GLabel 3250 7750 2    50   BiDi ~ 0
 DBUS+
-Text GLabel 2800 6600 2    50   BiDi ~ 0
+Text GLabel 3250 7450 2    50   BiDi ~ 0
 DBUS-
 Text GLabel 7450 6000 2    50   Output ~ 0
@@
 col5
 NoConn ~ 7450 5500
-Text GLabel 5300 9300 2    50   BiDi ~ 0
-D+
-Text GLabel 4600 9300 0    50   BiDi ~ 0
-DBUS+
-Text GLabel 4600 8200 0    50   BiDi ~ 0
-DBUS-
-Text GLabel 5300 8200 2    50   BiDi ~ 0
-D-
-Wire Wire Line
-	4900 8250 4900 8200
-Wire Wire Line
-	4900 8200 5000 8200
-Wire Wire Line
-	4900 9250 4900 9300
-Wire Wire Line
-	4900 9300 5000 9300
-Wire Wire Line
-	4700 9250 4700 9300
-Wire Wire Line
-	4700 9300 4600 9300
-Wire Wire Line
-	4600 8200 4700 8200
-Wire Wire Line
-	4700 8200 4700 8250
-$Comp
-L power:GND #PWR0122
-U 1 1 5E1D89BD
-P 4300 8750
-F 0 "#PWR0122" H 4300 8500 50  0001 C CNN
-F 1 "GND" V 4305 8622 50  0000 R CNN
-F 2 "" H 4300 8750 50  0001 C CNN
-F 3 "" H 4300 8750 50  0001 C CNN
-	1    4300 8750
-	0    1    1    0
-$EndComp
-Text GLabel 5500 8750 2    50   Input ~ 0
-VBUS
-$Comp
-L Ori-rescue:Power_Protection_USBLC6-2SC6-shark-cache U3
-U 1 1 5E0D13FE
-P 4800 8750
-F 0 "U3" V 4600 8900 50  0000 L CNN
-F 1 "USBLC6-2SC6" V 5050 8550 39  0000 L CNN
-F 2 "acheron_Components:SOT-23-6" H 4050 9150 50  0001 C CNN
-F 3 "" H 5000 9100 50  0001 C CNN
-	1    4800 8750
-	0    1    1    0
-$EndComp
 Wire Wire Line
 	2750 5400 2750 5450
@@
 Wire Wire Line
 	4750 5800 4900 5800
-$Comp
-L Device:R R3
-U 1 1 5E44C75B
-P 5150 9300
-F 0 "R3" V 5150 9250 28  0000 C CNN
-F 1 "22" V 5150 9350 28  0000 C CNN
-F 2 "Resistor_SMD:R_0805_2012Metric_Pad1.15x1.40mm_HandSolder" V 5080 9300 50  0001 C CNN
-F 3 "~" H 5150 9300 50  0001 C CNN
-	1    5150 9300
-	0    1    1    0
-$EndComp
-$Comp
-L Device:R R2
-U 1 1 5E4290AE
-P 5150 8200
-F 0 "R2" V 5150 8150 28  0000 C CNN
-F 1 "22" V 5150 8250 28  0000 C CNN
-F 2 "Resistor_SMD:R_0805_2012Metric_Pad1.15x1.40mm_HandSolder" V 5080 8200 50  0001 C CNN
-F 3 "~" H 5150 8200 50  0001 C CNN
-	1    5150 8200
-	0    1    1    0
-$EndComp
 Text GLabel 7450 5900 2    50   Output ~ 0
 col3
@@
 	0    1    1    0
 $EndComp
-Text Notes 4900 9500 0    50   ~ 0
-ESD Protection
 Wire Notes Line
 	3950 8100 3950 9550
@@
 	1    0    0    -1
 $EndComp
-$Comp
-L power:GND #PWR0136
-U 1 1 5FDDBA62
-P 1750 8350
-F 0 "#PWR0136" H 1750 8100 50  0001 C CNN
-F 1 "GND" H 1755 8177 50  0000 C CNN
-F 2 "" H 1750 8350 50  0001 C CNN
-F 3 "" H 1750 8350 50  0001 C CNN
-	1    1750 8350
-	1    0    0    -1
-$EndComp
-$Comp
-L Device:C_Small CESD1
-U 1 1 602BCDFE
-P 5400 8900
-F 0 "CESD1" H 5492 8929 28  0000 L CNN
-F 1 ".1uF" H 5492 8872 28  0000 L CNN
-F 2 "Capacitor_SMD:C_0805_2012Metric_Pad1.15x1.40mm_HandSolder" H 5400 8900 50  0001 C CNN
-F 3 "~" H 5400 8900 50  0001 C CNN
-	1    5400 8900
-	1    0    0    -1
-$EndComp
-$Comp
-L power:GND #PWR0137
-U 1 1 602BE2EB
-P 5400 9000
-F 0 "#PWR0137" H 5400 8750 50  0001 C CNN
-F 1 "GND" H 5405 8827 50  0000 C CNN
-F 2 "" H 5400 9000 50  0001 C CNN
-F 3 "" H 5400 9000 50  0001 C CNN
-	1    5400 9000
-	1    0    0    -1
-$EndComp
-Wire Wire Line
-	5300 8750 5400 8750
-Wire Wire Line
-	5400 8750 5400 8800
-Connection ~ 5400 8750
-Wire Wire Line
-	5400 8750 5500 8750
 Wire Notes Line
 	5800 8100 5800 9550
@@
 Text GLabel 7450 5600 2    50   Output ~ 0
 col6
-Wire Wire Line
-	1750 8300 1850 8300
-Connection ~ 1750 8300
-Wire Wire Line
-	1750 8350 1750 8300
-Wire Wire Line
-	1650 8300 1750 8300
-Connection ~ 1750 8100
-Wire Wire Line
-	1650 8100 1750 8100
-Wire Wire Line
-	1750 8100 1850 8100
-Wire Wire Line
-	1750 8000 1750 8100
-Wire Wire Line
-	1850 8000 1750 8000
-$Comp
-L Device:C_Small C7
-U 1 1 5FD5C0FE
-P 1650 8200
-F 0 "C7" H 1550 8250 28  0000 L CNN
-F 1 "4.7nF" H 1500 8150 28  0000 L CNN
-F 2 "Capacitor_SMD:C_0805_2012Metric_Pad1.15x1.40mm_HandSolder" H 1650 8200 50  0001 C CNN
-F 3 "~" H 1650 8200 50  0001 C CNN
-	1    1650 8200
-	1    0    0    -1
-$EndComp
-$Comp
-L Device:R_Small R5
-U 1 1 5FD5A7DC
-P 1850 8200
-F 0 "R5" H 1909 8229 28  0000 L CNN
-F 1 "1M" V 1850 8150 28  0000 L CNN
-F 2 "Resistor_SMD:R_0805_2012Metric_Pad1.15x1.40mm_HandSolder" H 1850 8200 50  0001 C CNN
-F 3 "~" H 1850 8200 50  0001 C CNN
-	1    1850 8200
-	1    0    0    -1
-$EndComp
+Text GLabel 5150 8750 2    50   Input ~ 0
+VBUS
+$Comp
+L power:GND #PWR0122
+U 1 1 5E1D89BD
+P 4500 8750
+F 0 "#PWR0122" H 4500 8500 50  0001 C CNN
+F 1 "GND" V 4505 8622 50  0000 R CNN
+F 2 "" H 4500 8750 50  0001 C CNN
+F 3 "" H 4500 8750 50  0001 C CNN
+	1    4500 8750
+	0    1    1    0
+$EndComp
+Text GLabel 5550 9000 3    50   BiDi ~ 0
+DBUS-
+Text GLabel 4100 8950 3    50   BiDi ~ 0
+DBUS+
+$Comp
+L keyboard_parts:PRTR5V0U2X U?
+U 1 1 616D1410
+P 4800 8600
+F 0 "U?" H 4825 8689 50  0000 C CNN
+F 1 "PRTR5V0U2X" H 4825 8590 60  0000 C CNN
+F 2 "" H 4800 8600 50  0001 C CNN
+F 3 "" H 4800 8600 50  0001 C CNN
+	1    4800 8600
+	1    0    0    -1
+$EndComp
+Text GLabel 3250 7150 2    50   BiDi ~ 0
+D+
+$Comp
+L Device:R R3
+U 1 1 5E44C75B
+P 4300 9050
+F 0 "R3" V 4300 9000 28  0000 C CNN
+F 1 "22" V 4300 9100 28  0000 C CNN
+F 2 "Resistor_SMD:R_0805_2012Metric_Pad1.15x1.40mm_HandSolder" V 4230 9050 50  0001 C CNN
+F 3 "~" H 4300 9050 50  0001 C CNN
+	1    4300 9050
+	-1   0    0    1
+$EndComp
+Text Notes 4900 9500 0    50   ~ 0
+ESD Protection
+$Comp
+L keyboard_parts:PRTR5V0U2X U?
+U 1 1 61869AB0
+P 3350 6600
+F 0 "U?" H 3400 6550 50  0000 C CNN
+F 1 "PRTR5V0U2X" H 3350 6200 60  0000 C CNN
+F 2 "" H 3350 6600 50  0001 C CNN
+F 3 "" H 3350 6600 50  0001 C CNN
+	1    3350 6600
+	1    0    0    -1
+$EndComp
+Wire Wire Line
+	3050 6900 2950 6900
+Connection ~ 2950 6900
+Wire Wire Line
+	2950 6900 2950 7150
+Wire Wire Line
+	2750 6550 2750 6600
+Wire Wire Line
+	2750 6850 2750 6900
+Wire Wire Line
+	2750 6900 2950 6900
+Connection ~ 2750 6900
+Wire Wire Line
+	2750 6900 2750 6950
+Connection ~ 2750 6600
+Wire Wire Line
+	2750 6600 2750 6650
+Wire Wire Line
+	3800 6900 3800 7150
+Connection ~ 3800 6900
+Wire Wire Line
+	3800 6900 3700 6900
+Wire Wire Line
+	4500 8900 4300 8900
+Wire Wire Line
+	4100 8900 4100 8950
+Wire Wire Line
+	5550 8900 5550 9000
+Text GLabel 4300 9200 3    50   BiDi ~ 0
+D+
+$Comp
+L Device:R R?
+U 1 1 61AB31D0
+P 3100 7150
+F 0 "R?" V 3100 7100 28  0000 C CNN
+F 1 "22" V 3100 7200 28  0000 C CNN
+F 2 "Resistor_SMD:R_0805_2012Metric_Pad1.15x1.40mm_HandSolder" V 3030 7150 50  0001 C CNN
+F 3 "~" H 3100 7150 50  0001 C CNN
+	1    3100 7150
+	0    1    1    0
+$EndComp
+Wire Wire Line
+	5150 8900 5350 8900
+$Comp
+L Device:R R2
+U 1 1 5E4290AE
+P 5350 9050
+F 0 "R2" V 5350 9000 28  0000 C CNN
+F 1 "22" V 5350 9100 28  0000 C CNN
+F 2 "Resistor_SMD:R_0805_2012Metric_Pad1.15x1.40mm_HandSolder" V 5280 9050 50  0001 C CNN
+F 3 "~" H 5350 9050 50  0001 C CNN
+	1    5350 9050
+	-1   0    0    1
+$EndComp
+Text GLabel 4100 7150 2    50   BiDi ~ 0
+D-
+$Comp
+L Device:R R?
+U 1 1 61B0952A
+P 3950 7150
+F 0 "R?" V 3950 7100 28  0000 C CNN
+F 1 "22" V 3950 7200 28  0000 C CNN
+F 2 "Resistor_SMD:R_0805_2012Metric_Pad1.15x1.40mm_HandSolder" V 3880 7150 50  0001 C CNN
+F 3 "~" H 3950 7150 50  0001 C CNN
+	1    3950 7150
+	0    1    1    0
+$EndComp
+Text GLabel 5350 9200 3    50   BiDi ~ 0
+D-
+$Comp
+L power:GND #PWR?
+U 1 1 61B33909
+P 3050 6750
+F 0 "#PWR?" H 3050 6500 50  0001 C CNN
+F 1 "GND" V 3055 6622 50  0000 R CNN
+F 2 "" H 3050 6750 50  0001 C CNN
+F 3 "" H 3050 6750 50  0001 C CNN
+	1    3050 6750
+	0    1    1    0
+$EndComp
+Text GLabel 3700 6750 2    50   Input ~ 0
+VBUS
+Wire Wire Line
+	4000 6600 4000 6900
+Wire Wire Line
+	3900 6900 3800 6900
+Wire Wire Line
+	2750 6600 4000 6600
+Wire Wire Line
+	3800 6900 4000 6900
 $Comp
 L Ori-rescue:TYPE-C-31-M12_13-acheronSymbols J1
@@
 	1    0    0    -1
 $EndComp
+Wire Wire Line
+	1850 8000 2050 8000
+Connection ~ 2050 8000
+Connection ~ 4300 8900
+Wire Wire Line
+	4300 8900 4100 8900
+Connection ~ 5350 8900
+Wire Wire Line
+	5350 8900 5550 8900
 $EndSCHEMATC

Commit message: update rev silkscreen
Parts:
- removed R? (x2): 22, Resistor_SMD:R_0805_2012Metric_Pad1.15x1.40mm_HandSolder, symbol Device:R
- removed U?: PRTR5V0U2X, symbol keyboard_parts:PRTR5V0U2X
- U2: renamed from U?; footprint (none) -> Keebio-Parts:SOT-143B
Connections:
- net DBUS+: now also J1.A6 (D+), J1.B6 (D+)
- net DBUS-: now also J1.A7 (D-), J1.B7 (D-)
Changed lines of the file:
@@
 Text GLabel 5300 6900 0    50   Input ~ 0
 XTAL2
-Text GLabel 3250 7750 2    50   BiDi ~ 0
-DBUS+
-Text GLabel 3250 7450 2    50   BiDi ~ 0
-DBUS-
 Text GLabel 7450 6000 2    50   Output ~ 0
 row1
@@
 	0    1    1    0
 $EndComp
-Wire Notes Line
-	3950 8100 3950 9550
 Text GLabel 4800 6650 0    50   Input ~ 0
 ISP_Reset
@@
 $EndComp
 Wire Notes Line
-	5800 8100 5800 9550
-Wire Notes Line
-	3950 8100 5800 8100
-Wire Notes Line
 	3950 9550 5800 9550
 $Comp
@@
 DBUS+
 $Comp
-L keyboard_parts:PRTR5V0U2X U?
+L keyboard_parts:PRTR5V0U2X U2
 U 1 1 616D1410
 P 4800 8600
-F 0 "U?" H 4825 8689 50  0000 C CNN
+F 0 "U2" H 4825 8689 50  0000 C CNN
 F 1 "PRTR5V0U2X" H 4825 8590 60  0000 C CNN
-F 2 "" H 4800 8600 50  0001 C CNN
+F 2 "Keebio-Parts:SOT-143B" H 4800 8600 50  0001 C CNN
 F 3 "" H 4800 8600 50  0001 C CNN
 	1    4800 8600
 	1    0    0    -1
 $EndComp
-Text GLabel 3250 7150 2    50   BiDi ~ 0
-D+
 $Comp
 L Device:R R3
@@
 Text Notes 4900 9500 0    50   ~ 0
 ESD Protection
-$Comp
-L keyboard_parts:PRTR5V0U2X U?
-U 1 1 61869AB0
-P 3350 6600
-F 0 "U?" H 3400 6550 50  0000 C CNN
-F 1 "PRTR5V0U2X" H 3350 6200 60  0000 C CNN
-F 2 "" H 3350 6600 50  0001 C CNN
-F 3 "" H 3350 6600 50  0001 C CNN
-	1    3350 6600
-	1    0    0    -1
-$EndComp
-Wire Wire Line
-	3050 6900 2950 6900
-Connection ~ 2950 6900
-Wire Wire Line
-	2950 6900 2950 7150
-Wire Wire Line
-	2750 6550 2750 6600
-Wire Wire Line
-	2750 6850 2750 6900
-Wire Wire Line
-	2750 6900 2950 6900
-Connection ~ 2750 6900
-Wire Wire Line
-	2750 6900 2750 6950
-Connection ~ 2750 6600
-Wire Wire Line
-	2750 6600 2750 6650
-Wire Wire Line
-	3800 6900 3800 7150
-Connection ~ 3800 6900
-Wire Wire Line
-	3800 6900 3700 6900
 Wire Wire Line
 	4500 8900 4300 8900
@@
 Text GLabel 4300 9200 3    50   BiDi ~ 0
 D+
-$Comp
-L Device:R R?
-U 1 1 61AB31D0
-P 3100 7150
-F 0 "R?" V 3100 7100 28  0000 C CNN
-F 1 "22" V 3100 7200 28  0000 C CNN
-F 2 "Resistor_SMD:R_0805_2012Metric_Pad1.15x1.40mm_HandSolder" V 3030 7150 50  0001 C CNN
-F 3 "~" H 3100 7150 50  0001 C CNN
-	1    3100 7150
-	0    1    1    0
-$EndComp
 Wire Wire Line
 	5150 8900 5350 8900
@@
 	-1   0    0    1
 $EndComp
-Text GLabel 4100 7150 2    50   BiDi ~ 0
-D-
-$Comp
-L Device:R R?
-U 1 1 61B0952A
-P 3950 7150
-F 0 "R?" V 3950 7100 28  0000 C CNN
-F 1 "22" V 3950 7200 28  0000 C CNN
-F 2 "Resistor_SMD:R_0805_2012Metric_Pad1.15x1.40mm_HandSolder" V 3880 7150 50  0001 C CNN
-F 3 "~" H 3950 7150 50  0001 C CNN
-	1    3950 7150
-	0    1    1    0
-$EndComp
 Text GLabel 5350 9200 3    50   BiDi ~ 0
 D-
-$Comp
-L power:GND #PWR?
-U 1 1 61B33909
-P 3050 6750
-F 0 "#PWR?" H 3050 6500 50  0001 C CNN
-F 1 "GND" V 3055 6622 50  0000 R CNN
-F 2 "" H 3050 6750 50  0001 C CNN
-F 3 "" H 3050 6750 50  0001 C CNN
-	1    3050 6750
-	0    1    1    0
-$EndComp
-Text GLabel 3700 6750 2    50   Input ~ 0
-VBUS
-Wire Wire Line
-	4000 6600 4000 6900
-Wire Wire Line
-	3900 6900 3800 6900
-Wire Wire Line
-	2750 6600 4000 6600
-Wire Wire Line
-	3800 6900 4000 6900
 $Comp
 L Ori-rescue:TYPE-C-31-M12_13-acheronSymbols J1
@@
 Wire Wire Line
 	5350 8900 5550 8900
+Text GLabel 2800 6600 2    50   BiDi ~ 0
+DBUS-
+Text GLabel 2800 6900 2    50   BiDi ~ 0
+DBUS+
+Wire Wire Line
+	2750 6550 2750 6600
+Wire Wire Line
+	2750 6850 2750 6900
+Wire Wire Line
+	2800 6600 2750 6600
+Connection ~ 2750 6600
+Wire Wire Line
+	2750 6600 2750 6650
+Wire Wire Line
+	2800 6900 2750 6900
+Connection ~ 2750 6900
+Wire Wire Line
+	2750 6900 2750 6950
+Wire Notes Line
+	3950 9550 3950 8400
+Wire Notes Line
+	3950 8400 5800 8400
+Wire Notes Line
+	5800 8400 5800 9550
 $EndSCHEMATC
