File: 02_top_plate/ori_top_plate.sch (KiCad schematic (older format))
At the start: 69 parts, among them U1 HOLE, U10 HOLE, U11 HOLE, U12 HOLE, U13 HOLE, U14 HOLE, U15 HOLE, U16 HOLE, U17 HOLE, U18 HOLE, U19 HOLE, U2 HOLE, U20 HOLE, U21 HOLE, U22 HOLE, U23 HOLE, U24 HOLE, U25 HOLE, U26 HOLE, U27 HOLE, U28 HOLE, U29 HOLE, U3 HOLE, U30 HOLE, U31 HOLE, U32 HOLE, U33 HOLE, U34 HOLE, U35 HOLE, U36 HOLE, U37 HOLE, U38 HOLE, U39 HOLE, U4 HOLE, U40 HOLE, U41 HOLE, U42 HOLE, U43 HOLE, U44 HOLE, U45 HOLE, U46 HOLE, U47 HOLE, U48 HOLE, U49 HOLE, U5 HOLE, U50 HOLE, U51 HOLE, U52 HOLE, U6 HOLE, U7 HOLE, U8 HOLE, U9 HOLE

Commit message: update rev silkscreen
Parts:
- removed H10, H11, H12, H13, H14, H17, H18, H9: MountingHole, MountingHole:MountingHole_2.2mm_M2_DIN965, symbol Mechanical:MountingHole
Other:
- note removed: "Tray mount holes"
Changed lines of the file:
@@
 Wire Notes Line
 	2350 4350 2350 3250
-$Comp
-L Mechanical:MountingHole H9
-U 1 1 6122943F
-P 4300 3450
-F 0 "H9" H 4400 3496 50  0000 L CNN
-F 1 "MountingHole" H 4400 3405 50  0000 L CNN
-F 2 "MountingHole:MountingHole_2.2mm_M2_DIN965" H 4300 3450 50  0001 C CNN
-F 3 "~" H 4300 3450 50  0001 C CNN
-	1    4300 3450
-	1    0    0    -1
-$EndComp
-$Comp
-L Mechanical:MountingHole H10
-U 1 1 61229445
-P 4300 3650
-F 0 "H10" H 4400 3696 50  0000 L CNN
-F 1 "MountingHole" H 4400 3605 50  0000 L CNN
-F 2 "MountingHole:MountingHole_2.2mm_M2_DIN965" H 4300 3650 50  0001 C CNN
-F 3 "~" H 4300 3650 50  0001 C CNN
-	1    4300 3650
-	1    0    0    -1
-$EndComp
-$Comp
-L Mechanical:MountingHole H11
-U 1 1 6122944B
-P 4300 3850
-F 0 "H11" H 4400 3896 50  0000 L CNN
-F 1 "MountingHole" H 4400 3805 50  0000 L CNN
-F 2 "MountingHole:MountingHole_2.2mm_M2_DIN965" H 4300 3850 50  0001 C CNN
-F 3 "~" H 4300 3850 50  0001 C CNN
-	1    4300 3850
-	1    0    0    -1
-$EndComp
-$Comp
-L Mechanical:MountingHole H12
-U 1 1 61229451
-P 4300 4050
-F 0 "H12" H 4400 4096 50  0000 L CNN
-F 1 "MountingHole" H 4400 4005 50  0000 L CNN
-F 2 "MountingHole:MountingHole_2.2mm_M2_DIN965" H 4300 4050 50  0001 C CNN
-F 3 "~" H 4300 4050 50  0001 C CNN
-	1    4300 4050
-	1    0    0    -1
-$EndComp
-$Comp
-L Mechanical:MountingHole H13
-U 1 1 61229457
-P 5150 3650
-F 0 "H13" H 5250 3696 50  0000 L CNN
-F 1 "MountingHole" H 5250 3605 50  0000 L CNN
-F 2 "MountingHole:MountingHole_2.2mm_M2_DIN965" H 5150 3650 50  0001 C CNN
-F 3 "~" H 5150 3650 50  0001 C CNN
-	1    5150 3650
-	1    0    0    -1
-$EndComp
-$Comp
-L Mechanical:MountingHole H14
-U 1 1 6122945D
-P 5150 3450
-F 0 "H14" H 5250 3496 50  0000 L CNN
-F 1 "MountingHole" H 5250 3405 50  0000 L CNN
-F 2 "MountingHole:MountingHole_2.2mm_M2_DIN965" H 5150 3450 50  0001 C CNN
-F 3 "~" H 5150 3450 50  0001 C CNN
-	1    5150 3450
-	1    0    0    -1
-$EndComp
-Text Notes 4650 4250 0    50   ~ 0
-Tray mount holes
-Wire Notes Line
-	5850 4350 4150 4350
-$Comp
-L Mechanical:MountingHole H17
-U 1 1 61235A30
-P 5150 3850
-F 0 "H17" H 5250 3896 50  0000 L CNN
-F 1 "MountingHole" H 5250 3805 50  0000 L CNN
-F 2 "MountingHole:MountingHole_2.2mm_M2_DIN965" H 5150 3850 50  0001 C CNN
-F 3 "~" H 5150 3850 50  0001 C CNN
-	1    5150 3850
-	1    0    0    -1
-$EndComp
-$Comp
-L Mechanical:MountingHole H18
-U 1 1 61235A36
-P 5150 4050
-F 0 "H18" H 5250 4096 50  0000 L CNN
-F 1 "MountingHole" H 5250 4005 50  0000 L CNN
-F 2 "MountingHole:MountingHole_2.2mm_M2_DIN965" H 5150 4050 50  0001 C CNN
-F 3 "~" H 5150 4050 50  0001 C CNN
-	1    5150 4050
-	1    0    0    -1
-$EndComp
-Wire Notes Line
-	5850 4350 5850 3250
-Wire Notes Line
-	5850 3250 4150 3250
-Wire Notes Line
-	4150 3250 4150 4350
 $EndSCHEMATC
