File: 02_top_plate/top_plate.kicad_pcb (KiCad board)
At the start: 2 copper layers, 252.4 x 84.5 mm, 61 parts, among them U1 HOLE, U10 HOLE, U11 HOLE, U12 HOLE, U13 HOLE, U14 HOLE, U15 HOLE, U16 HOLE, U17 HOLE, U18 HOLE, U19 HOLE, U2 HOLE, U20 HOLE, U21 HOLE, U22 HOLE, U23 HOLE, U24 HOLE, U25 HOLE, U26 HOLE, U27 HOLE, U28 HOLE, U29 HOLE, U3 HOLE, U30 HOLE, U31 HOLE, U32 HOLE, U33 HOLE, U34 HOLE, U35 HOLE, U36 HOLE, U37 HOLE, U38 HOLE, U39 HOLE, U4 HOLE, U40 HOLE, U41 HOLE, U42 HOLE, U43 HOLE, U44 HOLE, U45 HOLE, U46 HOLE, U47 HOLE, U48 HOLE, U49 HOLE, U5 HOLE, U50 HOLE, U51 HOLE, U52 HOLE, U6 HOLE, U7 HOLE, U8 HOLE, U9 HOLE

Commit message: create slots for top plate
Parts:
- removed D2: DIODE, Keeb_footprints:D_SOD-123_modified
- added R1: R_Small, Resistor_SMD:R_0603_1608Metric_Pad1.05x0.95mm_HandSolder, F.Cu at (377.4, 50.0)
- H8: footprint random-keyboard-parts:Generic-Mounthole -> Resistor_SMD:R_0603_1608Metric_Pad1.05x0.95mm_HandSolder
- U1, U10, U11, U12, U13, U14, U15, U16, U17, U18, U19, U2, U20, U21, U22, U23, U24, U25, U26, U27, U28, U29, U3, U30, U31, U32, U33, U34, U35, U36, U37, U38, U39, U4, U40, U41, U42, U43, U44, U45, U46, U47, U48, U49, U5, U50, U51, U52, U6, U7, U8, U9: footprint Keeb_footprints:MX100_cutout_plated -> Keeb_footprints:MX100_slot_plated
Routing:
- net GND1: track 2.52 -> 0.00 mm, vias 1 -> 0
- net GND: track 2.52 -> 1.51 mm
Other:
- board size 252.4 x 84.5 mm -> 252.4 x 85.7 mm

Commit message: update bottom plate
Parts:
- H8: footprint Resistor_SMD:R_0603_1608Metric_Pad1.05x0.95mm_HandSolder -> random-keyboard-parts:Generic-Mounthole
- R1: moved to B.Cu
- turned R1 to 270 degrees
Routing:
- net GND: track 1.51 -> 0.00 mm, vias 1 -> 0
- net (no net): track 0.00 -> 1.51 mm, vias 0 -> 1
Changed lines of the file:
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@@
     (uvia_drill 0.25)
     (add_net GND)
-    (add_net "Net-(R1-Pad2)")
   )
   (net_class Thick ""
@@
     (uvia_drill 0.2)
   )
-  (module Resistor_SMD:R_0603_1608Metric_Pad1.05x0.95mm_HandSolder (layer F.Cu)
-    (at 377.42967 50.00646 90)
-    (descr "Resistor SMD 0603 (1608 Metric), square (rectangular) end terminal, IPC_7351 nominal with elongated pad for handsoldering. (Body size source: http://www.tortai-tech.com/upload/download/2011102023233369053.pdf), generated with kicad-footprint-generator")
-    (tags "resistor handsolder")
-    (attr smd)
-    (fp_text reference R1 (at 0 -1.43 90) (layer Dwgs.User)
+  (module random-keyboard-parts:Generic-Mounthole (layer F.Cu)
+    (at 389.33589 118.46734)
+    (attr virtual)
+    (fp_text reference H8 (at 0 2) (layer Dwgs.User)
       (effects (font (size 1 1) (thickness 0.15)))
     )
-    (fp_text value R_Small (at 0 1.43 90) (layer F.Fab)
+    (fp_text value MountingHole (at 0 -2) (layer Dwgs.User)
       (effects (font (size 1 1) (thickness 0.15)))
     )
-    (fp_text user %R (at 0 0 90) (layer F.Fab)
-      (effects (font (size 0.4 0.4) (thickness 0.06)))
-    )
-    (fp_line (start 1.65 0.73) (end -1.65 0.73) (layer F.CrtYd) (width 0.05))
-    (fp_line (start 1.65 -0.73) (end 1.65 0.73) (layer F.CrtYd) (width 0.05))
-    (fp_line (start -1.65 -0.73) (end 1.65 -0.73) (layer F.CrtYd) (width 0.05))
-    (fp_line (start -1.65 0.73) (end -1.65 -0.73) (layer F.CrtYd) (width 0.05))
-    (fp_line (start 0.8 0.4) (end -0.8 0.4) (layer F.Fab) (width 0.1))
-    (fp_line (start 0.8 -0.4) (end 0.8 0.4) (layer F.Fab) (width 0.1))
-    (fp_line (start -0.8 -0.4) (end 0.8 -0.4) (layer F.Fab) (width 0.1))
-    (fp_line (start -0.8 0.4) (end -0.8 -0.4) (layer F.Fab) (width 0.1))
-    (pad 2 smd roundrect (at 0.875 0 90) (size 1.05 0.95) (layers F.Cu F.Paste F.Mask) (roundrect_rratio 0.25))
-    (pad 1 smd roundrect (at -0.875 0 90) (size 1.05 0.95) (layers F.Cu F.Paste F.Mask) (roundrect_rratio 0.25)
-      (net 1 GND))
-    (model ${KISYS3DMOD}/Resistor_SMD.3dshapes/R_0603_1608Metric.wrl
-      (at (xyz 0 0 0))
-      (scale (xyz 1 1 1))
-      (rotate (xyz 0 0 0))
-    )
+    (pad 1 thru_hole circle (at 0 0) (size 3.5 3.5) (drill 2.2) (layers *.Cu *.Mask))
   )
-  (module Resistor_SMD:R_0603_1608Metric_Pad1.05x0.95mm_HandSolder (layer F.Cu)
-    (at 389.33589 118.46734)
+  (module Resistor_SMD:R_0603_1608Metric_Pad1.05x0.95mm_HandSolder (layer B.Cu)
+    (at 377.42967 50.00646 270)
     (descr "Resistor SMD 0603 (1608 Metric), square (rectangular) end terminal, IPC_7351 nominal with elongated pad for handsoldering. (Body size source: http://www.tortai-tech.com/upload/download/2011102023233369053.pdf), generated with kicad-footprint-generator")
     (tags "resistor handsolder")
     (attr smd)
-    (fp_text reference H8 (at 0 -1.43) (layer F.SilkS)
+    (fp_text reference R1 (at 0 1.43 270) (layer Dwgs.User)
       (effects (font (size 1 1) (thickness 0.15)))
     )
-    (fp_text value MountingHole (at 0 1.43) (layer F.Fab)
-      (effects (font (size 1 1) (thickness 0.15)))
+    (fp_text value R_Small (at 0 -1.43 270) (layer B.Fab)
+      (effects (font (size 1 1) (thickness 0.15)) (justify mirror))
     )
-    (fp_text user %R (at 0 0) (layer F.Fab)
-      (effects (font (size 0.4 0.4) (thickness 0.06)))
+    (fp_text user %R (at 0 0 270) (layer B.Fab)
+      (effects (font (size 0.4 0.4) (thickness 0.06)) (justify mirror))
     )
-    (fp_line (start 1.65 0.73) (end -1.65 0.73) (layer F.CrtYd) (width 0.05))
-    (fp_line (start 1.65 -0.73) (end 1.65 0.73) (layer F.CrtYd) (width 0.05))
-    (fp_line (start -1.65 -0.73) (end 1.65 -0.73) (layer F.CrtYd) (width 0.05))
-    (fp_line (start -1.65 0.73) (end -1.65 -0.73) (layer F.CrtYd) (width 0.05))
-    (fp_line (start -0.171267 0.51) (end 0.171267 0.51) (layer F.SilkS) (width 0.12))
-    (fp_line (start -0.171267 -0.51) (end 0.171267 -0.51) (layer F.SilkS) (width 0.12))
-    (fp_line (start 0.8 0.4) (end -0.8 0.4) (layer F.Fab) (width 0.1))
-    (fp_line (start 0.8 -0.4) (end 0.8 0.4) (layer F.Fab) (width 0.1))
-    (fp_line (start -0.8 -0.4) (end 0.8 -0.4) (layer F.Fab) (width 0.1))
-    (fp_line (start -0.8 0.4) (end -0.8 -0.4) (layer F.Fab) (width 0.1))
-    (pad 2 smd roundrect (at 0.875 0) (size 1.05 0.95) (layers F.Cu F.Paste F.Mask) (roundrect_rratio 0.25))
-    (pad 1 smd roundrect (at -0.875 0) (size 1.05 0.95) (layers F.Cu F.Paste F.Mask) (roundrect_rratio 0.25))
+    (fp_line (start 1.65 -0.73) (end -1.65 -0.73) (layer B.CrtYd) (width 0.05))
+    (fp_line (start 1.65 0.73) (end 1.65 -0.73) (layer B.CrtYd) (width 0.05))
+    (fp_line (start -1.65 0.73) (end 1.65 0.73) (layer B.CrtYd) (width 0.05))
+    (fp_line (start -1.65 -0.73) (end -1.65 0.73) (layer B.CrtYd) (width 0.05))
+    (fp_line (start 0.8 -0.4) (end -0.8 -0.4) (layer B.Fab) (width 0.1))
+    (fp_line (start 0.8 0.4) (end 0.8 -0.4) (layer B.Fab) (width 0.1))
+    (fp_line (start -0.8 0.4) (end 0.8 0.4) (layer B.Fab) (width 0.1))
+    (fp_line (start -0.8 -0.4) (end -0.8 0.4) (layer B.Fab) (width 0.1))
+    (pad 2 smd roundrect (at 0.875 0 270) (size 1.05 0.95) (layers B.Cu B.Paste B.Mask) (roundrect_rratio 0.25))
+    (pad 1 smd roundrect (at -0.875 0 270) (size 1.05 0.95) (layers B.Cu B.Paste B.Mask) (roundrect_rratio 0.25)
+      (net 1 GND))
     (model ${KISYS3DMOD}/Resistor_SMD.3dshapes/R_0603_1608Metric.wrl
       (at (xyz 0 0 0))
@@
   (gr_arc (start 148.829842 114.300144) (end 146.449842 114.300156) (angle -89.99971111) (layer Edge.Cuts) (width 0.05))
   (gr_arc (start 148.829842 42.862728) (end 148.829842 40.481468) (angle -90) (layer Edge.Cuts) (width 0.05))
-  (gr_text JLCJLCJLCJLC (at 377.42967 107.156508 90) (layer B.SilkS)
+  (gr_text JLCJLCJLCJLC (at 377.42967 107.156508 -90) (layer B.SilkS)
     (effects (font (size 1 1) (thickness 0.15)) (justify mirror))
   )
@@
     (effects (font (size 1.25 1.25) (thickness 0.2)) (justify mirror))
   )
-  (via (at 377.42967 52.387712) (size 0.5) (drill 0.25) (layers F.Cu B.Cu) (net 1))
-  (segment (start 377.42967 50.88146) (end 377.42967 52.387712) (width 0.25) (layer F.Cu) (net 1))
+  (via (at 377.42967 52.387712) (size 0.5) (drill 0.25) (layers F.Cu B.Cu) (net 0))
+  (segment (start 377.42967 52.387712) (end 377.42967 50.88146) (width 0.25) (layer B.Cu) (net 0))
   (zone (net 1) (net_name GND) (layer B.Cu) (hatch edge 0.508)
     (connect_pads (clearance 0))
