File: 03_bottom_plate/ori_bottom_plate.kicad_pcb (KiCad board)
At the start: 2 copper layers, 252.4 x 82.2 mm, 62 parts, among them U1 HOLE, U10 HOLE, U11 HOLE, U12 HOLE, U13 HOLE, U14 HOLE, U15 HOLE, U16 HOLE, U17 HOLE, U18 HOLE, U19 HOLE, U2 HOLE, U20 HOLE, U21 HOLE, U22 HOLE, U23 HOLE, U24 HOLE, U25 HOLE, U26 HOLE, U27 HOLE, U28 HOLE, U29 HOLE, U3 HOLE, U30 HOLE, U31 HOLE, U32 HOLE, U33 HOLE, U34 HOLE, U35 HOLE, U36 HOLE, U37 HOLE, U38 HOLE, U39 HOLE, U4 HOLE, U40 HOLE, U41 HOLE, U42 HOLE, U43 HOLE, U44 HOLE, U45 HOLE, U46 HOLE, U47 HOLE, U48 HOLE, U49 HOLE, U5 HOLE, U53 HOLE, U57 HOLE, U6 HOLE, U61 HOLE, U7 HOLE, U8 HOLE, U9 HOLE

Commit message: move bottom mounting points and update previews
Parts:
- moved H2 1.19 mm to (156.0, 118.5)
- moved H3 1.19 mm to (233.4, 38.7)
- moved H4 1.19 mm to (233.4, 118.5)
- moved H5 1.19 mm to (312.0, 38.7)
- moved H6 1.19 mm to (312.0, 118.5)
- moved H7 1.19 mm to (389.4, 38.7)
- moved H8 1.19 mm to (389.4, 118.5)
- moved H1 1.19 mm to (156.0, 38.7)
Other:
- board size 252.4 x 82.2 mm -> 252.4 x 84.5 mm

Commit message: update rev silkscreen
Other:
- board text added: "ori rev 1.1"
- board text removed: "Ori Rev 1.0"
