File: 03_bottom_plate/lucy_bottom_plate.kicad_pcb (KiCad board)
At the start: 2 copper layers, 252.4 x 84.5 mm, 62 parts, among them U1 HOLE, U10 HOLE, U11 HOLE, U12 HOLE, U13 HOLE, U14 HOLE, U15 HOLE, U16 HOLE, U17 HOLE, U18 HOLE, U19 HOLE, U2 HOLE, U20 HOLE, U21 HOLE, U22 HOLE, U23 HOLE, U24 HOLE, U25 HOLE, U26 HOLE, U27 HOLE, U28 HOLE, U29 HOLE, U3 HOLE, U30 HOLE, U31 HOLE, U32 HOLE, U33 HOLE, U34 HOLE, U35 HOLE, U36 HOLE, U37 HOLE, U38 HOLE, U39 HOLE, U4 HOLE, U40 HOLE, U41 HOLE, U42 HOLE, U43 HOLE, U44 HOLE, U45 HOLE, U46 HOLE, U47 HOLE, U48 HOLE, U49 HOLE, U5 HOLE, U53 HOLE, U57 HOLE, U6 HOLE, U61 HOLE, U7 HOLE, U8 HOLE, U9 HOLE

Commit message: new gerbers with new name
Other:
- board text added: "lucy rev 1.2"
- board text removed: "ori rev 1.1"
Changed lines of the file:
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@@
-(kicad_pcb (version 20171130) (host pcbnew "(5.1.10-1-10_14)")
+(kicad_pcb (version 20171130) (host pcbnew "(5.1.4-0-10_14)")
   (general
     (thickness 1.6)
@@
     (effects (font (size 1.25 1.25) (thickness 0.2)))
   )
-  (gr_text "ori rev 1.1" (at 236.702148 113.136076) (layer F.SilkS)
+  (gr_text "lucy rev 1.2" (at 236.702148 113.136076) (layer F.SilkS)
     (effects (font (size 1.25 1.25) (thickness 0.2)))
   )
