File: 03_bottom_plate/bottom_plate.kicad_pcb (KiCad board)
At the start: 2 copper layers, 252.4 x 84.5 mm, 62 parts, among them U1 HOLE, U10 HOLE, U11 HOLE, U12 HOLE, U13 HOLE, U14 HOLE, U15 HOLE, U16 HOLE, U17 HOLE, U18 HOLE, U19 HOLE, U2 HOLE, U20 HOLE, U21 HOLE, U22 HOLE, U23 HOLE, U24 HOLE, U25 HOLE, U26 HOLE, U27 HOLE, U28 HOLE, U29 HOLE, U3 HOLE, U30 HOLE, U31 HOLE, U32 HOLE, U33 HOLE, U34 HOLE, U35 HOLE, U36 HOLE, U37 HOLE, U38 HOLE, U39 HOLE, U4 HOLE, U40 HOLE, U41 HOLE, U42 HOLE, U43 HOLE, U44 HOLE, U45 HOLE, U46 HOLE, U47 HOLE, U48 HOLE, U49 HOLE, U5 HOLE, U53 HOLE, U57 HOLE, U6 HOLE, U61 HOLE, U7 HOLE, U8 HOLE, U9 HOLE

Commit message: create slots for top plate
Parts:
- removed D1: DIODE, Keeb_footprints:D_SOD-123_modified
- added R1: R_Small, Resistor_SMD:R_0603_1608Metric_Pad1.05x0.95mm_HandSolder, F.Cu at (388.8, 59.5)
- moved H4 7.76 mm to (225.6, 119.1)
- moved H6 7.76 mm to (319.7, 119.1)
- moved H5 7.74 mm to (319.7, 38.7)
- moved H3 7.17 mm to (226.2, 38.1)
- moved H1 5.39 mm to (161.4, 38.1)
- moved H2 5.39 mm to (161.4, 119.1)
- moved H7 5.39 mm to (384.0, 38.1)
- moved H8 5.39 mm to (384.0, 119.1)
Other:
- board size 252.4 x 84.5 mm -> 252.4 x 85.7 mm
