File: 01_lucy-saved/lucy.sch (KiCad schematic (older format))
At the start: 127 parts, among them J1 TYPE-C-31-M12_13, J2 AVR-ISP-6_mod, K1 KEYSW, K10 KEYSW, K11 KEYSW, K12 KEYSW, K13 KEYSW, K14 KEYSW, K15 KEYSW, K16 KEYSW, K17 KEYSW, K18 KEYSW, K19 KEYSW, K2 KEYSW, K20 KEYSW, K21 KEYSW, K22 KEYSW, K23 KEYSW, K24 KEYSW, K25 KEYSW, K26 KEYSW, K27 KEYSW, K28 KEYSW, K29 KEYSW, K3 KEYSW, K30 KEYSW, K31 KEYSW, K32 KEYSW, K33 KEYSW, K34 KEYSW, K35 KEYSW, K36 KEYSW, K37 KEYSW, K38 KEYSW, K39 KEYSW, K4 KEYSW, K40 KEYSW, K41 KEYSW, K42 KEYSW, K43 KEYSW, K44 KEYSW, K45 KEYSW, K46 KEYSW, K47 KEYSW, K48 KEYSW, K49 KEYSW, K5 KEYSW, K50 KEYSW, K51 KEYSW, K52 KEYSW, K6 KEYSW, K7 KEYSW, K8 KEYSW, K9 KEYSW, SW1 SW_PUSH, SW2 Rotary_Encoder_Switch, U1 ATMEGA32U4, U2 PRTR5V0U2X, Y1 16MHz

Commit message: Complete re-routing
Parts:
- added C5: .1uF, Capacitor_SMD:C_0805_2012Metric_Pad1.15x1.40mm_HandSolder, symbol Device:C_Small
Connections:
- net GND: now also C5.2
- net VCC: now also C5.1
- net col0: now also U1.27 (T0/PD7)
- net col1: now also U1.28 (PB4); no longer J2.4 (MOSI), U1.10 (PB2/MOSI)
- net col10: now also J2.4 (MOSI), U1.10 (PB2/MOSI); no longer U1.32 (PC7)
- net col11: now also J2.3 (MISO), U1.11 (PB3/MISO); no longer U1.36 (PF7)
- net col12: now also U1.19 (PD1/INT1); no longer U1.37 (PF6)
- net col2: now also U1.12 (PB7/~RTS); no longer J2.3 (MISO), U1.11 (PB3/MISO)
- net col3: now also U1.38 (PF5); no longer U1.25 (ICP1/PD4)
- net col4: now also U1.39 (PF4); no longer U1.26 (T1/PD6)
- net col5: now also U1.40 (PF1); no longer U1.27 (T0/PD7)
- net col6: now also U1.41 (PF0); no longer U1.28 (PB4)
- net col7: now also U1.1 (PE6/AIN0); no longer U1.29 (PB5)
- net col8: now also U1.8 (PB0/SS); no longer U1.30 (PB6)
- net col9: now also J2.5 (SCK), U1.9 (PB1/SCK); no longer U1.31 (PC6)
- net enc0a: now also U1.21 (PD3/TXD1)
- net enc0b: now also U1.20 (PD2/RXD1)
- net row0: now also U1.36 (PF7); no longer J2.5 (SCK), U1.9 (PB1/SCK)
- net row1: now also U1.37 (PF6)
- net row2: now also U1.25 (ICP1/PD4)
- net row3: now also U1.26 (T1/PD6)
Changed lines of the file:
@@
 Text GLabel 5300 6900 0    50   Input ~ 0
 XTAL2
-Text GLabel 7850 6000 2    50   Output ~ 0
+Text GLabel 7450 6000 2    50   Output ~ 0
 row1
+Text GLabel 7450 6900 2    50   Output ~ 0
+col1
+Text GLabel 5300 6400 0    50   Output ~ 0
+col2
 Text GLabel 5300 6200 0    50   Output ~ 0
-col1
-Text GLabel 5300 6300 0    50   Output ~ 0
-col2
-Text GLabel 7450 6500 2    50   Output ~ 0
 col10
-Text GLabel 7450 6600 2    50   Output ~ 0
+Text GLabel 5300 6100 0    50   Output ~ 0
 col9
-Text GLabel 7450 6700 2    50   Output ~ 0
+Text GLabel 5300 6000 0    50   Output ~ 0
 col8
-Text GLabel 7450 6800 2    50   Output ~ 0
+Text GLabel 5300 5300 0    50   Output ~ 0
 col7
-Text GLabel 5300 6100 0    50   Output ~ 0
+Text GLabel 7450 6100 2    50   Output ~ 0
 row0
 $Comp
@@
 	0    1    1    0
 $EndComp
-Text GLabel 7450 7100 2    50   Output ~ 0
+Text GLabel 7450 5800 2    50   Output ~ 0
 col4
-Text GLabel 7450 7000 2    50   Output ~ 0
+Text GLabel 7450 5700 2    50   Output ~ 0
 col5
 NoConn ~ 7450 5500
@@
 Wire Wire Line
 	4750 5800 4900 5800
+Text GLabel 7450 5900 2    50   Output ~ 0
+col3
+Text GLabel 7450 7100 2    50   Output ~ 0
+row3
 Text GLabel 7450 7200 2    50   Output ~ 0
-col3
-Text GLabel 8250 7300 2    50   Output ~ 0
-row3
-Text GLabel 8250 7400 2    50   Output ~ 0
 row2
 $Comp
@@
 Text GLabel 14650 1700 1    50   Input ~ 0
 col12
-Text GLabel 5100 7250 0    50   Output ~ 0
+Text GLabel 5300 7200 0    50   Output ~ 0
 enc0b
-Text GLabel 5100 7350 0    50   Output ~ 0
+Text GLabel 5300 7300 0    50   Output ~ 0
 enc0a
-Text GLabel 8250 7200 2    50   Output ~ 0
+Text GLabel 7450 7000 2    50   Output ~ 0
 col0
 Text GLabel 2800 4250 0    50   Input ~ 0
@@
 Wire Notes Line
 	2900 9550 3850 9550
+$Comp
+L Device:C_Small C4
+U 1 1 5DFC24A4
+P 2400 9150
+F 0 "C4" H 2450 9200 30  0000 L CNN
+F 1 ".1uF" H 2450 9100 30  0000 L CNN
+F 2 "Capacitor_SMD:C_0805_2012Metric_Pad1.15x1.40mm_HandSolder" H 2400 9150 50  0001 C CNN
+F 3 "" H 2400 9150 50  0001 C CNN
+	1    2400 9150
+	1    0    0    -1
+$EndComp
 Wire Wire Line
 	1800 9000 1800 9050
+$Comp
+L Device:C_Small C5
+U 1 1 5E08E610
+P 2600 9150
+F 0 "C5" H 2650 9200 30  0000 L CNN
+F 1 ".1uF" H 2650 9100 30  0000 L CNN
+F 2 "Capacitor_SMD:C_0805_2012Metric_Pad1.15x1.40mm_HandSolder" H 2600 9150 50  0001 C CNN
+F 3 "" H 2600 9150 50  0001 C CNN
+	1    2600 9150
+	1    0    0    -1
+$EndComp
 $Comp
 L Device:C_Small C3
@@
 	1    0    0    -1
 $EndComp
+Wire Wire Line
+	2600 9050 2400 9050
 Connection ~ 1800 9050
 Connection ~ 2000 9050
 Wire Wire Line
 	2000 9050 1800 9050
+Connection ~ 2200 9050
 Wire Wire Line
 	2200 9050 2000 9050
+Connection ~ 2400 9050
+Wire Wire Line
+	2400 9050 2200 9050
+Wire Wire Line
+	2600 9250 2400 9250
 Connection ~ 2000 9250
 Wire Wire Line
 	2000 9250 1800 9250
+Connection ~ 2200 9250
 Wire Wire Line
 	2200 9250 2000 9250
+Connection ~ 2400 9250
+Wire Wire Line
+	2400 9250 2200 9250
 Connection ~ 1800 9250
 Wire Wire Line
@@
 	0    1    1    0
 $EndComp
+Text GLabel 6650 9050 3    50   Input ~ 0
+col11
 Text GLabel 6750 9050 3    50   Input ~ 0
-col1
-Text GLabel 6550 9050 3    50   Input ~ 0
-row0
+col10
 $Comp
 L power:GND #PWR0101
@@
 Text GLabel 5300 5500 0    50   BiDi ~ 0
 D-
-Text GLabel 6650 9050 3    50   Input ~ 0
-col2
+Text GLabel 6550 9050 3    50   Input ~ 0
+col9
 Text GLabel 6850 9050 3    50   Input ~ 0
 ISP_Reset
 Wire Wire Line
 	14600 1100 14750 1100
-Text GLabel 7450 6000 2    50   Output ~ 0
+Text GLabel 5300 7100 0    50   Output ~ 0
 col12
 Wire Wire Line
@@
 Wire Wire Line
 	14650 3200 14650 3900
-NoConn ~ 8450 6450
-NoConn ~ 8450 6650
-NoConn ~ 8450 6750
-NoConn ~ 8450 6950
-NoConn ~ 8450 6550
-NoConn ~ 8450 6850
+NoConn ~ 7450 6500
+NoConn ~ 7450 6700
+NoConn ~ 7450 6800
+NoConn ~ 5300 7400
+NoConn ~ 7450 6600
+NoConn ~ 5300 7000
 Wire Wire Line
 	14650 1800 14650 2500
@@
 Text GLabel 12500 1700 1    50   Input ~ 0
 col10
-Text GLabel 7450 6100 2    50   Output ~ 0
+Text GLabel 5300 6300 0    50   Output ~ 0
 col11
-Text GLabel 7450 6900 2    50   Output ~ 0
+Text GLabel 7450 5600 2    50   Output ~ 0
 col6
 Text GLabel 5150 8750 2    50   Input ~ 0
@@
 Wire Notes Line
 	5800 8400 5800 9550
-Connection ~ 2200 9250
-Connection ~ 2200 9050
-Wire Wire Line
-	2400 9250 2200 9250
-Wire Wire Line
-	2400 9050 2200 9050
-$Comp
-L Device:C_Small C4
-U 1 1 5DFC24A4
-P 2400 9150
-F 0 "C4" H 2450 9200 30  0000 L CNN
-F 1 ".1uF" H 2450 9100 30  0000 L CNN
-F 2 "Capacitor_SMD:C_0805_2012Metric_Pad1.15x1.40mm_HandSolder" H 2400 9150 50  0001 C CNN
-F 3 "" H 2400 9150 50  0001 C CNN
-	1    2400 9150
-	1    0    0    -1
-$EndComp
 $EndSCHEMATC
