File: 01_lucy/pcb.sch (KiCad schematic (older format))
At the start: 127 parts, among them J1 TYPE-C-31-M12_13, J2 AVR-ISP-6_mod, K1 KEYSW, K10 KEYSW, K11 KEYSW, K12 KEYSW, K13 KEYSW, K14 KEYSW, K15 KEYSW, K16 KEYSW, K17 KEYSW, K18 KEYSW, K19 KEYSW, K2 KEYSW, K20 KEYSW, K21 KEYSW, K22 KEYSW, K23 KEYSW, K24 KEYSW, K25 KEYSW, K26 KEYSW, K27 KEYSW, K28 KEYSW, K29 KEYSW, K3 KEYSW, K30 KEYSW, K31 KEYSW, K32 KEYSW, K33 KEYSW, K34 KEYSW, K35 KEYSW, K36 KEYSW, K37 KEYSW, K38 KEYSW, K39 KEYSW, K4 KEYSW, K40 KEYSW, K41 KEYSW, K42 KEYSW, K43 KEYSW, K44 KEYSW, K45 KEYSW, K46 KEYSW, K47 KEYSW, K48 KEYSW, K49 KEYSW, K5 KEYSW, K50 KEYSW, K51 KEYSW, K52 KEYSW, K6 KEYSW, K7 KEYSW, K8 KEYSW, K9 KEYSW, SW1 SW_PUSH, SW2 Rotary_Encoder_Switch, U1 ATMEGA32U4, U2 PRTR5V0U2X, Y1 16MHz

Commit message: moved AREF pin to pin 1
Parts:
- D1, D10, D11, D12, D13, D14, D15, D16, D17, D18, D19, D2, D20, D21, D22, D23, D24, D25, D26, D27, D28, D29, D3, D30, D31, D32, D33, D34, D35, D36, D37, D38, D39, D4, D40, D41, D42, D43, D44, D45, D46, D47, D48, D49, D5, D50, D51, D52, D6, D7, D8, D9: symbol lucy-rescue:D-keyboard_parts-Ori-rescue -> pcb-rescue:D-keyboard_parts-Ori-rescue-lucy-rescue
- J1: symbol lucy-rescue:TYPE-C-31-M12_13-acheronSymbols-Ori-rescue -> pcb-rescue:TYPE-C-31-M12_13-acheronSymbols-Ori-rescue-lucy-rescue
- J2: symbol lucy-rescue:AVR-ISP-6_mod-Connector-Ori-rescue -> pcb-rescue:AVR-ISP-6_mod-Connector-Ori-rescue-lucy-rescue
- K1, K10, K11, K12, K13, K14, K15, K16, K17, K18, K19, K2, K20, K21, K22, K23, K24, K25, K26, K27, K28, K29, K3, K30, K31, K32, K33, K34, K35, K36, K37, K38, K39, K4, K40, K41, K42, K43, K44, K45, K46, K47, K48, K49, K5, K50, K51, K52, K6, K7, K8, K9: symbol lucy-rescue:KEYSW-keyboard_parts-Ori-rescue -> pcb-rescue:KEYSW-keyboard_parts-Ori-rescue-lucy-rescue
- LED1: symbol lucy-rescue:LED-keyboard_parts-Ori-rescue -> pcb-rescue:LED-keyboard_parts-Ori-rescue-lucy-rescue
- SW1: symbol lucy-rescue:SW_PUSH-keyboard_parts-Ori-rescue -> pcb-rescue:SW_PUSH-keyboard_parts-Ori-rescue-lucy-rescue
- U1: symbol lucy-rescue:ATMEGA32U4-keyboard_parts-Ori-rescue -> pcb-rescue:ATMEGA32U4-keyboard_parts-Ori-rescue-lucy-rescue
Connections:
- net row2: now also U1.1 (PE6/AIN0); no longer U1.42 (AREF)
