File: 01_pcb/pcb.kicad_pcb (KiCad board)
At the start: 2 copper layers, 250 x 77.1 mm, 127 parts, among them J1 TYPE-C-31-M12_13, J2 AVR-ISP-6_mod, K1 KEYSW, K10 KEYSW, K11 KEYSW, K12 KEYSW, K13 KEYSW, K14 KEYSW, K15 KEYSW, K16 KEYSW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

Commit message: new plates
Routing:
- net row2: track 237.6 -> 239.5 mm, vias 6 -> 4
- net Net-(D2-Pad2): track 40.3 -> 38.9 mm
- net Net-(D1-Pad2): track 54.8 -> 53.3 mm
- net row0: track 255.3 -> 256.0 mm
- net GND: vias 1 -> 0
Other:
- board text added: "github.com/ricklicious"
- board text removed: "github.com/dierickdie"
