File: 03.0_bottom_plate/bottom_plate.sch (KiCad schematic (older format))
At the start: 70 parts, among them U1 HOLE, U10 HOLE, U11 HOLE, U12 HOLE, U13 HOLE, U14 HOLE, U15 HOLE, U16 HOLE, U17 HOLE, U18 HOLE, U19 HOLE, U2 HOLE, U20 HOLE, U21 HOLE, U22 HOLE, U23 HOLE, U24 HOLE, U25 HOLE, U26 HOLE, U27 HOLE, U28 HOLE, U29 HOLE, U3 HOLE, U30 HOLE, U31 HOLE, U32 HOLE, U33 HOLE, U34 HOLE, U35 HOLE, U36 HOLE, U37 HOLE, U38 HOLE, U39 HOLE, U4 HOLE, U40 HOLE, U41 HOLE, U42 HOLE, U43 HOLE, U44 HOLE, U45 HOLE, U46 HOLE, U47 HOLE, U48 HOLE, U49 HOLE, U5 HOLE, U53 HOLE, U57 HOLE, U6 HOLE, U61 HOLE, U7 HOLE, U8 HOLE, U9 HOLE

Commit message: new plates
Parts:
- H12: footprint random-keyboard-parts:Generic-Mounthole -> MountingHole:MountingHole_2.2mm_M2
Changed lines of the file:
@@
 F 0 "H12" H 4550 3746 50  0000 L CNN
 F 1 "MountingHole" H 4550 3655 50  0000 L CNN
-F 2 "random-keyboard-parts:Generic-Mounthole" H 4450 3700 50  0001 C CNN
+F 2 "MountingHole:MountingHole_2.2mm_M2" H 4450 3700 50  0001 C CNN
 F 3 "~" H 4450 3700 50  0001 C CNN
 	1    4450 3700
