File: 03.1_bottom_plate/bottom_plate.kicad_pcb (KiCad board)
At the start: 2 copper layers, 252.4 x 84.5 mm, 62 parts, among them U1 HOLE, U10 HOLE, U11 HOLE, U12 HOLE, U13 HOLE, U14 HOLE, U15 HOLE, U16 HOLE, U17 HOLE, U18 HOLE, U19 HOLE, U2 HOLE, U20 HOLE, U21 HOLE, U22 HOLE, U23 HOLE, U24 HOLE, U25 HOLE, U26 HOLE, U27 HOLE, U28 HOLE, U29 HOLE, U3 HOLE, U30 HOLE, U31 HOLE, U32 HOLE, U33 HOLE, U34 HOLE, U35 HOLE, U36 HOLE, U37 HOLE, U38 HOLE, U39 HOLE, U4 HOLE, U40 HOLE, U41 HOLE, U42 HOLE, U43 HOLE, U44 HOLE, U45 HOLE, U46 HOLE, U47 HOLE, U48 HOLE, U49 HOLE, U5 HOLE, U53 HOLE, U57 HOLE, U6 HOLE, U61 HOLE, U7 HOLE, U8 HOLE, U9 HOLE

Commit message: update bottom plate
Parts:
- moved H4 8.93 mm to (234.6, 118.5)
- moved H5 8.93 mm to (310.8, 38.7)
- moved H6 8.93 mm to (310.8, 118.5)
- moved H3 8.33 mm to (234.6, 38.7)
- moved H1 5.36 mm to (156.0, 38.7)
- moved H2 5.36 mm to (156.0, 118.5)
- moved H7 5.36 mm to (389.4, 38.7)
- moved H8 5.36 mm to (389.4, 118.5)
Other:
- board size 252.4 x 84.5 mm -> 252.4 x 85.7 mm

Commit message: update plates
Parts:
- moved H12 19.0 mm to (184.6, 50.0)
- moved H4 8.93 mm to (225.6, 118.5)
- moved H5 8.93 mm to (319.7, 38.7)
- moved H6 8.93 mm to (319.7, 118.5)
- moved H3 8.33 mm to (226.2, 38.7)
- moved H1 5.36 mm to (161.4, 38.7)
- moved H2 5.36 mm to (161.4, 118.5)
- moved H7 5.36 mm to (384.0, 38.7)
- moved H8 5.36 mm to (384.0, 118.5)
Other:
- board size 252.4 x 85.7 mm -> 252.4 x 84.5 mm

Commit message: new plates
Other:
- board text added: "github.com/ricklicious"
- board text removed: "github.com/dierickdie"
Changed lines of the file:
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@@
     (effects (font (size 1 1) (thickness 0.15)))
   )
-  (gr_text github.com/dierickdie (at 198.702248 113.136076) (layer F.SilkS)
+  (gr_text github.com/ricklicious (at 198.702248 113.136076) (layer F.SilkS)
     (effects (font (size 1.25 1.25) (thickness 0.2)))
   )

Commit message: added HS pcb, new plate design
Parts:
- moved H2 1.19 mm to (161.4, 119.6)
- moved H4 1.19 mm to (225.6, 119.6)
- moved H6 1.19 mm to (319.7, 119.6)
- moved H8 1.19 mm to (384.0, 119.6)
- moved H1 1.19 mm to (161.4, 37.5)
- moved H3 1.19 mm to (226.2, 37.5)
- moved H5 1.19 mm to (319.7, 37.5)
- moved H7 1.19 mm to (384.0, 37.5)
Other:
- board size 252.4 x 84.5 mm -> 252.4 x 86.9 mm
- net class Default removed
- net class Thick removed
