File: 03.2_bottom_plate/bottom_plate.kicad_pcb (KiCad board)
At the start: 2 copper layers, 252.4 x 85.7 mm, 62 parts, among them U1 HOLE, U10 HOLE, U11 HOLE, U12 HOLE, U13 HOLE, U14 HOLE, U15 HOLE, U16 HOLE, U17 HOLE, U18 HOLE, U19 HOLE, U2 HOLE, U20 HOLE, U21 HOLE, U22 HOLE, U23 HOLE, U24 HOLE, U25 HOLE, U26 HOLE, U27 HOLE, U28 HOLE, U29 HOLE, U3 HOLE, U30 HOLE, U31 HOLE, U32 HOLE, U33 HOLE, U34 HOLE, U35 HOLE, U36 HOLE, U37 HOLE, U38 HOLE, U39 HOLE, U4 HOLE, U40 HOLE, U41 HOLE, U42 HOLE, U43 HOLE, U44 HOLE, U45 HOLE, U46 HOLE, U47 HOLE, U48 HOLE, U49 HOLE, U5 HOLE, U53 HOLE, U57 HOLE, U6 HOLE, U61 HOLE, U7 HOLE, U8 HOLE, U9 HOLE

Commit message: added HS pcb, new plate design
Parts:
- moved H1 1.19 mm to (156.0, 37.5)
- moved H3 1.19 mm to (234.6, 37.5)
- moved H7 1.19 mm to (389.4, 37.5)
- moved H2 1.19 mm to (156.0, 119.6)
- moved H4 1.19 mm to (234.6, 119.6)
- moved H6 1.19 mm to (310.8, 119.6)
- moved H8 1.19 mm to (389.4, 119.6)
- moved H5 1.19 mm to (310.8, 37.5)
Other:
- board size 252.4 x 85.7 mm -> 252.4 x 86.9 mm
- net class Default removed
- net class Thick removed
