File: 02.0.1_top_plate/top_plate.kicad_pcb (KiCad board)
At the start: 2 copper layers, 252.4 x 86.9 mm, 53 parts, among them U1 HOLE, U10 HOLE, U11 HOLE, U12 HOLE, U13 HOLE, U14 HOLE, U15 HOLE, U16 HOLE, U17 HOLE, U18 HOLE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

Commit message: updated top plate
Other:
- outline, holes or cut-outs redrawn
