File: 01_pcb/hotswap/pcb.kicad_pcb (KiCad board)
At the start: 2 copper layers, 251.2 x 77.7 mm, 126 parts, among them J1 TYPE-C-31-M12_13, J2 AVR-ISP-6_mod, K1 KEYSW, K10 KEYSW, K12 KEYSW, K13 KEYSW, K14 KEYSW, K15 KEYSW, K16 KEYSW, K17 KEYSW, K18 KEYSW, K19 KEYSW, K2 KEYSW, K20 KEYSW, K21 KEYSW, K23 KEYSW, K24 KEYSW, K25 KEYSW, K26 KEYSW, K27 KEYSW, K28 KEYSW, K29 KEYSW, K3 KEYSW, K30 KEYSW, K31 KEYSW, K32 KEYSW, K33 KEYSW, K34 KEYSW, K36 KEYSW, K37 KEYSW, K38 KEYSW, K39 KEYSW, K4 KEYSW, K42 KEYSW, K43 KEYSW, K44 KEYSW, K45 KEYSW, K46 KEYSW, K47 KEYSW, K48 KEYSW, K5 KEYSW, K50 KEYSW, K51 KEYSW, K52 KEYSW, K6 KEYSW, K7 KEYSW, K8 KEYSW, K9 KEYSW, SW1 SW_PUSH, SW2 Rotary_Encoder_Switch, U1 ATMEGA32U4, U2 PRTR5V0U2X, Y1 16MHz

Commit message: added HS pcb, new plate design
Parts:
- added J3: Conn_01x01, TestPoint:TestPoint_Keystone_5000-5004_Miniature, B.Cu at (133.4, 77.5)
- added J4: Conn_01x01, TestPoint:TestPoint_Keystone_5000-5004_Miniature, B.Cu at (133.4, 75.0)
- added J5: Conn_01x01, TestPoint:TestPoint_Keystone_5000-5004_Miniature, B.Cu at (133.4, 72.4)
- added J6: Conn_01x01, TestPoint:TestPoint_Keystone_5000-5004_Miniature, B.Cu at (133.4, 69.9)
- added J7: Conn_01x01, TestPoint:TestPoint_Keystone_5000-5004_Miniature, B.Cu at (133.4, 67.3)
- C1, C2, C3, C5, C6, CX1, CX2: footprint Capacitor_SMD:C_0805_2012Metric_Pad1.15x1.40mm_HandSolder -> Capacitor_SMD:C_0805_2012Metric_Pad1.18x1.45mm_HandSolder
- J2: footprint Keeb_footprints:PIN_HEADER_1x6_OFFSET -> Keeb_footprints:ICSP-Header_small_pins
- moved J2 5.71 mm to (191.7, 52.9)
Connections:
- U1 pad 18: unconnected-(U1-Pad18) -> Net-(J3-Pad1)
- U1 pad 19: unconnected-(U1-Pad19) -> Net-(J4-Pad1)
- U1 pad 20: unconnected-(U1-Pad20) -> Net-(J5-Pad1)
- U1 pad 21: unconnected-(U1-Pad21) -> Net-(J6-Pad1)
- U1 pad 22: unconnected-(U1-Pad22) -> Net-(J7-Pad1)
Routing:
- net Net-(J6-Pad1): track 0.00 -> 22.9 mm, vias 0 -> 1
- net Net-(J4-Pad1): track 0.00 -> 22.2 mm, vias 0 -> 1
- net Net-(J3-Pad1): track 0.00 -> 22.1 mm, vias 0 -> 1
- net Net-(J5-Pad1): track 0.00 -> 22.0 mm, vias 0 -> 1
- net Net-(J7-Pad1): track 0.00 -> 20.3 mm, vias 0 -> 1
- net ISP_Reset: track 124.5 -> 130.8 mm
- net row1: track 275.3 -> 277.2 mm
- net col1: track 194.7 -> 196.3 mm
- net col2: track 205.9 -> 206.8 mm
- net VCC: track 215.9 -> 216.8 mm
- net row0: track 229.2 -> 229.9 mm
- net GND: track 32.4 -> 32.2 mm, vias 4 -> 5
Other:
- board text added: "lucy_hs rev 1.0"
- board text added: "lucy_hs rev. 1.0 2022.01.02"
- board text removed: "lucy rev 1.3"
- board text removed: "lucy_hs rev. 1.0 2021.12.31"

Commit message: update pcb
Parts:
- moved SW1 15.4 mm to (102.0, 60.7), turned to 90 degrees
- moved LED1 4.10 mm to (87.8, 61.5), turned to 90 degrees
- moved U2 3.71 mm to (96.5, 47.5)
- moved J1 3.55 mm to (96.4, 44.8)
- moved RCC2 3.22 mm to (105.4, 44.9), turned to 180 degrees
- moved RCC1 3.18 mm to (87.5, 44.9), turned to 0 degrees
- moved R4 2.28 mm to (90.1, 61.5), turned to -90 degrees
- moved F1 2.01 mm to (92.4, 61.5), turned to 90 degrees
- moved D13 0.84 mm to (90.8, 77.3)
- turned K1 to 0 degrees
- turned K2 to 0 degrees
Routing:
- net Net-(D2-Pad2): track 42.0 -> 31.1 mm, vias 2 -> 0
- net Net-(D1-Pad2): track 60.0 -> 49.2 mm
- net ISP_Reset: track 130.8 -> 120.2 mm, vias 3 -> 2
- net col0: track 95.5 -> 86.9 mm
- net Net-(LED1-Pad2): track 8.72 -> 2.30 mm
- net DBUS-: track 17.9 -> 21.5 mm
- net DBUS+: track 17.2 -> 20.8 mm
- net col1: track 196.3 -> 199.5 mm
- net row1: track 277.2 -> 278.7 mm
- net Net-(D14-Pad2): track 28.9 -> 30.4 mm
- net GND: track 32.2 -> 33.2 mm, vias 5 -> 6
- net VBUS: track 27.0 -> 26.0 mm
- net row0: track 229.9 -> 230.8 mm
- net Net-(D13-Pad2): track 12.8 -> 13.7 mm
- net col12: vias 4 -> 3
Other:
- board size 251.2 x 77.7 mm -> 252.4 x 81.9 mm

Commit message: add mounting support for encoder
Parts:
- added H1: MountingHole, MountingHole:MountingHole_2.2mm_M2_DIN965_Pad, F.Cu at (308.3, 53.2)
- moved RSW1 78.7 mm to (186.6, 61.0), turned to 90 degrees
- moved SW1 78.6 mm to (180.6, 60.9), turned to 180 degrees
- moved RCC1 16.9 mm to (84.8, 61.6), turned to 90 degrees
- moved RCC2 16.9 mm to (102.3, 61.5), turned to 90 degrees
- moved D49 8.10 mm to (304.0, 58.0), turned to -90 degrees
- moved D50 0.41 mm to (311.8, 62.7)
Routing:
- net col12: track 342.2 -> 317.4 mm, vias 3 -> 4
- net Net-(J1-PadA5): track 8.90 -> 24.5 mm
- net Net-(D49-Pad2): track 14.8 -> 29.9 mm
- net Net-(J1-PadB5): track 8.40 -> 20.0 mm
- net VCC: track 216.7 -> 209.1 mm
- net row0: track 230.8 -> 223.4 mm
- net GND: track 33.2 -> 39.1 mm, vias 6 -> 5
- net ISP_Reset: track 120.2 -> 124.3 mm
- net row1: track 278.7 -> 280.5 mm
- net D+: track 31.0 -> 31.7 mm
Other:
- board size 252.4 x 81.9 mm -> 251.2 x 81.3 mm
- board text removed: "github.com/ricklicious"
