File: 01_pcb/hotswap_v2_flex/pcb.kicad_pcb (KiCad board)
At the start: 2 copper layers, 251.2 x 81.3 mm, 131 parts, among them J1 TYPE-C-31-M12_13, J2 AVR-ISP-6_mod, J3 Conn_01x01, J4 Conn_01x01, J5 Conn_01x01, J6 Conn_01x01, J7 Conn_01x01, K1 KEYSW, K10 KEYSW, K12 KEYSW, K13 KEYSW, K14 KEYSW, K15 KEYSW, K16 KEYSW, K17 KEYSW, K18 KEYSW, K19 KEYSW, K2 KEYSW, K20 KEYSW, K21 KEYSW, K23 KEYSW, K24 KEYSW, K25 KEYSW, K26 KEYSW, K27 KEYSW, K28 KEYSW, K29 KEYSW, K3 KEYSW, K30 KEYSW, K31 KEYSW, K32 KEYSW, K33 KEYSW, K34 KEYSW, K36 KEYSW, K37 KEYSW, K38 KEYSW, K39 KEYSW, K4 KEYSW, K42 KEYSW, K43 KEYSW, K44 KEYSW, K45 KEYSW, K46 KEYSW, K47 KEYSW, K48 KEYSW, K5 KEYSW, K50 KEYSW, K51 KEYSW, K52 KEYSW, K6 KEYSW, K7 KEYSW, K8 KEYSW, K9 KEYSW, SW1 SW_PUSH, SW2 Rotary_Encoder_Switch, U1 ATMEGA32U4, U2 PRTR5V0U2X, Y1 16MHz

Commit message: finished routing
Parts:
- moved D14 19.5 mm to (113.5, 74.4), turned to 90 degrees
- moved D23 11.6 mm to (284.9, 74.4), turned to 90 degrees
- moved D24 11.6 mm to (288.0, 74.4), turned to 90 degrees
- moved D19 11.5 mm to (208.9, 74.4), turned to 90 degrees
- moved D20 11.5 mm to (212.0, 74.4), turned to 90 degrees
- moved D17 11.5 mm to (170.5, 74.4), turned to 90 degrees
- moved D18 11.5 mm to (173.6, 74.4), turned to 90 degrees
- moved D15 11.5 mm to (132.4, 74.4), turned to 90 degrees
- moved D16 11.5 mm to (135.6, 74.4), turned to 90 degrees
- moved D21 11.5 mm to (246.8, 74.4), turned to 90 degrees
- moved D22 11.5 mm to (249.9, 74.4), turned to 90 degrees
- moved J2 5.43 mm to (191.7, 47.4)
- moved RSW1 1.70 mm to (195.0, 58.8)
- moved SW1 0.40 mm to (200.6, 59.3)
Routing:
- net col6: track 616.5 -> 798.1 mm
- net col5: track 561.4 -> 720.2 mm
- net col7: track 525.6 -> 681.4 mm
- net col4: track 506.1 -> 627.7 mm
- net col8: track 433.1 -> 551.3 mm
- net col3: track 449.1 -> 532.7 mm
- net col9: track 340.6 -> 421.1 mm
- net row1: track 356.7 -> 428.2 mm
- net col2: track 455.8 -> 497.4 mm
- net col10: track 249.4 -> 263.4 mm
- net Net-(D14-Pad2): track 18.5 -> 6.29 mm
- net Net-(D20-Pad2): track 15.4 -> 23.8 mm
- net Net-(D24-Pad2): track 15.4 -> 23.8 mm
- net Net-(D16-Pad2): track 15.4 -> 23.7 mm
- net Net-(D22-Pad2): track 15.4 -> 23.6 mm
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Other:
- board text added: "lucy_hs_flex rev 1.0"
- board text added: "lucy_hs_flex rev. 1.0 2022.03.21"
- board text removed: "lucy_hs rev 1.0"
- board text removed: "lucy_hs rev. 1.0 2022.03.21"

Commit message: route lines away from crystal
Parts:
- moved D13 0.80 mm to (82.1, 60.8), turned to 90 degrees
Routing:
- net row1: track 428.2 -> 418.3 mm
- net col12: track 96.6 -> 104.0 mm, vias 7 -> 5
- net ISP_Reset: track 152.2 -> 159.5 mm
- net Net-(J3-Pad1): track 21.2 -> 26.6 mm
- net VCC: track 475.2 -> 479.8 mm
- net Net-(J4-Pad1): track 23.7 -> 28.0 mm
- net Net-(J5-Pad1): track 26.2 -> 30.2 mm
- net Net-(J7-Pad1): track 31.3 -> 35.3 mm
- net Net-(J6-Pad1): track 28.8 -> 32.8 mm
- net col2: track 497.4 -> 494.2 mm
- net Net-(D13-Pad2): track 12.7 -> 15.7 mm
- net col8: track 551.3 -> 549.0 mm
- net col9: track 421.1 -> 418.8 mm
- net col7: track 681.4 -> 679.3 mm
- net col10: track 263.4 -> 261.2 mm
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
Commit message: add mounting support for encoder
Parts:
- added H1: MountingHole, MountingHole:MountingHole_2.2mm_M2_DIN965_Pad, F.Cu at (308.3, 53.2)
- moved D50 4.75 mm to (313.6, 58.6), turned to 90 degrees
- moved D49 3.93 mm to (310.9, 58.6)
Routing:
- net Net-(D50-Pad2): track 15.8 -> 22.1 mm
- net Net-(D49-Pad2): track 14.8 -> 18.9 mm
- net col12: track 104.0 -> 107.4 mm, vias 5 -> 4
- net row1: track 418.3 -> 420.0 mm
- net row0: track 231.8 -> 232.9 mm
