File: 01_pcb/hotswap_v2_flex/pcb.kicad_sch (KiCad schematic)
At the start: 131 parts, among them J1 TYPE-C-31-M12_13, J2 AVR-ISP-6_mod, J3 Conn_01x01, J4 Conn_01x01, J5 Conn_01x01, J6 Conn_01x01, J7 Conn_01x01, K1 KEYSW, K10 KEYSW, K11 KEYSW, K12 KEYSW, K13 KEYSW, K14 KEYSW, K15 KEYSW, K16 KEYSW, K17 KEYSW, K18 KEYSW, K19 KEYSW, K2 KEYSW, K20 KEYSW, K21 KEYSW, K22 KEYSW, K23 KEYSW, K24 KEYSW, K25 KEYSW, K26 KEYSW, K27 KEYSW, K28 KEYSW, K29 KEYSW, K3 KEYSW, K30 KEYSW, K31 KEYSW, K32 KEYSW, K33 KEYSW, K34 KEYSW, K35 KEYSW, K36 KEYSW, K37 KEYSW, K38 KEYSW, K39 KEYSW, K4 KEYSW, K40 KEYSW, K41 KEYSW, K42 KEYSW, K43 KEYSW, K44 KEYSW, K45 KEYSW, K46 KEYSW, K47 KEYSW, K48 KEYSW, K5 KEYSW, K50 KEYSW, K51 KEYSW, K52 KEYSW, K6 KEYSW, K7 KEYSW, K8 KEYSW, K9 KEYSW, SW1 SW_PUSH, SW2 Rotary_Encoder_Switch, U1 ATMEGA32U4, U2 PRTR5V0U2X, Y1 16MHz

Commit message: add mounting support for encoder
Parts:
- added H1: MountingHole, MountingHole:MountingHole_2.2mm_M2_DIN965_Pad, symbol Mechanical:MountingHole
Changed lines of the file:
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@@
     (pin "1")
+  )
+  (symbol (lib_id "Mechanical:MountingHole") (at 213.36 217.17 0) (unit 1)
+    (in_bom yes) (on_board yes) (fields_autoplaced)
+    (property "Reference" "H1" (id 0) (at 215.9 215.8999 0)
+      (effects (font (size 1.27 1.27)) (justify left))
+    )
+    (property "Value" "MountingHole" (id 1) (at 215.9 218.4399 0)
+      (effects (font (size 1.27 1.27)) (justify left))
+    )
+    (property "Footprint" "MountingHole:MountingHole_2.2mm_M2_DIN965_Pad" (id 2) (at 213.36 217.17 0)
+      (effects (font (size 1.27 1.27)) hide)
+    )
+    (property "Datasheet" "~" (id 3) (at 213.36 217.17 0)
+      (effects (font (size 1.27 1.27)) hide)
+    )
   )
   (sheet_instances
@@
       (reference "F1") (unit 1) (value ".5A") (footprint "Fuse:Fuse_0805_2012Metric_Pad1.15x1.40mm_HandSolder")
     )
+    (path "/e4b85a39-5116-4e8e-ae5d-7a743dcd8940"
+      (reference "H1") (unit 1) (value "MountingHole") (footprint "MountingHole:MountingHole_2.2mm_M2_DIN965_Pad")
+    )
     (path "/00000000-0000-0000-0000-00005e315a49"
