File: 01_pcb/hotswap_flex/pcb.kicad_pcb (KiCad board)
At the start: 2 copper layers, 251.2 x 81.3 mm, 132 parts, among them J1 TYPE-C-31-M12_13, J2 AVR-ISP-6_mod, J3 Conn_01x01, J4 Conn_01x01, J5 Conn_01x01, J6 Conn_01x01, J7 Conn_01x01, K1 KEYSW, K10 KEYSW, K12 KEYSW, K13 KEYSW, K14 KEYSW, K15 KEYSW, K16 KEYSW, K17 KEYSW, K18 KEYSW, K19 KEYSW, K2 KEYSW, K20 KEYSW, K21 KEYSW, K23 KEYSW, K24 KEYSW, K25 KEYSW, K26 KEYSW, K27 KEYSW, K28 KEYSW, K29 KEYSW, K3 KEYSW, K30 KEYSW, K31 KEYSW, K32 KEYSW, K33 KEYSW, K34 KEYSW, K36 KEYSW, K37 KEYSW, K38 KEYSW, K39 KEYSW, K4 KEYSW, K42 KEYSW, K43 KEYSW, K44 KEYSW, K45 KEYSW, K46 KEYSW, K47 KEYSW, K48 KEYSW, K5 KEYSW, K50 KEYSW, K51 KEYSW, K52 KEYSW, K6 KEYSW, K7 KEYSW, K8 KEYSW, K9 KEYSW, SW1 SW_PUSH, SW2 Rotary_Encoder_Switch, U1 ATMEGA32U4, U2 PRTR5V0U2X, Y1 16MHz

Commit message: add flex plate files
Parts:
- moved D20 0.30 mm to (211.7, 74.4)
- moved D19 0.30 mm to (208.6, 74.4)
Routing:
- net Net-(D18-Pad2): track 23.6 -> 25.6 mm
- net Net-(D22-Pad2): track 23.6 -> 25.3 mm
- net row1: track 420.0 -> 421.4 mm
- net Net-(D20-Pad2): track 23.8 -> 25.2 mm
Other:
- board text added: "lucy_hs_flex rev. 1.0 2022.04.19"
- board text removed: "lucy_hs_flex rev. 1.0 2022.03.21"
