File: 01_pcb/2.0 hotswap_breakaway/pcb.kicad_pcb (KiCad board)
At the start: 2 copper layers, 251.2 x 81.6 mm, 137 parts, among them J1 TYPE-C-31-M12_13, J2 AVR-ISP-6_mod, K1 KEYSW, K10 KEYSW, K12 KEYSW, K13 KEYSW, K14 KEYSW, K15 KEYSW, K16 KEYSW, K17 KEYSW, K18 KEYSW, K19 KEYSW, K2 KEYSW, K20 KEYSW, K21 KEYSW, K23 KEYSW, K24 KEYSW, K25 KEYSW, K26 KEYSW, K27 KEYSW, K28 KEYSW, K29 KEYSW, K3 KEYSW, K30 KEYSW, K31 KEYSW, K32 KEYSW, K33 KEYSW, K34 KEYSW, K36 KEYSW, K37 KEYSW, K38 KEYSW, K39 KEYSW, K4 KEYSW, K42 KEYSW, K43 KEYSW, K44 KEYSW, K45 KEYSW, K46 KEYSW, K47 KEYSW, K48 KEYSW, K49 KEYSW, K5 KEYSW, K50 KEYSW, K51 KEYSW, K52 KEYSW, K6 KEYSW, K7 KEYSW, K8 KEYSW, K9 KEYSW, SW1 SW_PUSH, SW2 Rotary_Encoder_Switch, U1 ATMEGA32U4, U2 PRTR5V0U2X, Y1 16MHz

Commit message: kicad generated backups
Parts:
- removed H10: MountingHole, MountingHole:MountingHole_2.2mm_M2_DIN965_Pad
- moved H3 38.1 mm to (305.4, 91.3)
- moved H1 35.7 mm to (305.4, 53.2)
- moved D49 4.66 mm to (308.8, 58.3)
- moved D50 4.27 mm to (308.8, 66.2)
- moved D51 2.54 mm to (309.3, 92.6)
- moved D52 2.25 mm to (309.5, 112.2)
- moved SW2 0.13 mm to (320.3, 53.1)
Routing:
- net enc0a: track 250.0 -> 273.6 mm
- net enc0b: track 255.2 -> 268.3 mm
- net col2: track 209.1 -> 220.7 mm, vias 8 -> 6
- net ISP_Reset: track 111.7 -> 117.6 mm, vias 2 -> 0
- net Net-(D49-Pad2): track 17.6 -> 22.5 mm
- net row2: track 250.9 -> 246.2 mm
- net row0: track 242.7 -> 246.5 mm, vias 2 -> 0
- net Net-(D50-Pad2): track 15.8 -> 19.4 mm
- net col12: track 316.0 -> 318.5 mm
- net row3: track 260.8 -> 258.5 mm
- net Net-(D51-Pad2): track 25.7 -> 23.5 mm
- net GND: track 17.7 -> 19.4 mm, vias 2 -> 3
- net Net-(D2-Pad2): track 30.7 -> 31.7 mm
- net col4: track 114.1 -> 113.3 mm
- net row1: track 290.7 -> 291.4 mm
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Other:
- outline, holes or cut-outs redrawn
- board text removed: "Encoder"
- board text removed: "JLCJLCJLCJLC"
