File: 01_pcb/2.0 hotswap_flex/pcb.kicad_pcb (KiCad board)
At the start: 2 copper layers, 251.2 x 81.3 mm, 138 parts, among them J1 TYPE-C-31-M12_13, J2 AVR-ISP-6_mod, J3 Conn_01x01, J4 Conn_01x01, J5 Conn_01x01, J6 Conn_01x01, J7 Conn_01x01, J8 4PIN, K1 KEYSW, K10 KEYSW, K12 KEYSW, K13 KEYSW, K14 KEYSW, K15 KEYSW, K16 KEYSW, K17 KEYSW, K18 KEYSW, K19 KEYSW, K2 KEYSW, K20 KEYSW, K21 KEYSW, K23 KEYSW, K24 KEYSW, K25 KEYSW, K26 KEYSW, K27 KEYSW, K28 KEYSW, K29 KEYSW, K3 KEYSW, K30 KEYSW, K31 KEYSW, K32 KEYSW, K33 KEYSW, K34 KEYSW, K36 KEYSW, K37 KEYSW, K38 KEYSW, K39 KEYSW, K4 KEYSW, K42 KEYSW, K43 KEYSW, K44 KEYSW, K45 KEYSW, K46 KEYSW, K47 KEYSW, K48 KEYSW, K49 KEYSW, K5 KEYSW, K50 KEYSW, K51 KEYSW, K52 KEYSW, K6 KEYSW, K7 KEYSW, K8 KEYSW, K9 KEYSW, SW1 SW_PUSH, SW2 Rotary_Encoder_Switch, U1 ATMEGA32U4, U2 PRTR5V0U2X, Y1 16MHz

Commit message: Update pcb.kicad_pcb
Other:
- board text added: "lucy rev 2.0"
- board text added: "lucy rev. 2.0 2022.06.11"
- board text removed: "lucy hs flex rev 1.0"
- board text removed: "lucy rev. 2.0 flex 2022.06.11"
Changed lines of the file:
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@@
     (effects (font (size 1 1) (thickness 0.15)))
   )
-  (gr_text "lucy rev. 2.0 flex 2022.06.11" (at 111.38288 116.5) (layer "F.SilkS")
+  (gr_text "lucy rev. 2.0 2022.06.11" (at 111.38288 116.5) (layer "F.SilkS")
     (effects (font (size 1.25 1.25) (thickness 0.2)))
   )
-  (gr_text "lucy hs flex rev 1.0" (at 115.48288 116.5) (layer "B.Mask")
+  (gr_text "lucy rev 2.0" (at 115.48288 116.5) (layer "B.Mask")
     (effects (font (size 1.25 1.25) (thickness 0.2)) (justify mirror))
   )
