File: 02_plate/plate_a_flex/plate.kicad_sch (KiCad schematic)
At the start: 67 parts, among them U1 HOLE, U10 HOLE, U11 HOLE, U12 HOLE, U13 HOLE, U14 HOLE, U15 HOLE, U16 HOLE, U17 HOLE, U18 HOLE, U19 HOLE, U2 HOLE, U20 HOLE, U21 HOLE, U22 HOLE, U23 HOLE, U24 HOLE, U25 HOLE, U26 HOLE, U27 HOLE, U28 HOLE, U29 HOLE, U3 HOLE, U30 HOLE, U31 HOLE, U32 HOLE, U33 HOLE, U34 HOLE, U35 HOLE, U36 HOLE, U37 HOLE, U38 HOLE, U39 HOLE, U4 HOLE, U40 HOLE, U41 HOLE, U42 HOLE, U43 HOLE, U44 HOLE, U45 HOLE, U46 HOLE, U47 HOLE, U48 HOLE, U49 HOLE, U5 HOLE, U50 HOLE, U51 HOLE, U52 HOLE, U6 HOLE, U7 HOLE, U8 HOLE, U9 HOLE

Commit message: Sent to manu!
Parts:
- removed H10: MountingHole, random-keyboard-parts:Generic-Mounthole, symbol Mechanical:MountingHole
- H1, H11, H12, H13, H14, H2, H3, H4, H5, H6, H7, H8, H9: footprint random-keyboard-parts:Generic-Mounthole -> MountingHole:MountingHole_2.2mm_M2_DIN965_Pad
Other:
- moved on the sheet: H11, H12, H13, H14

Commit message: reduced tab distance
Parts:
- H11, H12, H13, H14, H9: footprint MountingHole:MountingHole_2.2mm_M2_DIN965_Pad -> MountingHole:MountingHole_2.2mm_M2
Changed lines of the file:
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@@
       (effects (font (size 1.27 1.27)) (justify left))
     )
-    (property "Footprint" "MountingHole:MountingHole_2.2mm_M2_DIN965_Pad" (id 2) (at 107.95 106.68 0)
+    (property "Footprint" "MountingHole:MountingHole_2.2mm_M2" (id 2) (at 107.95 106.68 0)
       (effects (font (size 1.27 1.27)) hide)
     )
@@
       (effects (font (size 1.27 1.27)) (justify left))
     )
-    (property "Footprint" "MountingHole:MountingHole_2.2mm_M2_DIN965_Pad" (id 2) (at 107.95 91.44 0)
+    (property "Footprint" "MountingHole:MountingHole_2.2mm_M2" (id 2) (at 107.95 91.44 0)
       (effects (font (size 1.27 1.27)) hide)
     )
@@
       (effects (font (size 1.27 1.27)) (justify left))
     )
-    (property "Footprint" "MountingHole:MountingHole_2.2mm_M2_DIN965_Pad" (id 2) (at 107.95 101.6 0)
+    (property "Footprint" "MountingHole:MountingHole_2.2mm_M2" (id 2) (at 107.95 101.6 0)
       (effects (font (size 1.27 1.27)) hide)
     )
@@
       (effects (font (size 1.27 1.27)) (justify left))
     )
-    (property "Footprint" "MountingHole:MountingHole_2.2mm_M2_DIN965_Pad" (id 2) (at 107.95 96.52 0)
+    (property "Footprint" "MountingHole:MountingHole_2.2mm_M2" (id 2) (at 107.95 96.52 0)
       (effects (font (size 1.27 1.27)) hide)
     )
@@
       (effects (font (size 1.27 1.27)) (justify left))
     )
-    (property "Footprint" "MountingHole:MountingHole_2.2mm_M2_DIN965_Pad" (id 2) (at 107.95 86.36 0)
+    (property "Footprint" "MountingHole:MountingHole_2.2mm_M2" (id 2) (at 107.95 86.36 0)
       (effects (font (size 1.27 1.27)) hide)
     )
@@
     )
     (path "/bcc40fb8-020a-4739-8e85-82c40b31a03a"
-      (reference "H9") (unit 1) (value "MountingHole") (footprint "MountingHole:MountingHole_2.2mm_M2_DIN965_Pad")
+      (reference "H9") (unit 1) (value "MountingHole") (footprint "MountingHole:MountingHole_2.2mm_M2")
     )
     (path "/138821c2-9a12-4c43-8043-49b56ea76806"
-      (reference "H11") (unit 1) (value "MountingHole") (footprint "MountingHole:MountingHole_2.2mm_M2_DIN965_Pad")
+      (reference "H11") (unit 1) (value "MountingHole") (footprint "MountingHole:MountingHole_2.2mm_M2")
     )
     (path "/aa07ccab-65da-4072-99a9-9fbd288c7e56"
-      (reference "H12") (unit 1) (value "MountingHole") (footprint "MountingHole:MountingHole_2.2mm_M2_DIN965_Pad")
+      (reference "H12") (unit 1) (value "MountingHole") (footprint "MountingHole:MountingHole_2.2mm_M2")
     )
     (path "/8144b458-a787-4588-b939-a2fa677a6fca"
-      (reference "H13") (unit 1) (value "MountingHole") (footprint "MountingHole:MountingHole_2.2mm_M2_DIN965_Pad")
+      (reference "H13") (unit 1) (value "MountingHole") (footprint "MountingHole:MountingHole_2.2mm_M2")
     )
     (path "/02bced4b-02ed-4aec-b0ba-10310e4c8990"
-      (reference "H14") (unit 1) (value "MountingHole") (footprint "MountingHole:MountingHole_2.2mm_M2_DIN965_Pad")
+      (reference "H14") (unit 1) (value "MountingHole") (footprint "MountingHole:MountingHole_2.2mm_M2")
     )
     (path "/00000000-0000-0000-0000-00006175f9b8"

Commit message: remove plating around switches
Parts:
- U1, U10, U11, U12, U13, U14, U15, U16, U17, U18, U19, U2, U20, U21, U22, U23, U24, U25, U26, U27, U28, U29, U3, U30, U31, U32, U33, U34, U35, U36, U37, U38, U39, U4, U40, U41, U42, U43, U44, U45, U46, U47, U48, U5, U50, U51, U52, U6, U7, U8, U9: footprint Keeb_footprints:MX100_cutout_plated -> Keeb_footprints:MX100_cutout

Commit message: update Plate A to include support for right macro
Parts:
- removed H1, H2, H3, H4, H5, H6, H7, H8: MountingHole, MountingHole:MountingHole_2.2mm_M2_DIN965_Pad, symbol Mechanical:MountingHole
- added H10: MountingHole, MountingHole:MountingHole_2.2mm_M2, symbol Mechanical:MountingHole
- U49: footprint Keeb_footprints:EC11_cutout_plated -> Keeb_footprints:EC11_cutout
- U52: footprint Keeb_footprints:MX100_cutout -> Keeb_footprints:EC11_cutout
Other:
- note removed: "Top mount holes"
Changed lines of the file:
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@@
   (paper "A4")
   (no_connect (at 171.45 97.79))
-  (polyline (pts (xy 102.87 110.49) (xy 59.69 110.49))
-    (stroke (width 0) (type default) (color 0 0 0 0))
-  )
-  (polyline (pts (xy 102.87 82.55) (xy 102.87 110.49))
-    (stroke (width 0) (type default) (color 0 0 0 0))
-  )
-  (polyline (pts (xy 59.69 110.49) (xy 59.69 82.55))
-    (stroke (width 0) (type default) (color 0 0 0 0))
-  )
-  (polyline (pts (xy 59.69 82.55) (xy 102.87 82.55))
-    (stroke (width 0) (type default) (color 0 0 0 0))
-  )
-  (text "Top mount holes" (at 72.39 107.95 0)
-    (effects (font (size 1.27 1.27)) (justify left bottom))
-  )
   (symbol (lib_id "lets_split-cache:HOLE") (at 67.31 39.37 0) (unit 1)
     (in_bom yes) (on_board yes)
@@
       (effects (font (size 1.524 1.524)) (justify left))
     )
-    (property "Footprint" "Keeb_footprints:EC11_cutout_plated" (id 2) (at 161.29 39.37 0)
+    (property "Footprint" "Keeb_footprints:EC11_cutout" (id 2) (at 161.29 39.37 0)
       (effects (font (size 1.524 1.524)) hide)
     )
@@
       (effects (font (size 1.524 1.524)) (justify left))
     )
-    (property "Footprint" "Keeb_footprints:MX100_cutout" (id 2) (at 161.29 62.23 0)
+    (property "Footprint" "Keeb_footprints:EC11_cutout" (id 2) (at 161.29 62.23 0)
       (effects (font (size 1.524 1.524)) hide)
     )
@@
     )
     (pin "1")
-  )
-  (symbol (lib_id "Mechanical:MountingHole") (at 85.09 96.52 0) (unit 1)
-    (in_bom yes) (on_board yes)
-    (property "Reference" "H7" (id 0) (at 87.63 95.3516 0)
-      (effects (font (size 1.27 1.27)) (justify left))
-    )
-    (property "Value" "MountingHole" (id 1) (at 87.63 97.663 0)
-      (effects (font (size 1.27 1.27)) (justify left))
-    )
-    (property "Footprint" "MountingHole:MountingHole_2.2mm_M2_DIN965_Pad" (id 2) (at 85.09 96.52 0)
-      (effects (font (size 1.27 1.27)) hide)
-    )
-    (property "Datasheet" "~" (id 3) (at 85.09 96.52 0)
-      (effects (font (size 1.27 1.27)) hide)
-    )
-  )
-  (symbol (lib_id "Mechanical:MountingHole") (at 85.09 101.6 0) (unit 1)
-    (in_bom yes) (on_board yes)
-    (property "Reference" "H8" (id 0) (at 87.63 100.4316 0)
-      (effects (font (size 1.27 1.27)) (justify left))
-    )
-    (property "Value" "MountingHole" (id 1) (at 87.63 102.743 0)
-      (effects (font (size 1.27 1.27)) (justify left))
-    )
-    (property "Footprint" "MountingHole:MountingHole_2.2mm_M2_DIN965_Pad" (id 2) (at 85.09 101.6 0)
-      (effects (font (size 1.27 1.27)) hide)
-    )
-    (property "Datasheet" "~" (id 3) (at 85.09 101.6 0)
-      (effects (font (size 1.27 1.27)) hide)
-    )
-  )
-  (symbol (lib_id "Mechanical:MountingHole") (at 63.5 86.36 0) (unit 1)
-    (in_bom yes) (on_board yes)
-    (property "Reference" "H1" (id 0) (at 66.04 85.1916 0)
-      (effects (font (size 1.27 1.27)) (justify left))
-    )
-    (property "Value" "MountingHole" (id 1) (at 66.04 87.503 0)
-      (effects (font (size 1.27 1.27)) (justify left))
-    )
-    (property "Footprint" "MountingHole:MountingHole_2.2mm_M2_DIN965_Pad" (id 2) (at 63.5 86.36 0)
-      (effects (font (size 1.27 1.27)) hide)
-    )
-    (property "Datasheet" "~" (id 3) (at 63.5 86.36 0)
-      (effects (font (size 1.27 1.27)) hide)
-    )
-  )
-  (symbol (lib_id "Mechanical:MountingHole") (at 63.5 91.44 0) (unit 1)
-    (in_bom yes) (on_board yes)
-    (property "Reference" "H2" (id 0) (at 66.04 90.2716 0)
-      (effects (font (size 1.27 1.27)) (justify left))
-    )
-    (property "Value" "MountingHole" (id 1) (at 66.04 92.583 0)
-      (effects (font (size 1.27 1.27)) (justify left))
-    )
-    (property "Footprint" "MountingHole:MountingHole_2.2mm_M2_DIN965_Pad" (id 2) (at 63.5 91.44 0)
-      (effects (font (size 1.27 1.27)) hide)
-    )
-    (property "Datasheet" "~" (id 3) (at 63.5 91.44 0)
-      (effects (font (size 1.27 1.27)) hide)
-    )
-  )
-  (symbol (lib_id "Mechanical:MountingHole") (at 63.5 96.52 0) (unit 1)
-    (in_bom yes) (on_board yes)
-    (property "Reference" "H3" (id 0) (at 66.04 95.3516 0)
-      (effects (font (size 1.27 1.27)) (justify left))
-    )
-    (property "Value" "MountingHole" (id 1) (at 66.04 97.663 0)
-      (effects (font (size 1.27 1.27)) (justify left))
-    )
-    (property "Footprint" "MountingHole:MountingHole_2.2mm_M2_DIN965_Pad" (id 2) (at 63.5 96.52 0)
-      (effects (font (size 1.27 1.27)) hide)
-    )
-    (property "Datasheet" "~" (id 3) (at 63.5 96.52 0)
-      (effects (font (size 1.27 1.27)) hide)
-    )
-  )
-  (symbol (lib_id "Mechanical:MountingHole") (at 63.5 101.6 0) (unit 1)
-    (in_bom yes) (on_board yes)
-    (property "Reference" "H4" (id 0) (at 66.04 100.4316 0)
-      (effects (font (size 1.27 1.27)) (justify left))
-    )
-    (property "Value" "MountingHole" (id 1) (at 66.04 102.743 0)
-      (effects (font (size 1.27 1.27)) (justify left))
-    )
-    (property "Footprint" "MountingHole:MountingHole_2.2mm_M2_DIN965_Pad" (id 2) (at 63.5 101.6 0)
-      (effects (font (size 1.27 1.27)) hide)
-    )
-    (property "Datasheet" "~" (id 3) (at 63.5 101.6 0)
-      (effects (font (size 1.27 1.27)) hide)
-    )
-  )
-  (symbol (lib_id "Mechanical:MountingHole") (at 85.09 86.36 0) (unit 1)
-    (in_bom yes) (on_board yes)
-    (property "Reference" "H5" (id 0) (at 87.63 85.1916 0)
-      (effects (font (size 1.27 1.27)) (justify left))
-    )
-    (property "Value" "MountingHole" (id 1) (at 87.63 87.503 0)
-      (effects (font (size 1.27 1.27)) (justify left))
-    )
-    (property "Footprint" "MountingHole:MountingHole_2.2mm_M2_DIN965_Pad" (id 2) (at 85.09 86.36 0)
-      (effects (font (size 1.27 1.27)) hide)
-    )
-    (property "Datasheet" "~" (id 3) (at 85.09 86.36 0)
-      (effects (font (size 1.27 1.27)) hide)
-    )
-  )
-  (symbol (lib_id "Mechanical:MountingHole") (at 85.09 91.44 0) (unit 1)
-    (in_bom yes) (on_board yes)
-    (property "Reference" "H6" (id 0) (at 87.63 90.2716 0)
-      (effects (font (size 1.27 1.27)) (justify left))
-    )
-    (property "Value" "MountingHole" (id 1) (at 87.63 92.583 0)
-      (effects (font (size 1.27 1.27)) (justify left))
-    )
-    (property "Footprint" "MountingHole:MountingHole_2.2mm_M2_DIN965_Pad" (id 2) (at 85.09 91.44 0)
-      (effects (font (size 1.27 1.27)) hide)
-    )
-    (property "Datasheet" "~" (id 3) (at 85.09 91.44 0)
-      (effects (font (size 1.27 1.27)) hide)
-    )
   )
   (symbol (lib_id "Device:R_Small") (at 173.99 97.79 270) (unit 1)
@@
     )
   )
+  (symbol (lib_id "Mechanical:MountingHole") (at 107.95 111.76 0) (unit 1)
+    (in_bom yes) (on_board yes)
+    (property "Reference" "H10" (id 0) (at 110.49 110.5916 0)
+      (effects (font (size 1.27 1.27)) (justify left))
+    )
+    (property "Value" "MountingHole" (id 1) (at 110.49 112.903 0)
+      (effects (font (size 1.27 1.27)) (justify left))
+    )
+    (property "Footprint" "MountingHole:MountingHole_2.2mm_M2" (id 2) (at 107.95 111.76 0)
+      (effects (font (size 1.27 1.27)) hide)
+    )
+    (property "Datasheet" "~" (id 3) (at 107.95 111.76 0)
+      (effects (font (size 1.27 1.27)) hide)
+    )
+  )
   (symbol (lib_id "Mechanical:MountingHole") (at 107.95 86.36 0) (unit 1)
     (in_bom yes) (on_board yes)
@@
       (reference "#PWR0101") (unit 1) (value "GND") (footprint "")
     )
-    (path "/00000000-0000-0000-0000-00006111b67c"
-      (reference "H1") (unit 1) (value "MountingHole") (footprint "MountingHole:MountingHole_2.2mm_M2_DIN965_Pad")
-    )
-    (path "/00000000-0000-0000-0000-00006111b682"
-      (reference "H2") (unit 1) (value "MountingHole") (footprint "MountingHole:MountingHole_2.2mm_M2_DIN965_Pad")
-    )
-    (path "/00000000-0000-0000-0000-00006111b688"
-      (reference "H3") (unit 1) (value "MountingHole") (footprint "MountingHole:MountingHole_2.2mm_M2_DIN965_Pad")
-    )
-    (path "/00000000-0000-0000-0000-00006111b68e"
-      (reference "H4") (unit 1) (value "MountingHole") (footprint "MountingHole:MountingHole_2.2mm_M2_DIN965_Pad")
-    )
-    (path "/00000000-0000-0000-0000-00006111b694"
-      (reference "H5") (unit 1) (value "MountingHole") (footprint "MountingHole:MountingHole_2.2mm_M2_DIN965_Pad")
-    )
-    (path "/00000000-0000-0000-0000-00006111b69a"
-      (reference "H6") (unit 1) (value "MountingHole") (footprint "MountingHole:MountingHole_2.2mm_M2_DIN965_Pad")
-    )
-    (path "/00000000-0000-0000-0000-00006111adf9"
-      (reference "H7") (unit 1) (value "MountingHole") (footprint "MountingHole:MountingHole_2.2mm_M2_DIN965_Pad")
-    )
-    (path "/00000000-0000-0000-0000-00006111adff"
-      (reference "H8") (unit 1) (value "MountingHole") (footprint "MountingHole:MountingHole_2.2mm_M2_DIN965_Pad")
-    )
     (path "/bcc40fb8-020a-4739-8e85-82c40b31a03a"
       (reference "H9") (unit 1) (value "MountingHole") (footprint "MountingHole:MountingHole_2.2mm_M2")
     )
+    (path "/af063e8a-3547-4957-9f02-3570954b66b3"
+      (reference "H10") (unit 1) (value "MountingHole") (footprint "MountingHole:MountingHole_2.2mm_M2")
+    )
     (path "/138821c2-9a12-4c43-8043-49b56ea76806"
       (reference "H11") (unit 1) (value "MountingHole") (footprint "MountingHole:MountingHole_2.2mm_M2")
@@
     )
     (path "/00000000-0000-0000-0000-00005f4bc82b"
-      (reference "U49") (unit 1) (value "HOLE") (footprint "Keeb_footprints:EC11_cutout_plated")
+      (reference "U49") (unit 1) (value "HOLE") (footprint "Keeb_footprints:EC11_cutout")
     )
     (path "/00000000-0000-0000-0000-00005f4bc843"
@@
     )
     (path "/00000000-0000-0000-0000-00005f4bc873"
-      (reference "U52") (unit 1) (value "HOLE") (footprint "Keeb_footprints:MX100_cutout")
-    )
-  )
+      (reference "U52") (unit 1) (value "HOLE") (footprint "Keeb_footprints:EC11_cutout")
+    )
+  )
