File: 02_plate/plate_a_flex/plate.kicad_pcb (KiCad board)
At the start: 2 copper layers, 252.4 x 88.1 mm, 67 parts, among them U1 HOLE, U10 HOLE, U11 HOLE, U12 HOLE, U13 HOLE, U14 HOLE, U15 HOLE, U16 HOLE, U17 HOLE, U18 HOLE, U19 HOLE, U2 HOLE, U20 HOLE, U21 HOLE, U22 HOLE, U23 HOLE, U24 HOLE, U25 HOLE, U26 HOLE, U27 HOLE, U28 HOLE, U29 HOLE, U3 HOLE, U30 HOLE, U31 HOLE, U32 HOLE, U33 HOLE, U34 HOLE, U35 HOLE, U36 HOLE, U37 HOLE, U38 HOLE, U39 HOLE, U4 HOLE, U40 HOLE, U41 HOLE, U42 HOLE, U43 HOLE, U44 HOLE, U45 HOLE, U46 HOLE, U47 HOLE, U48 HOLE, U49 HOLE, U5 HOLE, U50 HOLE, U51 HOLE, U52 HOLE, U6 HOLE, U7 HOLE, U8 HOLE, U9 HOLE

Commit message: Sent to manu!
Parts:
- removed H10: MountingHole, random-keyboard-parts:Generic-Mounthole
Other:
- outline, holes or cut-outs redrawn

Commit message: reduced tab distance
Parts:
- H1, H2, H3, H4, H5, H6, H7, H8: footprint random-keyboard-parts:Generic-Mounthole -> MountingHole:MountingHole_2.2mm_M2_DIN965_Pad
- H11, H12, H13, H14, H9: footprint random-keyboard-parts:Generic-Mounthole -> MountingHole:MountingHole_2.2mm_M2
Other:
- outline, holes or cut-outs redrawn

Commit message: remove plating around switches
Parts:
- U1, U10, U11, U12, U13, U14, U15, U16, U17, U18, U19, U2, U20, U21, U22, U23, U24, U25, U26, U27, U28, U29, U3, U30, U31, U32, U33, U34, U35, U36, U37, U38, U39, U4, U40, U41, U42, U43, U44, U45, U46, U47, U48, U5, U50, U51, U52, U6, U7, U8, U9: footprint Keeb_footprints:MX100_cutout_plated -> Keeb_footprints:MX100_cutout
Other:
- board size 252.4 x 88.1 mm -> 252.4 x 88.7 mm

Commit message: update Plate A to include support for right macro
Parts:
- removed H1, H2, H3, H4, H5, H6, H7, H8: MountingHole, MountingHole:MountingHole_2.2mm_M2_DIN965_Pad
- added H10: MountingHole, MountingHole:MountingHole_2.2mm_M2, F.Cu at (377.4, 97.6)
- U49: footprint Keeb_footprints:EC11_cutout_plated -> Keeb_footprints:EC11_cutout
- U52: footprint Keeb_footprints:MX100_cutout -> Keeb_footprints:EC11_cutout
- turned U49 to 0 degrees
Other:
- board size 252.4 x 88.7 mm -> 252.4 x 88.1 mm

Commit message: renamed folder
Parts:
- moved H10 9.53 mm to (377.4, 107.2)
- moved H14 5.95 mm to (350.0, 97.6)
Other:
- outline, holes or cut-outs redrawn
- board text added: "lucy plate a"
- board text removed: "lucy plate a rev 1.0"
Changed lines of the file:
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@@
   )
   (footprint "MountingHole:MountingHole_2.2mm_M2" (layer "F.Cu")
-    (at 355.997174 97.631332)
+    (at 350.044044 97.631332)
     (descr "Mounting Hole 2.2mm, no annular, M2")
     (tags "mounting hole 2.2mm no annular m2")
@@
   )
   (footprint "MountingHole:MountingHole_2.2mm_M2" (layer "F.Cu")
-    (at 377.428442 97.631332)
+    (at 377.428442 107.15634)
     (descr "Mounting Hole 2.2mm, no annular, M2")
     (tags "mounting hole 2.2mm no annular m2")
@@
   (gr_arc (start 165.497015 122.634477) (mid 164.655115 122.285751) (end 164.306389 121.443851) (layer "Edge.Cuts") (width 0.05))
   (gr_arc (start 357.187739 117.871974) (mid 356.592556 117.2767) (end 357.187739 116.681348) (layer "Edge.Cuts") (width 0.05))
-  (gr_arc (start 378.023755 94.654767) (mid 377.428442 95.25008) (end 376.833129 94.654767) (layer "Edge.Cuts") (width 0.05))
+  (gr_arc (start 378.023755 104.179775) (mid 377.428442 104.775088) (end 376.833129 104.179775) (layer "Edge.Cuts") (width 0.05))
   (gr_line (start 357.187739 117.871974) (end 379.809693 117.871975) (layer "Edge.Cuts") (width 0.05))
   (gr_arc (start 219.670497 58.935987) (mid 220.265831 59.5313) (end 219.670497 60.126613) (layer "Edge.Cuts") (width 0.05))
@@
   (gr_arc (start 188.118908 116.681397) (mid 188.714194 117.2767) (end 188.118908 117.872023) (layer "Edge.Cuts") (width 0.05))
   (gr_line (start 188.118945 40.48162) (end 150.615417 40.481452) (layer "Edge.Cuts") (width 0.05))
-  (gr_line (start 378.023755 94.654767) (end 378.023755 52.982857) (layer "Edge.Cuts") (width 0.05))
+  (gr_line (start 378.023755 104.179775) (end 378.023755 52.982857) (layer "Edge.Cuts") (width 0.05))
   (gr_line (start 225.028313 35.718781) (end 225.028313 38.100031) (layer "Edge.Cuts") (width 0.05))
   (gr_line (start 301.823713 60.126613) (end 353.020609 60.126613) (layer "Edge.Cuts") (width 0.05))
@@
   (gr_arc (start 168.473619 79.176629) (mid 167.87825 78.5813) (end 168.473619 77.986003) (layer "Edge.Cuts") (width 0.05))
   (gr_line (start 219.670476 77.986019) (end 168.473619 77.986003) (layer "Edge.Cuts") (width 0.05))
-  (gr_line (start 301.823713 98.226677) (end 353.020609 98.226645) (layer "Edge.Cuts") (width 0.05))
+  (gr_line (start 301.823713 98.226677) (end 347.06752 98.226645) (layer "Edge.Cuts") (width 0.05))
   (gr_line (start 381.00032 121.443852) (end 381.000319 119.062601) (layer "Edge.Cuts") (width 0.05))
   (gr_line (start 201.215915 117.871862) (end 223.837687 117.871975) (layer "Edge.Cuts") (width 0.05))
@@
   (gr_line (start 381.00032 35.71878) (end 381.000318 38.100031) (layer "Edge.Cuts") (width 0.05))
   (gr_line (start 320.278395 119.062601) (end 320.278395 121.443851) (layer "Edge.Cuts") (width 0.05))
-  (gr_arc (start 353.020618 97.036019) (mid 353.61589 97.6313) (end 353.020618 98.226645) (layer "Edge.Cuts") (width 0.05))
+  (gr_arc (start 347.06752 97.036019) (mid 347.662783 97.6313) (end 347.06752 98.226645) (layer "Edge.Cuts") (width 0.05))
   (gr_line (start 295.870531 97.036051) (end 225.623658 97.036019) (layer "Edge.Cuts") (width 0.05))
   (gr_arc (start 353.020609 58.935987) (mid 353.615922 59.5313) (end 353.020609 60.126613) (layer "Edge.Cuts") (width 0.05))
-  (gr_line (start 353.020609 97.036019) (end 301.823713 97.036051) (layer "Edge.Cuts") (width 0.05))
+  (gr_line (start 347.06752 97.036019) (end 301.823713 97.036051) (layer "Edge.Cuts") (width 0.05))
   (gr_arc (start 301.823713 79.176645) (mid 301.228362 78.581316) (end 301.823713 77.986019) (layer "Edge.Cuts") (width 0.05))
-  (gr_line (start 376.833129 52.982857) (end 376.833129 94.654767) (layer "Edge.Cuts") (width 0.05))
+  (gr_line (start 376.833129 52.982857) (end 376.833129 104.179775) (layer "Edge.Cuts") (width 0.05))
   (gr_arc (start 165.497015 39.290657) (mid 164.655115 38.941931) (end 164.306389 38.100031) (layer "Edge.Cuts") (width 0.05))
   (gr_line (start 188.118945 39.290994) (end 165.497015 39.290657) (layer "Edge.Cuts") (width 0.05))
@@
     (effects (font (size 1 1) (thickness 0.15)) (justify mirror))
   )
-  (gr_text "lucy plate a rev 1.0" (at 350.639357 36.909406) (layer "B.Mask")
-    (effects (font (size 1.25 1.25) (thickness 0.2)) (justify mirror))
+  (gr_text "lucy plate a" (at 350.639357 36.909406) (layer "B.SilkS")
+    (effects (font (size 1.5 1.5) (thickness 0.15)) (justify mirror))
+  )
+  (gr_text "lucy" (at 350.044044 120.253226 180) (layer "F.Mask")
+    (effects (font (size 2 2) (thickness 0.3)))
   )
   (gr_text "lucy" (at 194.667351 36.909406) (layer "F.Mask")
