File: 01_pcb/2.0 hotswap_flex - lefty_lucy/pcb.kicad_pcb (KiCad board)
At the start: 2 copper layers, 251.2 x 81.3 mm, 138 parts, among them J1 TYPE-C-31-M12_13, J2 AVR-ISP-6_mod, J3 Conn_01x01, J4 Conn_01x01, J5 Conn_01x01, J6 Conn_01x01, J7 Conn_01x01, J8 4PIN, K1 KEYSW, K10 KEYSW, K12 KEYSW, K13 KEYSW, K14 KEYSW, K15 KEYSW, K16 KEYSW, K17 KEYSW, K18 KEYSW, K19 KEYSW, K2 KEYSW, K20 KEYSW, K21 KEYSW, K23 KEYSW, K24 KEYSW, K25 KEYSW, K26 KEYSW, K27 KEYSW, K28 KEYSW, K29 KEYSW, K3 KEYSW, K30 KEYSW, K31 KEYSW, K32 KEYSW, K33 KEYSW, K34 KEYSW, K36 KEYSW, K37 KEYSW, K38 KEYSW, K39 KEYSW, K4 KEYSW, K42 KEYSW, K43 KEYSW, K44 KEYSW, K45 KEYSW, K46 KEYSW, K47 KEYSW, K48 KEYSW, K49 KEYSW, K5 KEYSW, K50 KEYSW, K51 KEYSW, K52 KEYSW, K6 KEYSW, K7 KEYSW, K8 KEYSW, K9 KEYSW, SW1 SW_PUSH, SW2 Rotary_Encoder_Switch, U1 ATMEGA32U4, U2 PRTR5V0U2X, Y1 16MHz

Commit message: new gerbers
Parts:
- moved J6 0.07 mm to (58.0, 112.8)
- moved J7 0.07 mm to (60.6, 112.8)
Routing:
- net col8: track 395.6 -> 288.7 mm
- net col9: track 481.7 -> 411.1 mm
- net col10: track 399.7 -> 433.7 mm, vias 6 -> 7
- net row0: track 409.6 -> 406.1 mm
Other:
- board text added: "lefty lucy rev 2.0.1"
- board text removed: "lucy rev 2.0.1 lm"
