File: 02_plate/plate_a/plate.kicad_sch (KiCad schematic)
At the start: 59 parts, among them U1 HOLE, U10 HOLE, U11 HOLE, U12 HOLE, U13 HOLE, U14 HOLE, U15 HOLE, U16 HOLE, U17 HOLE, U18 HOLE, U19 HOLE, U2 HOLE, U20 HOLE, U21 HOLE, U22 HOLE, U23 HOLE, U24 HOLE, U25 HOLE, U26 HOLE, U27 HOLE, U28 HOLE, U29 HOLE, U3 HOLE, U30 HOLE, U31 HOLE, U32 HOLE, U33 HOLE, U34 HOLE, U35 HOLE, U36 HOLE, U37 HOLE, U38 HOLE, U39 HOLE, U4 HOLE, U40 HOLE, U41 HOLE, U42 HOLE, U43 HOLE, U44 HOLE, U45 HOLE, U46 HOLE, U47 HOLE, U48 HOLE, U49 HOLE, U5 HOLE, U50 HOLE, U51 HOLE, U52 HOLE, U6 HOLE, U7 HOLE, U8 HOLE, U9 HOLE

Commit message: remove flex cuts, move mounting points
Parts:
- removed H10, H11, H12, H13, H14, H9: MountingHole, MountingHole:MountingHole_2.2mm_M2, symbol Mechanical:MountingHole
- R1: footprint Resistor_SMD:R_0603_1608Metric_Pad1.05x0.95mm_HandSolder -> Resistor_SMD:R_0201_0603Metric_Pad0.64x0.40mm_HandSolder
- U48: footprint Keeb_footprints:MX100_cutout -> Keeb_footprints:MX_100_cutout
- U49, U52: footprint Keeb_footprints:EC11_cutout -> Keeb_footprints:MX_100_cutout
Connections:
- net GND: now also R1.2; no longer R1.1
Changed lines of the file:
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@@
 (kicad_sch (version 20211123) (generator eeschema)
   (paper "A4")
-  (no_connect (at 171.45 97.79))
+  (no_connect (at 148.59 88.9))
   (symbol (lib_id "lets_split-cache:HOLE") (at 67.31 39.37 0) (unit 1)
     (in_bom yes) (on_board yes)
@@
       (effects (font (size 1.524 1.524)) (justify left))
     )
-    (property "Footprint" "Keeb_footprints:MX100_cutout" (id 2) (at 151.13 62.23 0)
+    (property "Footprint" "Keeb_footprints:MX_100_cutout" (id 2) (at 151.13 62.23 0)
       (effects (font (size 1.524 1.524)) hide)
     )
@@
       (effects (font (size 1.524 1.524)) (justify left))
     )
-    (property "Footprint" "Keeb_footprints:EC11_cutout" (id 2) (at 161.29 39.37 0)
+    (property "Footprint" "Keeb_footprints:MX_100_cutout" (id 2) (at 161.29 39.37 0)
       (effects (font (size 1.524 1.524)) hide)
     )
@@
       (effects (font (size 1.524 1.524)) (justify left))
     )
-    (property "Footprint" "Keeb_footprints:EC11_cutout" (id 2) (at 161.29 62.23 0)
+    (property "Footprint" "Keeb_footprints:MX_100_cutout" (id 2) (at 161.29 62.23 0)
       (effects (font (size 1.524 1.524)) hide)
     )
@@
     )
   )
-  (symbol (lib_id "power:GND") (at 176.53 97.79 0) (unit 1)
-    (in_bom yes) (on_board yes)
-    (property "Reference" "#PWR0101" (id 0) (at 176.53 104.14 0)
+  (symbol (lib_id "component:GND") (at 153.67 90.17 0) (unit 1)
+    (in_bom yes) (on_board yes) (fields_autoplaced)
+    (property "Reference" "#PWR0101" (id 0) (at 153.67 90.17 0)
+      (effects (font (size 0.762 0.762)) hide)
+    )
+    (property "Value" "GND" (id 1) (at 153.67 91.948 0)
+      (effects (font (size 0.762 0.762)) hide)
+    )
+    (property "Footprint" "" (id 2) (at 153.67 90.17 0)
       (effects (font (size 1.27 1.27)) hide)
     )
-    (property "Value" "GND" (id 1) (at 176.657 102.1842 0))
-    (property "Footprint" "" (id 2) (at 176.53 97.79 0)
+    (property "Datasheet" "" (id 3) (at 153.67 90.17 0)
       (effects (font (size 1.27 1.27)) hide)
     )
-    (property "Datasheet" "" (id 3) (at 176.53 97.79 0)
+    (pin "1")
+  )
+  (symbol (lib_id "Device:R_Small") (at 151.13 88.9 90) (unit 1)
+    (in_bom yes) (on_board yes) (fields_autoplaced)
+    (property "Reference" "R1" (id 0) (at 151.13 82.55 90))
+    (property "Value" "R_Small" (id 1) (at 151.13 85.09 90))
+    (property "Footprint" "Resistor_SMD:R_0201_0603Metric_Pad0.64x0.40mm_HandSolder" (id 2) (at 151.13 88.9 0)
       (effects (font (size 1.27 1.27)) hide)
     )
-    (pin "1")
-  )
-  (symbol (lib_id "Device:R_Small") (at 173.99 97.79 270) (unit 1)
-    (in_bom yes) (on_board yes)
-    (property "Reference" "R1" (id 0) (at 173.99 92.8116 90))
-    (property "Value" "R_Small" (id 1) (at 173.99 95.123 90))
-    (property "Footprint" "Resistor_SMD:R_0603_1608Metric_Pad1.05x0.95mm_HandSolder" (id 2) (at 173.99 97.79 0)
-      (effects (font (size 1.27 1.27)) hide)
-    )
-    (property "Datasheet" "~" (id 3) (at 173.99 97.79 0)
+    (property "Datasheet" "~" (id 3) (at 151.13 88.9 0)
       (effects (font (size 1.27 1.27)) hide)
     )
@@
     (pin "2")
   )
-  (symbol (lib_id "Mechanical:MountingHole") (at 107.95 106.68 0) (unit 1)
-    (in_bom yes) (on_board yes)
-    (property "Reference" "H14" (id 0) (at 110.49 105.5116 0)
-      (effects (font (size 1.27 1.27)) (justify left))
-    )
-    (property "Value" "MountingHole" (id 1) (at 110.49 107.823 0)
-      (effects (font (size 1.27 1.27)) (justify left))
-    )
-    (property "Footprint" "MountingHole:MountingHole_2.2mm_M2" (id 2) (at 107.95 106.68 0)
-      (effects (font (size 1.27 1.27)) hide)
-    )
-    (property "Datasheet" "~" (id 3) (at 107.95 106.68 0)
-      (effects (font (size 1.27 1.27)) hide)
-    )
-  )
-  (symbol (lib_id "Mechanical:MountingHole") (at 107.95 91.44 0) (unit 1)
-    (in_bom yes) (on_board yes)
-    (property "Reference" "H11" (id 0) (at 110.49 90.2716 0)
-      (effects (font (size 1.27 1.27)) (justify left))
-    )
-    (property "Value" "MountingHole" (id 1) (at 110.49 92.583 0)
-      (effects (font (size 1.27 1.27)) (justify left))
-    )
-    (property "Footprint" "MountingHole:MountingHole_2.2mm_M2" (id 2) (at 107.95 91.44 0)
-      (effects (font (size 1.27 1.27)) hide)
-    )
-    (property "Datasheet" "~" (id 3) (at 107.95 91.44 0)
-      (effects (font (size 1.27 1.27)) hide)
-    )
-  )
-  (symbol (lib_id "Mechanical:MountingHole") (at 107.95 101.6 0) (unit 1)
-    (in_bom yes) (on_board yes)
-    (property "Reference" "H13" (id 0) (at 110.49 100.4316 0)
-      (effects (font (size 1.27 1.27)) (justify left))
-    )
-    (property "Value" "MountingHole" (id 1) (at 110.49 102.743 0)
-      (effects (font (size 1.27 1.27)) (justify left))
-    )
-    (property "Footprint" "MountingHole:MountingHole_2.2mm_M2" (id 2) (at 107.95 101.6 0)
-      (effects (font (size 1.27 1.27)) hide)
-    )
-    (property "Datasheet" "~" (id 3) (at 107.95 101.6 0)
-      (effects (font (size 1.27 1.27)) hide)
-    )
-  )
-  (symbol (lib_id "Mechanical:MountingHole") (at 107.95 96.52 0) (unit 1)
-    (in_bom yes) (on_board yes)
-    (property "Reference" "H12" (id 0) (at 110.49 95.3516 0)
-      (effects (font (size 1.27 1.27)) (justify left))
-    )
-    (property "Value" "MountingHole" (id 1) (at 110.49 97.663 0)
-      (effects (font (size 1.27 1.27)) (justify left))
-    )
-    (property "Footprint" "MountingHole:MountingHole_2.2mm_M2" (id 2) (at 107.95 96.52 0)
-      (effects (font (size 1.27 1.27)) hide)
-    )
-    (property "Datasheet" "~" (id 3) (at 107.95 96.52 0)
-      (effects (font (size 1.27 1.27)) hide)
-    )
-  )
-  (symbol (lib_id "Mechanical:MountingHole") (at 107.95 111.76 0) (unit 1)
-    (in_bom yes) (on_board yes)
-    (property "Reference" "H10" (id 0) (at 110.49 110.5916 0)
-      (effects (font (size 1.27 1.27)) (justify left))
-    )
-    (property "Value" "MountingHole" (id 1) (at 110.49 112.903 0)
-      (effects (font (size 1.27 1.27)) (justify left))
-    )
-    (property "Footprint" "MountingHole:MountingHole_2.2mm_M2" (id 2) (at 107.95 111.76 0)
-      (effects (font (size 1.27 1.27)) hide)
-    )
-    (property "Datasheet" "~" (id 3) (at 107.95 111.76 0)
-      (effects (font (size 1.27 1.27)) hide)
-    )
-  )
-  (symbol (lib_id "Mechanical:MountingHole") (at 107.95 86.36 0) (unit 1)
-    (in_bom yes) (on_board yes)
-    (property "Reference" "H9" (id 0) (at 110.49 85.1916 0)
-      (effects (font (size 1.27 1.27)) (justify left))
-    )
-    (property "Value" "MountingHole" (id 1) (at 110.49 87.503 0)
-      (effects (font (size 1.27 1.27)) (justify left))
-    )
-    (property "Footprint" "MountingHole:MountingHole_2.2mm_M2" (id 2) (at 107.95 86.36 0)
-      (effects (font (size 1.27 1.27)) hide)
-    )
-    (property "Datasheet" "~" (id 3) (at 107.95 86.36 0)
-      (effects (font (size 1.27 1.27)) hide)
-    )
-  )
   (sheet_instances
     (path "/" (page "1"))
   )
   (symbol_instances
-    (path "/00000000-0000-0000-0000-000060e9d8fe"
+    (path "/a08525ba-978e-412d-8dac-93a6d97d6296"
       (reference "#PWR0101") (unit 1) (value "GND") (footprint "")
     )
-    (path "/bcc40fb8-020a-4739-8e85-82c40b31a03a"
-      (reference "H9") (unit 1) (value "MountingHole") (footprint "MountingHole:MountingHole_2.2mm_M2")
-    )
-    (path "/af063e8a-3547-4957-9f02-3570954b66b3"
-      (reference "H10") (unit 1) (value "MountingHole") (footprint "MountingHole:MountingHole_2.2mm_M2")
-    )
-    (path "/138821c2-9a12-4c43-8043-49b56ea76806"
-      (reference "H11") (unit 1) (value "MountingHole") (footprint "MountingHole:MountingHole_2.2mm_M2")
-    )
-    (path "/aa07ccab-65da-4072-99a9-9fbd288c7e56"
-      (reference "H12") (unit 1) (value "MountingHole") (footprint "MountingHole:MountingHole_2.2mm_M2")
-    )
-    (path "/8144b458-a787-4588-b939-a2fa677a6fca"
-      (reference "H13") (unit 1) (value "MountingHole") (footprint "MountingHole:MountingHole_2.2mm_M2")
-    )
-    (path "/02bced4b-02ed-4aec-b0ba-10310e4c8990"
-      (reference "H14") (unit 1) (value "MountingHole") (footprint "MountingHole:MountingHole_2.2mm_M2")
-    )
-    (path "/00000000-0000-0000-0000-00006175f9b8"
-      (reference "R1") (unit 1) (value "R_Small") (footprint "Resistor_SMD:R_0603_1608Metric_Pad1.05x0.95mm_HandSolder")
+    (path "/bfb28203-c05d-457c-8485-e24c70b0fe2f"
+      (reference "R1") (unit 1) (value "R_Small") (footprint "Resistor_SMD:R_0201_0603Metric_Pad0.64x0.40mm_HandSolder")
     )
     (path "/00000000-0000-0000-0000-00005f4b4d1c"
@@
     )
     (path "/00000000-0000-0000-0000-00005f4b9509"
-      (reference "U48") (unit 1) (value "HOLE") (footprint "Keeb_footprints:MX100_cutout")
+      (reference "U48") (unit 1) (value "HOLE") (footprint "Keeb_footprints:MX_100_cutout")
     )
     (path "/00000000-0000-0000-0000-00005f4bc82b"
-      (reference "U49") (unit 1) (value "HOLE") (footprint "Keeb_footprints:EC11_cutout")
+      (reference "U49") (unit 1) (value "HOLE") (footprint "Keeb_footprints:MX_100_cutout")
     )
     (path "/00000000-0000-0000-0000-00005f4bc843"
@@
     )
     (path "/00000000-0000-0000-0000-00005f4bc873"
-      (reference "U52") (unit 1) (value "HOLE") (footprint "Keeb_footprints:EC11_cutout")
-    )
-  )
+      (reference "U52") (unit 1) (value "HOLE") (footprint "Keeb_footprints:MX_100_cutout")
+    )
+  )
