File: 02_plate/plate_b/plate.kicad_pcb (KiCad board)
At the start: 2 copper layers, 252.4 x 88.1 mm, 67 parts, among them U1 HOLE, U10 HOLE, U11 HOLE, U12 HOLE, U13 HOLE, U14 HOLE, U15 HOLE, U16 HOLE, U17 HOLE, U18 HOLE, U19 HOLE, U2 HOLE, U20 HOLE, U21 HOLE, U22 HOLE, U23 HOLE, U24 HOLE, U25 HOLE, U26 HOLE, U27 HOLE, U28 HOLE, U29 HOLE, U3 HOLE, U30 HOLE, U31 HOLE, U32 HOLE, U33 HOLE, U34 HOLE, U35 HOLE, U36 HOLE, U37 HOLE, U38 HOLE, U39 HOLE, U4 HOLE, U40 HOLE, U41 HOLE, U42 HOLE, U43 HOLE, U44 HOLE, U45 HOLE, U46 HOLE, U47 HOLE, U48 HOLE, U49 HOLE, U5 HOLE, U50 HOLE, U51 HOLE, U52 HOLE, U6 HOLE, U7 HOLE, U8 HOLE, U9 HOLE

Commit message: Sent to manu!
Parts:
- removed H10: MountingHole, random-keyboard-parts:Generic-Mounthole
Changed lines of the file:
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@@
     (fp_arc (start -6.992893 -7.025) (mid -6.7 -7.732107) (end -5.992893 -8.025) (layer "F.Mask") (width 2))
     (fp_arc (start -5.992893 7.975) (mid -6.7 7.682107) (end -6.992893 6.975) (layer "F.Mask") (width 2))
-    (fp_arc (start 6.992893 6.974999) (mid 6.7 7.682106) (end 5.992893 7.974999) (layer "F.Mask") (width 2))
-    (fp_arc (start 5.992893 -8.025) (mid 6.7 -7.732107) (end 6.992893 -7.025) (layer "F.Mask") (width 2))
+    (fp_arc (start 6.992893 6.974999) (mid 6.7 7.682104) (end 5.992893 7.974999) (layer "F.Mask") (width 2))
+    (fp_arc (start 5.992893 -8.025) (mid 6.700004 -7.732109) (end 6.992893 -7.025) (layer "F.Mask") (width 2))
     (fp_line (start 7 -6) (end 7 -8) (layer "Dwgs.User") (width 0.15))
     (fp_line (start 7 -8) (end 5 -8) (layer "Dwgs.User") (width 0.15))
@@
   )
   (footprint "random-keyboard-parts:Generic-Mounthole" (layer "F.Cu")
-    (at 377.428442 107.15634)
-    (property "Sheetfile" "plate.kicad_sch")
-    (property "Sheetname" "")
-    (attr exclude_from_pos_files)
-    (fp_text reference "H10" (at 0 2) (layer "Dwgs.User")
-      (effects (font (size 1 1) (thickness 0.15)))
-    )
-    (fp_text value "MountingHole" (at 0 -2) (layer "F.Fab")
-      (effects (font (size 1 1) (thickness 0.15)))
-    )
-    (pad "1" thru_hole circle locked (at 0 0) (size 3.5 3.5) (drill 2.2) (layers *.Cu *.Mask))
-  )
-  (footprint "random-keyboard-parts:Generic-Mounthole" (layer "F.Cu")

Commit message: reduced tab distance
Parts:
- H1, H2, H3, H4, H5, H6, H7, H8: footprint random-keyboard-parts:Generic-Mounthole -> MountingHole:MountingHole_2.2mm_M2_DIN965_Pad
- H11, H12, H13, H14, H9: footprint random-keyboard-parts:Generic-Mounthole -> MountingHole:MountingHole_2.2mm_M2

Commit message: Plate B updates
Parts:
- R1: footprint Resistor_SMD:R_0603_1608Metric_Pad1.05x0.95mm_HandSolder -> Resistor_SMD:R_0201_0603Metric_Pad0.64x0.40mm_HandSolder
- U1, U10, U11, U12, U13, U14, U15, U16, U17, U18, U19, U2, U20, U21, U22, U23, U24, U25, U26, U27, U28, U29, U3, U30, U31, U32, U33, U34, U35, U36, U37, U38, U39, U4, U40, U41, U42, U43, U44, U45, U46, U47, U48, U5, U50, U51, U52, U6, U7, U8, U9: footprint Keeb_footprints:MX100_cutout_plated -> Keeb_footprints:MX100_cutout
- U49: footprint Keeb_footprints:EC11_cutout_plated -> Keeb_footprints:EC11_cutout
- moved R1 0.60 mm to (389.3, 60.1), turned to 180 degrees
Connections:
- R1 pad 1: GND -> unconnected-(R1-Pad1)
- R1 pad 2: unconnected-(R1-Pad2) -> GND
Routing:
- added copper zone on B.Cu, net (none)
- added copper zone on F.Cu, net (none)
- removed copper zone on B.Cu, net GND
- removed copper zone on F.Cu, net GND

Commit message: renamed folder
Parts:
- added H10: MountingHole, MountingHole:MountingHole_2.2mm_M2, F.Cu at (377.4, 107.2)
- moved H14 5.95 mm to (350.0, 97.6)
Changed lines of the file:
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@@
   )
   (footprint "MountingHole:MountingHole_2.2mm_M2" (layer "F.Cu")
-    (at 355.997174 97.631332)
+    (at 350.044044 97.631332)
     (descr "Mounting Hole 2.2mm, no annular, M2")
     (tags "mounting hole 2.2mm no annular m2")
@@
     (attr exclude_from_pos_files)
     (fp_text reference "H13" (at 0 -3.2) (layer "Dwgs.User")
+      (effects (font (size 1 1) (thickness 0.15)))
+    )
+    (fp_text value "MountingHole" (at 0 3.2) (layer "F.Fab")
+      (effects (font (size 1 1) (thickness 0.15)))
+    )
+    (fp_text user "${REFERENCE}" (at 0 0) (layer "F.Fab")
+      (effects (font (size 1 1) (thickness 0.15)))
+    )
+    (fp_circle (center 0 0) (end 2.2 0) (layer "Cmts.User") (width 0.15) (fill none))
+    (fp_circle (center 0 0) (end 2.45 0) (layer "F.CrtYd") (width 0.05) (fill none))
+    (pad "" np_thru_hole circle (at 0 0) (size 2.2 2.2) (drill 2.2) (layers *.Cu *.Mask))
+  )
+  (footprint "MountingHole:MountingHole_2.2mm_M2" (layer "F.Cu")
+    (at 377.428442 107.15634)
+    (descr "Mounting Hole 2.2mm, no annular, M2")
+    (tags "mounting hole 2.2mm no annular m2")
+    (property "Sheetfile" "plate.kicad_sch")
+    (property "Sheetname" "")
+    (attr exclude_from_pos_files)
+    (fp_text reference "H10" (at 0 -3.2) (layer "Dwgs.User")
       (effects (font (size 1 1) (thickness 0.15)))
     )
@@
     (effects (font (size 1.25 1.25) (thickness 0.2)) (justify mirror))
   )
+  (gr_text "lucy" (at 353.020609 119.657913 -180) (layer "F.Mask")
+    (effects (font (size 2 2) (thickness 0.3)))
+  )
   (gr_text "lucy" (at 194.072038 37.504719) (layer "F.Mask")

Commit message: remove flex cuts, move mounting points
Parts:
- removed H1, H2, H3, H4, H5, H6, H7, H8: MountingHole, MountingHole:MountingHole_2.2mm_M2_DIN965_Pad
- removed H10, H11, H12, H13, H14, H9: MountingHole, MountingHole:MountingHole_2.2mm_M2
- U48, U52: footprint Keeb_footprints:MX100_cutout -> Keeb_footprints:MX_100_cutout
- U49: footprint Keeb_footprints:EC11_cutout -> Keeb_footprints:MX_100_cutout
Other:
- board size 252.4 x 88.1 mm -> 252.4 x 86.2 mm
- board text removed: "lucy plate b rev 1.0"
