File: 02_plate/plate_b/plate.kicad_sch (KiCad schematic)
At the start: 67 parts, among them U1 HOLE, U10 HOLE, U11 HOLE, U12 HOLE, U13 HOLE, U14 HOLE, U15 HOLE, U16 HOLE, U17 HOLE, U18 HOLE, U19 HOLE, U2 HOLE, U20 HOLE, U21 HOLE, U22 HOLE, U23 HOLE, U24 HOLE, U25 HOLE, U26 HOLE, U27 HOLE, U28 HOLE, U29 HOLE, U3 HOLE, U30 HOLE, U31 HOLE, U32 HOLE, U33 HOLE, U34 HOLE, U35 HOLE, U36 HOLE, U37 HOLE, U38 HOLE, U39 HOLE, U4 HOLE, U40 HOLE, U41 HOLE, U42 HOLE, U43 HOLE, U44 HOLE, U45 HOLE, U46 HOLE, U47 HOLE, U48 HOLE, U49 HOLE, U5 HOLE, U50 HOLE, U51 HOLE, U52 HOLE, U6 HOLE, U7 HOLE, U8 HOLE, U9 HOLE

Commit message: Sent to manu!
Parts:
- removed H10: MountingHole, random-keyboard-parts:Generic-Mounthole, symbol Mechanical:MountingHole
Other:
- note added: "Standoffs"
- note removed: "HW standoffs"
- moved on the sheet: H11, H12, H13, H14, H9
Changed lines of the file:
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@@
   (paper "A4")
   (no_connect (at 171.45 97.79))
+  (polyline (pts (xy 128.27 80.01) (xy 128.27 110.49))
+    (stroke (width 0) (type default) (color 0 0 0 0))
+  )
   (polyline (pts (xy 102.87 110.49) (xy 59.69 110.49))
     (stroke (width 0) (type default) (color 0 0 0 0))
   )
-  (polyline (pts (xy 107.95 82.55) (xy 107.95 119.38))
+  (polyline (pts (xy 106.68 110.49) (xy 106.68 80.01))
     (stroke (width 0) (type default) (color 0 0 0 0))
   )
-  (polyline (pts (xy 129.54 82.55) (xy 129.54 119.38))
-    (stroke (width 0) (type default) (color 0 0 0 0))
-  )
-  (polyline (pts (xy 107.95 82.55) (xy 129.54 82.55))
+  (polyline (pts (xy 106.68 80.01) (xy 128.27 80.01))
     (stroke (width 0) (type default) (color 0 0 0 0))
   )
@@
     (stroke (width 0) (type default) (color 0 0 0 0))
   )
-  (polyline (pts (xy 129.54 119.38) (xy 107.95 119.38))
+  (polyline (pts (xy 128.27 110.49) (xy 106.68 110.49))
     (stroke (width 0) (type default) (color 0 0 0 0))
   )
@@
     (effects (font (size 1.27 1.27)) (justify left bottom))
   )
-  (text "HW standoffs" (at 113.03 116.84 0)
+  (text "Standoffs" (at 111.76 109.22 0)
     (effects (font (size 1.27 1.27)) (justify left bottom))
   )
@@
     (pin "2")
   )
-  (symbol (lib_id "Mechanical:MountingHole") (at 111.76 101.6 0) (unit 1)
-    (in_bom yes) (on_board yes)
-    (property "Reference" "H12" (id 0) (at 114.3 100.4316 0)
-      (effects (font (size 1.27 1.27)) (justify left))
-    )
-    (property "Value" "MountingHole" (id 1) (at 114.3 102.743 0)
-      (effects (font (size 1.27 1.27)) (justify left))
-    )
-    (property "Footprint" "random-keyboard-parts:Generic-Mounthole" (id 2) (at 111.76 101.6 0)
-      (effects (font (size 1.27 1.27)) hide)
-    )
-    (property "Datasheet" "~" (id 3) (at 111.76 101.6 0)
-      (effects (font (size 1.27 1.27)) hide)
-    )
-  )
-  (symbol (lib_id "Mechanical:MountingHole") (at 111.76 91.44 0) (unit 1)
-    (in_bom yes) (on_board yes)
-    (property "Reference" "H10" (id 0) (at 114.3 90.2716 0)
-      (effects (font (size 1.27 1.27)) (justify left))
-    )
-    (property "Value" "MountingHole" (id 1) (at 114.3 92.583 0)
-      (effects (font (size 1.27 1.27)) (justify left))
-    )
-    (property "Footprint" "random-keyboard-parts:Generic-Mounthole" (id 2) (at 111.76 91.44 0)
-      (effects (font (size 1.27 1.27)) hide)
-    )
-    (property "Datasheet" "~" (id 3) (at 111.76 91.44 0)
-      (effects (font (size 1.27 1.27)) hide)
-    )
-  )
-  (symbol (lib_id "Mechanical:MountingHole") (at 111.76 106.68 0) (unit 1)
-    (in_bom yes) (on_board yes)
-    (property "Reference" "H13" (id 0) (at 114.3 105.5116 0)
-      (effects (font (size 1.27 1.27)) (justify left))
-    )
-    (property "Value" "MountingHole" (id 1) (at 114.3 107.823 0)
-      (effects (font (size 1.27 1.27)) (justify left))
-    )
-    (property "Footprint" "random-keyboard-parts:Generic-Mounthole" (id 2) (at 111.76 106.68 0)
-      (effects (font (size 1.27 1.27)) hide)
-    )
-    (property "Datasheet" "~" (id 3) (at 111.76 106.68 0)
-      (effects (font (size 1.27 1.27)) hide)
-    )
-  )
-  (symbol (lib_id "Mechanical:MountingHole") (at 111.76 96.52 0) (unit 1)
-    (in_bom yes) (on_board yes)
-    (property "Reference" "H11" (id 0) (at 114.3 95.3516 0)
-      (effects (font (size 1.27 1.27)) (justify left))
-    )
-    (property "Value" "MountingHole" (id 1) (at 114.3 97.663 0)
-      (effects (font (size 1.27 1.27)) (justify left))
-    )
-    (property "Footprint" "random-keyboard-parts:Generic-Mounthole" (id 2) (at 111.76 96.52 0)
-      (effects (font (size 1.27 1.27)) hide)
-    )
-    (property "Datasheet" "~" (id 3) (at 111.76 96.52 0)
-      (effects (font (size 1.27 1.27)) hide)
-    )
-  )
-  (symbol (lib_id "Mechanical:MountingHole") (at 111.76 111.76 0) (unit 1)
-    (in_bom yes) (on_board yes)
-    (property "Reference" "H14" (id 0) (at 114.3 110.5916 0)
-      (effects (font (size 1.27 1.27)) (justify left))
-    )
-    (property "Value" "MountingHole" (id 1) (at 114.3 112.903 0)
-      (effects (font (size 1.27 1.27)) (justify left))
-    )
-    (property "Footprint" "random-keyboard-parts:Generic-Mounthole" (id 2) (at 111.76 111.76 0)
-      (effects (font (size 1.27 1.27)) hide)
-    )
-    (property "Datasheet" "~" (id 3) (at 111.76 111.76 0)
-      (effects (font (size 1.27 1.27)) hide)
-    )
-  )
-  (symbol (lib_id "Mechanical:MountingHole") (at 111.76 86.36 0) (unit 1)
-    (in_bom yes) (on_board yes)
-    (property "Reference" "H9" (id 0) (at 114.3 85.1916 0)
-      (effects (font (size 1.27 1.27)) (justify left))
-    )
-    (property "Value" "MountingHole" (id 1) (at 114.3 87.503 0)
-      (effects (font (size 1.27 1.27)) (justify left))
-    )
-    (property "Footprint" "random-keyboard-parts:Generic-Mounthole" (id 2) (at 111.76 86.36 0)
-      (effects (font (size 1.27 1.27)) hide)
-    )
-    (property "Datasheet" "~" (id 3) (at 111.76 86.36 0)
+  (symbol (lib_id "Mechanical:MountingHole") (at 110.49 93.98 0) (unit 1)
+    (in_bom yes) (on_board yes)
+    (property "Reference" "H12" (id 0) (at 113.03 92.8116 0)
+      (effects (font (size 1.27 1.27)) (justify left))
+    )
+    (property "Value" "MountingHole" (id 1) (at 113.03 95.123 0)
+      (effects (font (size 1.27 1.27)) (justify left))
+    )
+    (property "Footprint" "random-keyboard-parts:Generic-Mounthole" (id 2) (at 110.49 93.98 0)
+      (effects (font (size 1.27 1.27)) hide)
+    )
+    (property "Datasheet" "~" (id 3) (at 110.49 93.98 0)
+      (effects (font (size 1.27 1.27)) hide)
+    )
+  )
+  (symbol (lib_id "Mechanical:MountingHole") (at 110.49 99.06 0) (unit 1)
+    (in_bom yes) (on_board yes)
+    (property "Reference" "H13" (id 0) (at 113.03 97.8916 0)
+      (effects (font (size 1.27 1.27)) (justify left))
+    )
+    (property "Value" "MountingHole" (id 1) (at 113.03 100.203 0)
+      (effects (font (size 1.27 1.27)) (justify left))
+    )
+    (property "Footprint" "random-keyboard-parts:Generic-Mounthole" (id 2) (at 110.49 99.06 0)
+      (effects (font (size 1.27 1.27)) hide)
+    )
+    (property "Datasheet" "~" (id 3) (at 110.49 99.06 0)
+      (effects (font (size 1.27 1.27)) hide)
+    )
+  )
+  (symbol (lib_id "Mechanical:MountingHole") (at 110.49 88.9 0) (unit 1)
+    (in_bom yes) (on_board yes)
+    (property "Reference" "H11" (id 0) (at 113.03 87.7316 0)
+      (effects (font (size 1.27 1.27)) (justify left))
+    )
+    (property "Value" "MountingHole" (id 1) (at 113.03 90.043 0)
+      (effects (font (size 1.27 1.27)) (justify left))
+    )
+    (property "Footprint" "random-keyboard-parts:Generic-Mounthole" (id 2) (at 110.49 88.9 0)
+      (effects (font (size 1.27 1.27)) hide)
+    )
+    (property "Datasheet" "~" (id 3) (at 110.49 88.9 0)
+      (effects (font (size 1.27 1.27)) hide)
+    )
+  )
+  (symbol (lib_id "Mechanical:MountingHole") (at 110.49 104.14 0) (unit 1)
+    (in_bom yes) (on_board yes)
+    (property "Reference" "H14" (id 0) (at 113.03 102.9716 0)
+      (effects (font (size 1.27 1.27)) (justify left))
+    )
+    (property "Value" "MountingHole" (id 1) (at 113.03 105.283 0)
+      (effects (font (size 1.27 1.27)) (justify left))
+    )
+    (property "Footprint" "random-keyboard-parts:Generic-Mounthole" (id 2) (at 110.49 104.14 0)
+      (effects (font (size 1.27 1.27)) hide)
+    )
+    (property "Datasheet" "~" (id 3) (at 110.49 104.14 0)
+      (effects (font (size 1.27 1.27)) hide)
+    )
+  )
+  (symbol (lib_id "Mechanical:MountingHole") (at 110.49 83.82 0) (unit 1)
+    (in_bom yes) (on_board yes)
+    (property "Reference" "H9" (id 0) (at 113.03 82.6516 0)
+      (effects (font (size 1.27 1.27)) (justify left))
+    )
+    (property "Value" "MountingHole" (id 1) (at 113.03 84.963 0)
+      (effects (font (size 1.27 1.27)) (justify left))
+    )
+    (property "Footprint" "random-keyboard-parts:Generic-Mounthole" (id 2) (at 110.49 83.82 0)
+      (effects (font (size 1.27 1.27)) hide)
+    )
+    (property "Datasheet" "~" (id 3) (at 110.49 83.82 0)
       (effects (font (size 1.27 1.27)) hide)
     )
@@
       (reference "H9") (unit 1) (value "MountingHole") (footprint "random-keyboard-parts:Generic-Mounthole")
     )
-    (path "/2a7d09aa-6af8-4fd8-8830-bfd57a7ed38c"
-      (reference "H10") (unit 1) (value "MountingHole") (footprint "random-keyboard-parts:Generic-Mounthole")
-    )
     (path "/4125bf3c-e5a4-4ba0-80cb-eef115b53706"

Commit message: reduced tab distance
Parts:
- H1, H2, H3, H4, H5, H6, H7, H8: footprint random-keyboard-parts:Generic-Mounthole -> MountingHole:MountingHole_2.2mm_M2_DIN965_Pad
- H11, H12, H13, H14, H9: footprint random-keyboard-parts:Generic-Mounthole -> MountingHole:MountingHole_2.2mm_M2
Changed lines of the file:
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@@
       (effects (font (size 1.27 1.27)) (justify left))
     )
-    (property "Footprint" "random-keyboard-parts:Generic-Mounthole" (id 2) (at 85.09 96.52 0)
+    (property "Footprint" "MountingHole:MountingHole_2.2mm_M2_DIN965_Pad" (id 2) (at 85.09 96.52 0)
       (effects (font (size 1.27 1.27)) hide)
     )
@@
       (effects (font (size 1.27 1.27)) (justify left))
     )
-    (property "Footprint" "random-keyboard-parts:Generic-Mounthole" (id 2) (at 85.09 101.6 0)
+    (property "Footprint" "MountingHole:MountingHole_2.2mm_M2_DIN965_Pad" (id 2) (at 85.09 101.6 0)
       (effects (font (size 1.27 1.27)) hide)
     )
@@
       (effects (font (size 1.27 1.27)) (justify left))
     )
-    (property "Footprint" "random-keyboard-parts:Generic-Mounthole" (id 2) (at 63.5 86.36 0)
+    (property "Footprint" "MountingHole:MountingHole_2.2mm_M2_DIN965_Pad" (id 2) (at 63.5 86.36 0)
       (effects (font (size 1.27 1.27)) hide)
     )
@@
       (effects (font (size 1.27 1.27)) (justify left))
     )
-    (property "Footprint" "random-keyboard-parts:Generic-Mounthole" (id 2) (at 63.5 91.44 0)
+    (property "Footprint" "MountingHole:MountingHole_2.2mm_M2_DIN965_Pad" (id 2) (at 63.5 91.44 0)
       (effects (font (size 1.27 1.27)) hide)
     )
@@
       (effects (font (size 1.27 1.27)) (justify left))
     )
-    (property "Footprint" "random-keyboard-parts:Generic-Mounthole" (id 2) (at 63.5 96.52 0)
+    (property "Footprint" "MountingHole:MountingHole_2.2mm_M2_DIN965_Pad" (id 2) (at 63.5 96.52 0)
       (effects (font (size 1.27 1.27)) hide)
     )
@@
       (effects (font (size 1.27 1.27)) (justify left))
     )
-    (property "Footprint" "random-keyboard-parts:Generic-Mounthole" (id 2) (at 63.5 101.6 0)
+    (property "Footprint" "MountingHole:MountingHole_2.2mm_M2_DIN965_Pad" (id 2) (at 63.5 101.6 0)
       (effects (font (size 1.27 1.27)) hide)
     )
@@
       (effects (font (size 1.27 1.27)) (justify left))
     )
-    (property "Footprint" "random-keyboard-parts:Generic-Mounthole" (id 2) (at 85.09 86.36 0)
+    (property "Footprint" "MountingHole:MountingHole_2.2mm_M2_DIN965_Pad" (id 2) (at 85.09 86.36 0)
       (effects (font (size 1.27 1.27)) hide)
     )
@@
       (effects (font (size 1.27 1.27)) (justify left))
     )
-    (property "Footprint" "random-keyboard-parts:Generic-Mounthole" (id 2) (at 85.09 91.44 0)
+    (property "Footprint" "MountingHole:MountingHole_2.2mm_M2_DIN965_Pad" (id 2) (at 85.09 91.44 0)
       (effects (font (size 1.27 1.27)) hide)
     )
@@
       (effects (font (size 1.27 1.27)) (justify left))
     )
-    (property "Footprint" "random-keyboard-parts:Generic-Mounthole" (id 2) (at 110.49 93.98 0)
+    (property "Footprint" "MountingHole:MountingHole_2.2mm_M2" (id 2) (at 110.49 93.98 0)
       (effects (font (size 1.27 1.27)) hide)
     )
@@
       (effects (font (size 1.27 1.27)) (justify left))
     )
-    (property "Footprint" "random-keyboard-parts:Generic-Mounthole" (id 2) (at 110.49 99.06 0)
+    (property "Footprint" "MountingHole:MountingHole_2.2mm_M2" (id 2) (at 110.49 99.06 0)
       (effects (font (size 1.27 1.27)) hide)
     )
@@
       (effects (font (size 1.27 1.27)) (justify left))
     )
-    (property "Footprint" "random-keyboard-parts:Generic-Mounthole" (id 2) (at 110.49 88.9 0)
+    (property "Footprint" "MountingHole:MountingHole_2.2mm_M2" (id 2) (at 110.49 88.9 0)
       (effects (font (size 1.27 1.27)) hide)
     )
@@
       (effects (font (size 1.27 1.27)) (justify left))
     )
-    (property "Footprint" "random-keyboard-parts:Generic-Mounthole" (id 2) (at 110.49 104.14 0)
+    (property "Footprint" "MountingHole:MountingHole_2.2mm_M2" (id 2) (at 110.49 104.14 0)
       (effects (font (size 1.27 1.27)) hide)
     )
@@
       (effects (font (size 1.27 1.27)) (justify left))
     )
-    (property "Footprint" "random-keyboard-parts:Generic-Mounthole" (id 2) (at 110.49 83.82 0)
+    (property "Footprint" "MountingHole:MountingHole_2.2mm_M2" (id 2) (at 110.49 83.82 0)
       (effects (font (size 1.27 1.27)) hide)
     )
@@
     )
     (path "/00000000-0000-0000-0000-00006111b67c"
-      (reference "H1") (unit 1) (value "MountingHole") (footprint "random-keyboard-parts:Generic-Mounthole")
+      (reference "H1") (unit 1) (value "MountingHole") (footprint "MountingHole:MountingHole_2.2mm_M2_DIN965_Pad")
     )
     (path "/00000000-0000-0000-0000-00006111b682"
-      (reference "H2") (unit 1) (value "MountingHole") (footprint "random-keyboard-parts:Generic-Mounthole")
+      (reference "H2") (unit 1) (value "MountingHole") (footprint "MountingHole:MountingHole_2.2mm_M2_DIN965_Pad")
     )
     (path "/00000000-0000-0000-0000-00006111b688"
-      (reference "H3") (unit 1) (value "MountingHole") (footprint "random-keyboard-parts:Generic-Mounthole")
+      (reference "H3") (unit 1) (value "MountingHole") (footprint "MountingHole:MountingHole_2.2mm_M2_DIN965_Pad")
     )
     (path "/00000000-0000-0000-0000-00006111b68e"
-      (reference "H4") (unit 1) (value "MountingHole") (footprint "random-keyboard-parts:Generic-Mounthole")
+      (reference "H4") (unit 1) (value "MountingHole") (footprint "MountingHole:MountingHole_2.2mm_M2_DIN965_Pad")
     )
     (path "/00000000-0000-0000-0000-00006111b694"
-      (reference "H5") (unit 1) (value "MountingHole") (footprint "random-keyboard-parts:Generic-Mounthole")
+      (reference "H5") (unit 1) (value "MountingHole") (footprint "MountingHole:MountingHole_2.2mm_M2_DIN965_Pad")
     )
     (path "/00000000-0000-0000-0000-00006111b69a"
-      (reference "H6") (unit 1) (value "MountingHole") (footprint "random-keyboard-parts:Generic-Mounthole")
+      (reference "H6") (unit 1) (value "MountingHole") (footprint "MountingHole:MountingHole_2.2mm_M2_DIN965_Pad")
     )
     (path "/00000000-0000-0000-0000-00006111adf9"
-      (reference "H7") (unit 1) (value "MountingHole") (footprint "random-keyboard-parts:Generic-Mounthole")
+      (reference "H7") (unit 1) (value "MountingHole") (footprint "MountingHole:MountingHole_2.2mm_M2_DIN965_Pad")
     )
     (path "/00000000-0000-0000-0000-00006111adff"
-      (reference "H8") (unit 1) (value "MountingHole") (footprint "random-keyboard-parts:Generic-Mounthole")
+      (reference "H8") (unit 1) (value "MountingHole") (footprint "MountingHole:MountingHole_2.2mm_M2_DIN965_Pad")
     )
     (path "/bcc40fb8-020a-4739-8e85-82c40b31a03a"
-      (reference "H9") (unit 1) (value "MountingHole") (footprint "random-keyboard-parts:Generic-Mounthole")
+      (reference "H9") (unit 1) (value "MountingHole") (footprint "MountingHole:MountingHole_2.2mm_M2")
     )
     (path "/4125bf3c-e5a4-4ba0-80cb-eef115b53706"
-      (reference "H11") (unit 1) (value "MountingHole") (footprint "random-keyboard-parts:Generic-Mounthole")
+      (reference "H11") (unit 1) (value "MountingHole") (footprint "MountingHole:MountingHole_2.2mm_M2")
     )
     (path "/0020d0ea-8d9d-4dfe-880a-001f8e7583fa"
-      (reference "H12") (unit 1) (value "MountingHole") (footprint "random-keyboard-parts:Generic-Mounthole")
+      (reference "H12") (unit 1) (value "MountingHole") (footprint "MountingHole:MountingHole_2.2mm_M2")
     )
     (path "/308df6f4-9077-4108-9839-cf6f6eca2987"
-      (reference "H13") (unit 1) (value "MountingHole") (footprint "random-keyboard-parts:Generic-Mounthole")
+      (reference "H13") (unit 1) (value "MountingHole") (footprint "MountingHole:MountingHole_2.2mm_M2")
     )
     (path "/6d76b69f-13fd-4d71-a5b4-e26d6a201478"
-      (reference "H14") (unit 1) (value "MountingHole") (footprint "random-keyboard-parts:Generic-Mounthole")
+      (reference "H14") (unit 1) (value "MountingHole") (footprint "MountingHole:MountingHole_2.2mm_M2")
     )
     (path "/00000000-0000-0000-0000-00006175f9b8"

Commit message: Plate B updates
Parts:
- R1: footprint Resistor_SMD:R_0603_1608Metric_Pad1.05x0.95mm_HandSolder -> Resistor_SMD:R_0201_0603Metric_Pad0.64x0.40mm_HandSolder
- U1, U10, U11, U12, U13, U14, U15, U16, U17, U18, U19, U2, U20, U21, U22, U23, U24, U25, U26, U27, U28, U29, U3, U30, U31, U32, U33, U34, U35, U36, U37, U38, U39, U4, U40, U41, U42, U43, U44, U45, U46, U47, U48, U5, U50, U51, U52, U6, U7, U8, U9: footprint Keeb_footprints:MX100_cutout_plated -> Keeb_footprints:MX100_cutout
- U49: footprint Keeb_footprints:EC11_cutout_plated -> Keeb_footprints:EC11_cutout
Connections:
- net GND: now also R1.2; no longer R1.1

Commit message: renamed folder
Parts:
- added H10: MountingHole, MountingHole:MountingHole_2.2mm_M2, symbol Mechanical:MountingHole
- U52: footprint Keeb_footprints:MX100_cutout -> Keeb_footprints:EC11_cutout
Changed lines of the file:
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@@
       (effects (font (size 1.524 1.524)) (justify left))
     )
-    (property "Footprint" "Keeb_footprints:MX100_cutout" (id 2) (at 161.29 62.23 0)
+    (property "Footprint" "Keeb_footprints:EC11_cutout" (id 2) (at 161.29 62.23 0)
       (effects (font (size 1.524 1.524)) hide)
     )
@@
     )
     (property "Datasheet" "~" (id 3) (at 110.49 104.14 0)
+      (effects (font (size 1.27 1.27)) hide)
+    )
+  )
+  (symbol (lib_id "Mechanical:MountingHole") (at 132.08 104.14 0) (unit 1)
+    (in_bom yes) (on_board yes)
+    (property "Reference" "H10" (id 0) (at 134.62 102.9716 0)
+      (effects (font (size 1.27 1.27)) (justify left))
+    )
+    (property "Value" "MountingHole" (id 1) (at 134.62 105.283 0)
+      (effects (font (size 1.27 1.27)) (justify left))
+    )
+    (property "Footprint" "MountingHole:MountingHole_2.2mm_M2" (id 2) (at 132.08 104.14 0)
+      (effects (font (size 1.27 1.27)) hide)
+    )
+    (property "Datasheet" "~" (id 3) (at 132.08 104.14 0)
       (effects (font (size 1.27 1.27)) hide)
     )
@@
       (reference "H9") (unit 1) (value "MountingHole") (footprint "MountingHole:MountingHole_2.2mm_M2")
     )
+    (path "/6ee99e3f-5741-4564-ac73-17280593745c"
+      (reference "H10") (unit 1) (value "MountingHole") (footprint "MountingHole:MountingHole_2.2mm_M2")
+    )
     (path "/4125bf3c-e5a4-4ba0-80cb-eef115b53706"
       (reference "H11") (unit 1) (value "MountingHole") (footprint "MountingHole:MountingHole_2.2mm_M2")
@@
     )
     (path "/00000000-0000-0000-0000-00005f4bc873"
-      (reference "U52") (unit 1) (value "HOLE") (footprint "Keeb_footprints:MX100_cutout")
-    )
-  )
+      (reference "U52") (unit 1) (value "HOLE") (footprint "Keeb_footprints:EC11_cutout")
+    )
+  )
