File: 01_pcb/1.0 solder/pcb.kicad_sch (KiCad schematic)
At the start: 128 parts, among them J1 TYPE-C-31-M12_13, J2 AVR-ISP-6_mod, K1 KEYSW, K10 KEYSW, K11 KEYSW, K12 KEYSW, K13 KEYSW, K14 KEYSW, K15 KEYSW, K16 KEYSW, K17 KEYSW, K18 KEYSW, K19 KEYSW, K2 KEYSW, K20 KEYSW, K21 KEYSW, K22 KEYSW, K23 KEYSW, K24 KEYSW, K25 KEYSW, K26 KEYSW, K27 KEYSW, K28 KEYSW, K29 KEYSW, K3 KEYSW, K30 KEYSW, K31 KEYSW, K32 KEYSW, K33 KEYSW, K34 KEYSW, K35 KEYSW, K36 KEYSW, K37 KEYSW, K38 KEYSW, K39 KEYSW, K4 KEYSW, K40 KEYSW, K41 KEYSW, K42 KEYSW, K43 KEYSW, K44 KEYSW, K45 KEYSW, K46 KEYSW, K47 KEYSW, K48 KEYSW, K49 KEYSW, K5 KEYSW, K50 KEYSW, K51 KEYSW, K52 KEYSW, K6 KEYSW, K7 KEYSW, K8 KEYSW, K9 KEYSW, SW1 SW_PUSH, SW2 Rotary_Encoder_Switch, U1 ATMEGA32U4, U2 PRTR5V0U2X, Y1 16MHz

Commit message: add 3d models to kicad footprints
Parts:
- C1: footprint Capacitor_SMD:C_0805_2012Metric_Pad1.18x1.45mm_HandSolder -> Keeb_footprints:C_0805_2012Metric_Pad1.18x1.45mm_HandSolder
- C2, C3, C5, C6, CX1, CX2: footprint Capacitor_SMD:C_0805_2012Metric_Pad1.15x1.40mm_HandSolder -> Keeb_footprints:C_0805_2012Metric_Pad1.18x1.45mm_HandSolder
- R1, R2, R3, R4, RCC1, RCC2, RSW1: footprint Resistor_SMD:R_0805_2012Metric_Pad1.15x1.40mm_HandSolder -> Keeb_footprints:R_0805_2012Metric_Pad1.20x1.40mm_HandSolder
Changed lines of the file:
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@@
       (effects (font (size 0.762 0.762)) (justify left))
     )
-    (property "Footprint" "Capacitor_SMD:C_0805_2012Metric_Pad1.15x1.40mm_HandSolder" (id 2) (at 80.01 231.14 0)
+    (property "Footprint" "Keeb_footprints:C_0805_2012Metric_Pad1.18x1.45mm_HandSolder" (id 2) (at 80.01 231.14 0)
       (effects (font (size 1.27 1.27)) hide)
     )
@@
       (effects (font (size 0.762 0.762)) (justify left))
     )
-    (property "Footprint" "Capacitor_SMD:C_0805_2012Metric_Pad1.15x1.40mm_HandSolder" (id 2) (at 90.17 231.14 0)
+    (property "Footprint" "Keeb_footprints:C_0805_2012Metric_Pad1.18x1.45mm_HandSolder" (id 2) (at 90.17 231.14 0)
       (effects (font (size 1.27 1.27)) hide)
     )
@@
       (effects (font (size 0.7112 0.7112)))
     )
-    (property "Footprint" "Resistor_SMD:R_0805_2012Metric_Pad1.15x1.40mm_HandSolder" (id 2) (at 72.39 154.94 0)
+    (property "Footprint" "Keeb_footprints:R_0805_2012Metric_Pad1.20x1.40mm_HandSolder" (id 2) (at 72.39 154.94 0)
       (effects (font (size 1.27 1.27)) hide)
     )
@@
       (effects (font (size 0.7112 0.7112)))
     )
-    (property "Footprint" "Resistor_SMD:R_0805_2012Metric_Pad1.15x1.40mm_HandSolder" (id 2) (at 72.39 149.86 0)
+    (property "Footprint" "Keeb_footprints:R_0805_2012Metric_Pad1.20x1.40mm_HandSolder" (id 2) (at 72.39 149.86 0)
       (effects (font (size 1.27 1.27)) hide)
     )
@@
       (effects (font (size 0.762 0.762)) (justify left))
     )
-    (property "Footprint" "Capacitor_SMD:C_0805_2012Metric_Pad1.15x1.40mm_HandSolder" (id 2) (at 45.72 232.41 0)
+    (property "Footprint" "Keeb_footprints:C_0805_2012Metric_Pad1.18x1.45mm_HandSolder" (id 2) (at 45.72 232.41 0)
       (effects (font (size 1.27 1.27)) hide)
     )
@@
       (effects (font (size 0.762 0.762)) (justify left))
     )
-    (property "Footprint" "Capacitor_SMD:C_0805_2012Metric_Pad1.18x1.45mm_HandSolder" (id 2) (at 50.8 232.41 0)
+    (property "Footprint" "Keeb_footprints:C_0805_2012Metric_Pad1.18x1.45mm_HandSolder" (id 2) (at 50.8 232.41 0)
       (effects (font (size 1.27 1.27)) hide)
     )
@@
       (effects (font (size 0.762 0.762)) (justify left))
     )
-    (property "Footprint" "Capacitor_SMD:C_0805_2012Metric_Pad1.15x1.40mm_HandSolder" (id 2) (at 55.88 232.41 0)
+    (property "Footprint" "Keeb_footprints:C_0805_2012Metric_Pad1.18x1.45mm_HandSolder" (id 2) (at 55.88 232.41 0)
       (effects (font (size 1.27 1.27)) hide)
     )
@@
       (effects (font (size 0.762 0.762)) (justify left))
     )
-    (property "Footprint" "Capacitor_SMD:C_0805_2012Metric_Pad1.15x1.40mm_HandSolder" (id 2) (at 60.96 232.41 0)
+    (property "Footprint" "Keeb_footprints:C_0805_2012Metric_Pad1.18x1.45mm_HandSolder" (id 2) (at 60.96 232.41 0)
       (effects (font (size 1.27 1.27)) hide)
     )
@@
       (effects (font (size 0.7112 0.7112)))
     )
-    (property "Footprint" "Resistor_SMD:R_0805_2012Metric_Pad1.15x1.40mm_HandSolder" (id 2) (at 118.11 156.972 90)
+    (property "Footprint" "Keeb_footprints:R_0805_2012Metric_Pad1.20x1.40mm_HandSolder" (id 2) (at 118.11 156.972 90)
       (effects (font (size 1.27 1.27)) hide)
     )
@@
       (effects (font (size 0.762 0.762)))
     )
-    (property "Footprint" "Resistor_SMD:R_0805_2012Metric_Pad1.15x1.40mm_HandSolder" (id 2) (at 195.58 160.782 90)
+    (property "Footprint" "Keeb_footprints:R_0805_2012Metric_Pad1.20x1.40mm_HandSolder" (id 2) (at 195.58 160.782 90)
       (effects (font (size 1.27 1.27)) hide)
     )
@@
       (effects (font (size 0.7112 0.7112)))
     )
-    (property "Footprint" "Resistor_SMD:R_0805_2012Metric_Pad1.15x1.40mm_HandSolder" (id 2) (at 137.668 229.87 90)
+    (property "Footprint" "Keeb_footprints:R_0805_2012Metric_Pad1.20x1.40mm_HandSolder" (id 2) (at 137.668 229.87 90)
       (effects (font (size 1.27 1.27)) hide)
     )
@@
       (effects (font (size 0.7112 0.7112)))
     )
-    (property "Footprint" "Resistor_SMD:R_0805_2012Metric_Pad1.15x1.40mm_HandSolder" (id 2) (at 110.998 229.87 90)
+    (property "Footprint" "Keeb_footprints:R_0805_2012Metric_Pad1.20x1.40mm_HandSolder" (id 2) (at 110.998 229.87 90)
       (effects (font (size 1.27 1.27)) hide)
     )
@@
       (effects (font (size 0.7112 0.7112)))
     )
-    (property "Footprint" "Capacitor_SMD:C_0805_2012Metric_Pad1.15x1.40mm_HandSolder" (id 2) (at 123.19 147.32 0)
+    (property "Footprint" "Keeb_footprints:C_0805_2012Metric_Pad1.18x1.45mm_HandSolder" (id 2) (at 123.19 147.32 0)
       (effects (font (size 1.27 1.27)) hide)
     )
@@
       (effects (font (size 0.762 0.762)))
     )
-    (property "Footprint" "Resistor_SMD:R_0805_2012Metric_Pad1.15x1.40mm_HandSolder" (id 2) (at 204.47 237.49 0)
+    (property "Footprint" "Keeb_footprints:R_0805_2012Metric_Pad1.20x1.40mm_HandSolder" (id 2) (at 204.47 237.49 0)
       (effects (font (size 1.27 1.27)) hide)
     )
@@
     )
     (path "/00000000-0000-0000-0000-00005df8174e"
-      (reference "C1") (unit 1) (value ".1uF") (footprint "Capacitor_SMD:C_0805_2012Metric_Pad1.18x1.45mm_HandSolder")
+      (reference "C1") (unit 1) (value ".1uF") (footprint "Keeb_footprints:C_0805_2012Metric_Pad1.18x1.45mm_HandSolder")
     )
     (path "/00000000-0000-0000-0000-00005dfa1ef6"
-      (reference "C2") (unit 1) (value ".1uF") (footprint "Capacitor_SMD:C_0805_2012Metric_Pad1.15x1.40mm_HandSolder")
+      (reference "C2") (unit 1) (value ".1uF") (footprint "Keeb_footprints:C_0805_2012Metric_Pad1.18x1.45mm_HandSolder")
     )
     (path "/00000000-0000-0000-0000-00005dfc24a4"
-      (reference "C3") (unit 1) (value ".1uF") (footprint "Capacitor_SMD:C_0805_2012Metric_Pad1.15x1.40mm_HandSolder")
+      (reference "C3") (unit 1) (value ".1uF") (footprint "Keeb_footprints:C_0805_2012Metric_Pad1.18x1.45mm_HandSolder")
     )
     (path "/00000000-0000-0000-0000-00005df80643"
-      (reference "C5") (unit 1) (value "10uF") (footprint "Capacitor_SMD:C_0805_2012Metric_Pad1.15x1.40mm_HandSolder")
+      (reference "C5") (unit 1) (value "10uF") (footprint "Keeb_footprints:C_0805_2012Metric_Pad1.18x1.45mm_HandSolder")
     )
     (path "/00000000-0000-0000-0000-00005e589c1c"
-      (reference "C6") (unit 1) (value "1uF") (footprint "Capacitor_SMD:C_0805_2012Metric_Pad1.15x1.40mm_HandSolder")
+      (reference "C6") (unit 1) (value "1uF") (footprint "Keeb_footprints:C_0805_2012Metric_Pad1.18x1.45mm_HandSolder")
     )
     (path "/00000000-0000-0000-0000-00005dd7acb1"
-      (reference "CX1") (unit 1) (value "22pF") (footprint "Capacitor_SMD:C_0805_2012Metric_Pad1.15x1.40mm_HandSolder")
+      (reference "CX1") (unit 1) (value "22pF") (footprint "Keeb_footprints:C_0805_2012Metric_Pad1.18x1.45mm_HandSolder")
     )
     (path "/00000000-0000-0000-0000-00005dd7ba72"
-      (reference "CX2") (unit 1) (value "22pF") (footprint "Capacitor_SMD:C_0805_2012Metric_Pad1.15x1.40mm_HandSolder")
+      (reference "CX2") (unit 1) (value "22pF") (footprint "Keeb_footprints:C_0805_2012Metric_Pad1.18x1.45mm_HandSolder")
     )
     (path "/00000000-0000-0000-0000-00005db57a33"
@@
     )
     (path "/00000000-0000-0000-0000-00005e28a0b7"
-      (reference "R1") (unit 1) (value "10k") (footprint "Resistor_SMD:R_0805_2012Metric_Pad1.15x1.40mm_HandSolder")
+      (reference "R1") (unit 1) (value "10k") (footprint "Keeb_footprints:R_0805_2012Metric_Pad1.20x1.40mm_HandSolder")
     )
     (path "/00000000-0000-0000-0000-00005e4290ae"
-      (reference "R2") (unit 1) (value "22") (footprint "Resistor_SMD:R_0805_2012Metric_Pad1.15x1.40mm_HandSolder")
+      (reference "R2") (unit 1) (value "22") (footprint "Keeb_footprints:R_0805_2012Metric_Pad1.20x1.40mm_HandSolder")
     )
     (path "/00000000-0000-0000-0000-00005e44c75b"
-      (reference "R3") (unit 1) (value "22") (footprint "Resistor_SMD:R_0805_2012Metric_Pad1.15x1.40mm_HandSolder")
+      (reference "R3") (unit 1) (value "22") (footprint "Keeb_footprints:R_0805_2012Metric_Pad1.20x1.40mm_HandSolder")
     )
     (path "/00000000-0000-0000-0000-00005f9dc91d"
-      (reference "R4") (unit 1) (value "1k") (footprint "Resistor_SMD:R_0805_2012Metric_Pad1.15x1.40mm_HandSolder")
+      (reference "R4") (unit 1) (value "1k") (footprint "Keeb_footprints:R_0805_2012Metric_Pad1.20x1.40mm_HandSolder")
     )
     (path "/00000000-0000-0000-0000-00005dd97927"
-      (reference "RCC1") (unit 1) (value "5.1k") (footprint "Resistor_SMD:R_0805_2012Metric_Pad1.15x1.40mm_HandSolder")
+      (reference "RCC1") (unit 1) (value "5.1k") (footprint "Keeb_footprints:R_0805_2012Metric_Pad1.20x1.40mm_HandSolder")
     )
     (path "/00000000-0000-0000-0000-00005dd95fdc"
-      (reference "RCC2") (unit 1) (value "5.1k") (footprint "Resistor_SMD:R_0805_2012Metric_Pad1.15x1.40mm_HandSolder")
+      (reference "RCC2") (unit 1) (value "5.1k") (footprint "Keeb_footprints:R_0805_2012Metric_Pad1.20x1.40mm_HandSolder")
     )
     (path "/00000000-0000-0000-0000-00005e1f1159"
-      (reference "RSW1") (unit 1) (value "10k") (footprint "Resistor_SMD:R_0805_2012Metric_Pad1.15x1.40mm_HandSolder")
+      (reference "RSW1") (unit 1) (value "10k") (footprint "Keeb_footprints:R_0805_2012Metric_Pad1.20x1.40mm_HandSolder")
     )
     (path "/00000000-0000-0000-0000-00005e1efd9f"
