File: 01_pcb/2.1 hotswap/pcb.kicad_pcb (KiCad board)
At the start: 2 copper layers, 251.2 x 81.3 mm, 138 parts, among them J1 TYPE-C-31-M12_13, J2 AVR-ISP-6_mod, J3 Conn_01x01, J4 Conn_01x01, J5 Conn_01x01, J6 Conn_01x01, J7 Conn_01x01, J8 4PIN, K1 KEYSW, K10 KEYSW, K12 KEYSW, K13 KEYSW, K14 KEYSW, K15 KEYSW, K16 KEYSW, K17 KEYSW, K18 KEYSW, K19 KEYSW, K2 KEYSW, K20 KEYSW, K21 KEYSW, K23 KEYSW, K24 KEYSW, K25 KEYSW, K26 KEYSW, K27 KEYSW, K28 KEYSW, K29 KEYSW, K3 KEYSW, K30 KEYSW, K31 KEYSW, K32 KEYSW, K33 KEYSW, K34 KEYSW, K36 KEYSW, K37 KEYSW, K38 KEYSW, K39 KEYSW, K4 KEYSW, K42 KEYSW, K43 KEYSW, K44 KEYSW, K45 KEYSW, K46 KEYSW, K47 KEYSW, K48 KEYSW, K49 KEYSW, K5 KEYSW, K50 KEYSW, K51 KEYSW, K52 KEYSW, K6 KEYSW, K7 KEYSW, K8 KEYSW, K9 KEYSW, SW1 SW_PUSH, SW2 Rotary_Encoder_Switch, U1 ATMEGA32U4, U2 PRTR5V0U2X, Y1 16MHz

Commit message: remove flex cuts and encoder
Parts:
- removed H1, H2, H3, H4, H5: MountingHole, MountingHole:MountingHole_2.2mm_M2_DIN965_Pad
- removed SW2: Rotary_Encoder_Switch, Keebio-Parts:RotaryEncoder_EC11
- K49: footprint MX_Only:MXOnly-1U-NoLED -> MX_Only:MXOnly-1U-Hotswap
Connections:
- U1 pad 38: enc0a -> unconnected-(U1-Pad38)
- U1 pad 39: enc0b -> unconnected-(U1-Pad39)
Routing:
- net col6: track 436.5 -> 234.8 mm
- net col2: track 556.6 -> 356.0 mm
- net col7: track 395.1 -> 225.1 mm
- net col3: track 460.7 -> 293.1 mm
- net col5: track 364.2 -> 256.8 mm
- net col9: track 295.7 -> 189.0 mm
- net enc0a: track 87.8 -> 0.00 mm, vias 1 -> 0
- net enc0b: track 86.0 -> 0.00 mm, vias 1 -> 0
- net col10: track 239.8 -> 171.6 mm
- net col12: track 112.4 -> 97.1 mm, vias 4 -> 5
- net col1: track 385.9 -> 375.2 mm
- net col11: track 112.0 -> 105.3 mm
- net Net-(D49-Pad2): track 22.0 -> 25.6 mm
- net col4: track 278.3 -> 275.8 mm
- net row0: track 237.4 -> 235.2 mm
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Other:
- outline, holes or cut-outs redrawn
- board text added: "lucy rev 2.1"
- board text added: "lucy rev. 2.1 2023.01.25"
- board text removed: "lucy rev 2.0"
- board text removed: "lucy rev. 2.0 2022.08.31"

Commit message: add 3d models to kicad footprints
Parts:
- R1, R2, R3, R4, RCC1, RCC2, RSW1: footprint Resistor_SMD:R_0805_2012Metric_Pad1.15x1.40mm_HandSolder -> Keeb_footprints:R_0805_2012Metric_Pad1.20x1.40mm_HandSolder

Commit message: ¯\_(ツ)_/¯
Parts:
- removed J4, J5, J6, J7: Conn_01x01, TestPoint:TestPoint_Keystone_5000-5004_Miniature
- J3: value Conn_01x01 -> Conn_01x05_Female; footprint TestPoint:TestPoint_Keystone_5000-5004_Miniature -> Connector_PinHeader_2.54mm:PinHeader_1x05_P2.54mm_Vertical
- moved J8 16.1 mm to (103.1, 61.3), turned to -90 degrees
- moved J3 10.0 mm to (308.2, 62.9)
- moved RCC2 3.08 mm to (110.3, 56.2), turned to 180 degrees
Connections:
- J3 pad 1: Net-(J3-Pad1) -> Net-(U1-Pad22)
- U1 pad 18: Net-(J3-Pad1) -> Net-(U1-Pad18)
- U1 pad 19: Net-(J4-Pad1) -> Net-(U1-Pad19)
- U1 pad 20: Net-(J5-Pad1) -> Net-(U1-Pad20)
- U1 pad 21: Net-(J6-Pad1) -> Net-(U1-Pad21)
- U1 pad 22: Net-(J7-Pad1) -> Net-(U1-Pad22)
Routing:
- net Net-(J7-Pad1): track 35.3 -> 0.00 mm, vias 1 -> 0
- net Net-(U1-Pad22): track 0.00 -> 35.2 mm, vias 0 -> 1
- net Net-(J6-Pad1): track 32.8 -> 0.00 mm, vias 1 -> 0
- net Net-(U1-Pad21): track 0.00 -> 32.7 mm, vias 0 -> 1
- net Net-(J5-Pad1): track 30.2 -> 0.00 mm, vias 1 -> 0
- net Net-(U1-Pad20): track 0.00 -> 30.2 mm, vias 0 -> 1
- net Net-(J4-Pad1): track 28.0 -> 0.00 mm, vias 1 -> 0
- net Net-(U1-Pad19): track 0.00 -> 27.7 mm, vias 0 -> 1
- net Net-(J3-Pad1): track 26.6 -> 0.00 mm, vias 1 -> 0
- net Net-(U1-Pad18): track 0.00 -> 26.3 mm, vias 0 -> 1
- net D+: track 247.3 -> 257.1 mm
- net VCC: track 483.5 -> 491.6 mm, vias 8 -> 10
- net D-: track 247.4 -> 254.9 mm
- net col1: track 375.2 -> 381.4 mm
- net Net-(J1-PadB5): track 23.1 -> 22.6 mm
