File: 01_pcb/2.2 hotswap/pcb.kicad_sch (KiCad schematic)
At the start: 128 parts, among them J1 TYPE-C-31-M12_13, J2 AVR-ISP-6_mod, J3 Conn_01x05_Female, J8 4PIN, K1 KEYSW, K10 KEYSW, K11 KEYSW, K12 KEYSW, K13 KEYSW, K14 KEYSW, K15 KEYSW, K16 KEYSW, K17 KEYSW, K18 KEYSW, K19 KEYSW, K2 KEYSW, K20 KEYSW, K21 KEYSW, K22 KEYSW, K23 KEYSW, K24 KEYSW, K25 KEYSW, K26 KEYSW, K27 KEYSW, K28 KEYSW, K29 KEYSW, K3 KEYSW, K30 KEYSW, K31 KEYSW, K32 KEYSW, K33 KEYSW, K34 KEYSW, K35 KEYSW, K36 KEYSW, K37 KEYSW, K38 KEYSW, K39 KEYSW, K4 KEYSW, K40 KEYSW, K41 KEYSW, K42 KEYSW, K43 KEYSW, K44 KEYSW, K45 KEYSW, K46 KEYSW, K47 KEYSW, K48 KEYSW, K49 KEYSW, K5 KEYSW, K50 KEYSW, K51 KEYSW, K52 KEYSW, K6 KEYSW, K7 KEYSW, K8 KEYSW, K9 KEYSW, SW1 SW_PUSH, U1 ATMEGA32U4, U2 PRTR5V0U2X, Y1 16MHz

Commit message: moved USB port data line resistors
also added 3d models, etc.
Connections:
- net D+: no longer J8.3
- net D-: no longer J8.2
- net DBUS+: now also J8.3
- net DBUS-: now also J8.2
- net XTAL1: now also CX2.1, Y1.3; no longer CX1.1, Y1.1
- net XTAL2: now also CX1.1, Y1.1; no longer CX2.1, Y1.3
- net col1 renamed col1/sck
- net col2 renamed col2/miso
- net row0 renamed row0/mosi
Other:
- moved on the sheet: J2, RSW1, SW1
