File: 01_pcb/3.0 hotswap/pcb/pcb.kicad_pcb (KiCad board)
At the start: 2 copper layers, 256 x 75 mm, 128 parts, among them J1 TYPE-C-31-M12_13, J2 AVR-ISP-6_mod, J3 4PIN, J5 Conn_01x08, SW1 SW_PUSH, U1 ATmega32U4-M, U2 PRTR5V0U2X, Y1 16MHz

Commit message: add stitching vias
Parts:
- removed LED1: LED, LED_SMD:LED_0805_2012Metric_Pad1.15x1.40mm_HandSolder
- removed R4: 1k, Resistor_SMD:R_0603_1608Metric
- removed U2: PRTR5V0U2X, Package_TO_SOT_SMD:SOT-143
- added U4: USBLC6-2SC6, Package_TO_SOT_SMD:SOT-23-6, B.Cu at (44.2, 36.7)
- moved R2 2.00 mm to (257.0, 48.1)
- moved R3 1.93 mm to (258.9, 48.1), turned to -90 degrees
- moved F1 0.47 mm to (40.5, 39.7)
Connections:
- R2 pad 1: D+ -> D-
- R2 pad 2: DBUS+ -> DBUS-
- R3 pad 1: D- -> DBUS+
- R3 pad 2: DBUS- -> D+
Routing:
- net GND: track 220.0 -> 321.7 mm, vias 73 -> 195
- net VCC: track 319.2 -> 313.5 mm
- net Net-(LED1-A): track 2.48 -> 0.00 mm
- net DBUS+: track 237.9 -> 240.1 mm
- net DBUS-: track 238.1 -> 239.7 mm
- net ISP_Reset: track 35.1 -> 34.2 mm
- net col11/miso: track 118.7 -> 119.5 mm
- net col10/mosi: track 137.1 -> 137.9 mm
- net VBUS: track 21.5 -> 22.0 mm

Commit message: replaced SRV05-4 footprint
Parts:
- U4: footprint Package_TO_SOT_SMD:SOT-23-6 -> marbastlib-various:SOT-23-6-routable
Routing:
- net GND: track 321.7 -> 451.7 mm, vias 195 -> 328
- net row3: track 292.1 -> 273.6 mm
- net DBUS+: track 240.1 -> 242.9 mm
- net col11/miso: track 119.5 -> 120.5 mm
- net col10/mosi: track 137.9 -> 138.9 mm
- net ISP_Reset: track 34.2 -> 35.1 mm
- net DBUS-: track 239.7 -> 240.2 mm
- net Net-(J1-CC2): track 11.2 -> 10.7 mm

Commit message: backups
Parts:
- moved R1 0.68 mm to (254.9, 63.6)
Routing:
- net GND: track 451.7 -> 484.3 mm, vias 328 -> 337
- net col12/sck: track 116.3 -> 121.8 mm
- net row1: track 243.3 -> 244.8 mm
- net row2: track 257.1 -> 258.0 mm
- net Net-(U1-~{HWB}/PE2): track 3.46 -> 4.33 mm
- net col1: track 300.7 -> 301.3 mm
