File: 01_pcb/3.0_hotswap-QFN-0603/pcb/pcb.kicad_pcb (KiCad board)
At the start: 2 copper layers, 256 x 75 mm, 126 parts, among them J1 TYPE-C-31-M12_13, J2 AVR-ISP-6_mod, J3 4PIN, J5 Conn_01x08, SW1 SW_PUSH, U1 ATmega32U4-M, U4 USBLC6-2SC6, Y1 16MHz

Commit message: added text
Other:
- board text added: "anything is possible with a dremel and a little courage"
- board text added: "lucy rev 3.0"
- board text added: "lucy v3-QFN 2023.04.12"
Changed lines of the file:
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@@
       (outputformat 1)
       (mirror false)
-      (drillshape 1)
+      (drillshape 0)
       (scaleselection 1)
-      (outputdirectory "")
+      (outputdirectory "gerbers/")
     )
   )
@@
     (fp_line (start 1 0.6) (end 1 -0.6)
       (stroke (width 0.1) (type solid)) (layer "B.Fab"))
-    (pad "1" smd roundrect (at -1.025 0 90) (size 1.15 1.4) (layers "B.Cu" "B.Paste" "B.Mask") (roundrect_rratio 0.217391)
+    (pad "1" smd roundrect (at -1.025 0 90) (size 1.15 1.4) (layers "B.Cu" "B.Paste" "B.Mask") (roundrect_rratio 0.2173913043)
       (net 3 "VCC") (pintype "passive"))
-    (pad "2" smd roundrect (at 1.025 0 90) (size 1.15 1.4) (layers "B.Cu" "B.Paste" "B.Mask") (roundrect_rratio 0.217391)
+    (pad "2" smd roundrect (at 1.025 0 90) (size 1.15 1.4) (layers "B.Cu" "B.Paste" "B.Mask") (roundrect_rratio 0.2173913043)
       (net 59 "VBUS") (pintype "passive"))
     (model "${KICAD6_3DMODEL_DIR}/Fuse.3dshapes/Fuse_0805_2012Metric.wrl"
@@
     (fp_line (start 3.5 3.5) (end 3.5 -3.5)
       (stroke (width 0.1) (type solid)) (layer "B.Fab"))
-    (pad "" smd roundrect (at -1.95 -1.95 270) (size 1.05 1.05) (layers "B.Paste") (roundrect_rratio 0.238095))
-    (pad "" smd roundrect (at -1.95 -0.65 270) (size 1.05 1.05) (layers "B.Paste") (roundrect_rratio 0.238095))
-    (pad "" smd roundrect (at -1.95 0.65 270) (size 1.05 1.05) (layers "B.Paste") (roundrect_rratio 0.238095))
-    (pad "" smd roundrect (at -1.95 1.95 270) (size 1.05 1.05) (layers "B.Paste") (roundrect_rratio 0.238095))
-    (pad "" smd roundrect (at -0.65 -1.95 270) (size 1.05 1.05) (layers "B.Paste") (roundrect_rratio 0.238095))
-    (pad "" smd roundrect (at -0.65 -0.65 270) (size 1.05 1.05) (layers "B.Paste") (roundrect_rratio 0.238095))
-    (pad "" smd roundrect (at -0.65 0.65 270) (size 1.05 1.05) (layers "B.Paste") (roundrect_rratio 0.238095))
-    (pad "" smd roundrect (at -0.65 1.95 270) (size 1.05 1.05) (layers "B.Paste") (roundrect_rratio 0.238095))
-    (pad "" smd roundrect (at 0.65 -1.95 270) (size 1.05 1.05) (layers "B.Paste") (roundrect_rratio 0.238095))
-    (pad "" smd roundrect (at 0.65 -0.65 270) (size 1.05 1.05) (layers "B.Paste") (roundrect_rratio 0.238095))
-    (pad "" smd roundrect (at 0.65 0.65 270) (size 1.05 1.05) (layers "B.Paste") (roundrect_rratio 0.238095))
-    (pad "" smd roundrect (at 0.65 1.95 270) (size 1.05 1.05) (layers "B.Paste") (roundrect_rratio 0.238095))
-    (pad "" smd roundrect (at 1.95 -1.95 270) (size 1.05 1.05) (layers "B.Paste") (roundrect_rratio 0.238095))
-    (pad "" smd roundrect (at 1.95 -0.65 270) (size 1.05 1.05) (layers "B.Paste") (roundrect_rratio 0.238095))
-    (pad "" smd roundrect (at 1.95 0.65 270) (size 1.05 1.05) (layers "B.Paste") (roundrect_rratio 0.238095))
-    (pad "" smd roundrect (at 1.95 1.95 270) (size 1.05 1.05) (layers "B.Paste") (roundrect_rratio 0.238095))
+    (pad "" smd roundrect (at -1.95 -1.95 270) (size 1.05 1.05) (layers "B.Paste") (roundrect_rratio 0.2380952381))
+    (pad "" smd roundrect (at -1.95 -0.65 270) (size 1.05 1.05) (layers "B.Paste") (roundrect_rratio 0.2380952381))
+    (pad "" smd roundrect (at -1.95 0.65 270) (size 1.05 1.05) (layers "B.Paste") (roundrect_rratio 0.2380952381))
+    (pad "" smd roundrect (at -1.95 1.95 270) (size 1.05 1.05) (layers "B.Paste") (roundrect_rratio 0.2380952381))
+    (pad "" smd roundrect (at -0.65 -1.95 270) (size 1.05 1.05) (layers "B.Paste") (roundrect_rratio 0.2380952381))
+    (pad "" smd roundrect (at -0.65 -0.65 270) (size 1.05 1.05) (layers "B.Paste") (roundrect_rratio 0.2380952381))
+    (pad "" smd roundrect (at -0.65 0.65 270) (size 1.05 1.05) (layers "B.Paste") (roundrect_rratio 0.2380952381))
+    (pad "" smd roundrect (at -0.65 1.95 270) (size 1.05 1.05) (layers "B.Paste") (roundrect_rratio 0.2380952381))
+    (pad "" smd roundrect (at 0.65 -1.95 270) (size 1.05 1.05) (layers "B.Paste") (roundrect_rratio 0.2380952381))
+    (pad "" smd roundrect (at 0.65 -0.65 270) (size 1.05 1.05) (layers "B.Paste") (roundrect_rratio 0.2380952381))
+    (pad "" smd roundrect (at 0.65 0.65 270) (size 1.05 1.05) (layers "B.Paste") (roundrect_rratio 0.2380952381))
+    (pad "" smd roundrect (at 0.65 1.95 270) (size 1.05 1.05) (layers "B.Paste") (roundrect_rratio 0.2380952381))
+    (pad "" smd roundrect (at 1.95 -1.95 270) (size 1.05 1.05) (layers "B.Paste") (roundrect_rratio 0.2380952381))
+    (pad "" smd roundrect (at 1.95 -0.65 270) (size 1.05 1.05) (layers "B.Paste") (roundrect_rratio 0.2380952381))
+    (pad "" smd roundrect (at 1.95 0.65 270) (size 1.05 1.05) (layers "B.Paste") (roundrect_rratio 0.2380952381))
+    (pad "" smd roundrect (at 1.95 1.95 270) (size 1.05 1.05) (layers "B.Paste") (roundrect_rratio 0.2380952381))
     (pad "1" smd roundrect (at -3.3375 2.5 270) (size 1.075 0.25) (layers "B.Cu" "B.Paste" "B.Mask") (roundrect_rratio 0.25)
       (net 81 "row1") (pinfunction "PE6") (pintype "bidirectional"))
@@
     (pad "4" smd roundrect (at 1.5 2 90) (size 0.6 1.55) (layers "B.Cu" "B.Paste" "B.Mask") (roundrect_rratio 0.25)
       (net 2 "GND") (pinfunction "4") (pintype "power_in"))
-    (pad "MP" smd roundrect (at -2.8 -1.875 90) (size 1.2 1.8) (layers "B.Cu" "B.Paste" "B.Mask") (roundrect_rratio 0.208333))
-    (pad "MP" smd roundrect (at 2.8 -1.875 90) (size 1.2 1.8) (layers "B.Cu" "B.Paste" "B.Mask") (roundrect_rratio 0.208333))
+    (pad "MP" smd roundrect (at -2.8 -1.875 90) (size 1.2 1.8) (layers "B.Cu" "B.Paste" "B.Mask") (roundrect_rratio 0.2083333333))
+    (pad "MP" smd roundrect (at 2.8 -1.875 90) (size 1.2 1.8) (layers "B.Cu" "B.Paste" "B.Mask") (roundrect_rratio 0.2083333333))
     (model "${KICAD6_3DMODEL_DIR}/Connector_JST.3dshapes/JST_SH_SM04B-SRSS-TB_1x04-1MP_P1.00mm_Horizontal.wrl"
       (offset (xyz 0 0 0))
@@
   (gr_arc (start 27.979711 95.845393) (mid 26.295912 95.14794) (end 25.598459 93.464141)
     (stroke (width 0.1) (type default)) (layer "Edge.Cuts"))
+  (gr_text "anything is possible with a dremel and a little courage" (at 228.7 94.15) (layer "B.SilkS")
+    (effects (font (size 1 1) (thickness 0.15)) (justify mirror))
+  )
+  (gr_text "lucy v3-QFN 2023.04.12" (at 233.75 94.2) (layer "F.SilkS")
+    (effects (font (size 1 1) (thickness 0.15)))
+  )
+  (gr_text "lucy rev 3.0" (at 58.3 94.15) (layer "B.Mask")
+    (effects (font (size 1.5 1.5) (thickness 0.3) bold) (justify left bottom mirror))
+  )
   (segment (start 261.025 49.575) (end 261.025 48.975) (width 0.254) (layer "B.Cu") (net 1))
   (segment (start 259.25 53.2875) (end 259.25 51.35) (width 0.254) (layer "B.Cu") (net 1))
@@
   (via (at 81.25 55.625) (size 0.8128) (drill 0.4064) (layers "F.Cu" "B.Cu") (net 2))
   (via (at 164.85 40.475) (size 0.8128) (drill 0.4064) (layers "F.Cu" "B.Cu") (free) (net 2))
-  (via (at 234.525 93.9) (size 0.8128) (drill 0.4064) (layers "F.Cu" "B.Cu") (free) (net 2))
+  (via (at 234.55 92.55) (size 0.8128) (drill 0.4064) (layers "F.Cu" "B.Cu") (free) (net 2))
   (via (at 242.95 40.475) (size 0.8128) (drill 0.4064) (layers "F.Cu" "B.Cu") (free) (net 2))
   (via (at 152.6 70.925) (size 0.8128) (drill 0.4064) (layers "F.Cu" "B.Cu") (free) (net 2))
