File: 01_pcb/3.0_hotswap-QFP-0805/pcb/pcb.kicad_pcb (KiCad board)
At the start: 2 copper layers, 256 x 75 mm, 126 parts, among them J1 TYPE-C-31-M12_13, J2 AVR-ISP-6_mod, J3 4PIN, J5 Conn_01x08, SW1 SW_PUSH, U1 ATmega32U4-A, U4 USBLC6-2SC6, Y1 16MHz

Commit message: rename folders
Parts:
- moved R3 0.29 mm to (258.0, 44.6)
- moved R2 0.25 mm to (255.6, 44.6)
Routing:
- net D+: track 4.97 -> 5.50 mm
- net D-: track 4.98 -> 5.49 mm
Changed lines of the file:
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@@
   )
   (footprint "Resistor_SMD:R_0805_2012Metric" (layer "B.Cu")
-    (at 257.7 44.55 -90)
+    (at 257.975 44.65 -90)
     (descr "Resistor SMD 0805 (2012 Metric), square (rectangular) end terminal, IPC_7351 nominal, (Body size source: IPC-SM-782 page 72, https://www.pcb-3d.com/wordpress/wp-content/uploads/ipc-sm-782a_amendment_1_and_2.pdf), generated with kicad-footprint-generator")
     (tags "resistor")
@@
   )
   (footprint "Resistor_SMD:R_0805_2012Metric" (layer "B.Cu")
-    (at 255.775 44.55 90)
+    (at 255.55 44.65 90)
     (descr "Resistor SMD 0805 (2012 Metric), square (rectangular) end terminal, IPC_7351 nominal, (Body size source: IPC-SM-782 page 72, https://www.pcb-3d.com/wordpress/wp-content/uploads/ipc-sm-782a_amendment_1_and_2.pdf), generated with kicad-footprint-generator")
     (tags "resistor")
@@
   (segment (start 44.694788 40.404) (end 43.920999 39.630211) (width 0.254) (layer "B.Cu") (net 60))
   (segment (start 42.707849 28.487981) (end 42.707849 26.789085) (width 0.254) (layer "B.Cu") (net 60))
-  (segment (start 256.483499 39.542711) (end 256.483499 42.929001) (width 0.254) (layer "B.Cu") (net 60))
+  (segment (start 256.483499 39.542711) (end 256.483499 42.05) (width 0.254) (layer "B.Cu") (net 60))
   (segment (start 241.175 37.804001) (end 254.744789 37.804001) (width 0.254) (layer "B.Cu") (net 60))
   (segment (start 43.282263 37.65) (end 43.920999 37.011264) (width 0.254) (layer "B.Cu") (net 60))
@@
   (segment (start 43.920999 38.570999) (end 43 37.65) (width 0.254) (layer "B.Cu") (net 60))
   (segment (start 54.030211 37.804001) (end 51.430212 40.404) (width 0.254) (layer "B.Cu") (net 60))
-  (segment (start 256.483499 42.929001) (end 255.775 43.6375) (width 0.254) (layer "B.Cu") (net 60))
   (segment (start 42.707849 26.789085) (end 42.707849 26.577636) (width 0.2032) (layer "B.Cu") (net 60))
   (segment (start 238.475 37.804001) (end 54.030211 37.804001) (width 0.254) (layer "B.Cu") (net 60))
@@
   (segment (start 254.744789 37.804001) (end 255.420394 38.479606) (width 0.254) (layer "B.Cu") (net 60))
   (segment (start 255.789218 39.383573) (end 255.789217 39.383574) (width 0.254) (layer "B.Cu") (net 60))
+  (segment (start 256.483499 42.804001) (end 255.55 43.7375) (width 0.254) (layer "B.Cu") (net 60))
+  (segment (start 256.483499 42.05) (end 256.483499 42.804001) (width 0.254) (layer "B.Cu") (net 60))
   (segment (start 238.720999 38.05) (end 238.475 37.804001) (width 0.254) (layer "B.Cu") (net 60))
   (segment (start 239.9 38.05) (end 238.720999 38.05) (width 0.254) (layer "B.Cu") (net 60))
@@
   (arc (start 255.420394 38.479606) (mid 255.508262 38.691739) (end 255.420393 38.903871) (width 0.254) (layer "B.Cu") (net 60))
   (segment (start 44.905212 39.896) (end 51.219788 39.896) (width 0.254) (layer "B.Cu") (net 61))
-  (segment (start 256.991501 42.929001) (end 256.991501 39.332289) (width 0.254) (layer "B.Cu") (net 61))
+  (segment (start 256.991501 42.025) (end 256.991501 39.332289) (width 0.254) (layer "B.Cu") (net 61))
   (segment (start 45.067737 37.65) (end 44.429001 37.011264) (width 0.254) (layer "B.Cu") (net 61))
   (segment (start 239.9 37.05) (end 240.929001 37.05) (width 0.254) (layer "B.Cu") (net 61))
@@
   (segment (start 44.729001 30.975) (end 44.948693 30.975) (width 0.254) (layer "B.Cu") (net 61))
   (segment (start 44.948693 30.375) (end 44.729001 30.375) (width 0.254) (layer "B.Cu") (net 61))
+  (segment (start 256.991501 42.025) (end 256.991501 42.754001) (width 0.254) (layer "B.Cu") (net 61))
   (segment (start 44.429001 38.570999) (end 44.429001 39.419789) (width 0.254) (layer "B.Cu") (net 61))
   (segment (start 44.429001 30.009215) (end 44.429001 29.475) (width 0.254) (layer "B.Cu") (net 61))
@@
   (segment (start 51.219788 39.896) (end 53.819789 37.295999) (width 0.254) (layer "B.Cu") (net 61))
   (segment (start 44.729001 32.175) (end 44.948693 32.175) (width 0.254) (layer "B.Cu") (net 61))
-  (segment (start 257.7 43.6375) (end 256.991501 42.929001) (width 0.254) (layer "B.Cu") (net 61))
   (segment (start 70.05 37.295999) (end 238.525 37.295999) (width 0.254) (layer "B.Cu") (net 61))
   (segment (start 44.429001 39.419789) (end 44.905212 39.896) (width 0.254) (layer "B.Cu") (net 61))
   (segment (start 43.203849 28.249848) (end 43.7645 28.8105) (width 0.254) (layer "B.Cu") (net 61))
   (segment (start 44.429001 29.475) (end 43.7645 28.8105) (width 0.254) (layer "B.Cu") (net 61))
+  (segment (start 256.991501 42.754001) (end 257.975 43.7375) (width 0.254) (layer "B.Cu") (net 61))
   (arc (start 69.15 36.917639) (mid 69.237868 36.705507) (end 69.45 36.617639) (width 0.254) (layer "B.Cu") (net 61))
   (arc (start 69.75 36.995999) (mid 69.837868 37.208131) (end 70.05 37.295999) (width 0.254) (layer "B.Cu") (net 61))
@@
   (segment (start 254.125 64.25) (end 254.75 63.625) (width 0.254) (layer "B.Cu") (net 70))
   (segment (start 254.125 64.95) (end 254.125 64.25) (width 0.254) (layer "B.Cu") (net 70))
-  (segment (start 257.15 50.2) (end 257.15 46.0125) (width 0.254) (layer "B.Cu") (net 71))
-  (segment (start 257.15 46.0125) (end 257.7 45.4625) (width 0.254) (layer "B.Cu") (net 71))
-  (segment (start 256.35 46.0375) (end 255.775 45.4625) (width 0.254) (layer "B.Cu") (net 72))
-  (segment (start 256.35 50.2) (end 256.35 46.0375) (width 0.254) (layer "B.Cu") (net 72))
+  (segment (start 257.15 50.725) (end 257.15 46.3875) (width 0.254) (layer "B.Cu") (net 71))
+  (segment (start 257.15 46.3875) (end 257.975 45.5625) (width 0.254) (layer "B.Cu") (net 71))
+  (segment (start 256.35 46.3625) (end 255.55 45.5625) (width 0.254) (layer "B.Cu") (net 72))
+  (segment (start 256.35 50.725) (end 256.35 46.3625) (width 0.254) (layer "B.Cu") (net 72))
   (segment (start 42.225 28.975) (end 41.5 28.25) (width 0.254) (layer "F.Cu") (net 73))
   (segment (start 37.5 28.25) (end 41.5 28.25) (width 0.254) (layer "F.Cu") (net 73))

Commit message: added text
Parts:
- removed U4: USBLC6-2SC6, marbastlib-various:SOT-23-6-routable
- added U2: PRTR5V0U2X, Package_TO_SOT_SMD:SOT-143, B.Cu at (44.1, 36.8)
- renumbered J1 to USB1
Routing:
- net VBUS: track 22.0 -> 21.1 mm
- net GND: track 463.6 -> 464.0 mm, vias 345 -> 344
Other:
- board text added: "anything is possible with a dremel and a little courage"
- board text added: "lucy rev 3.0"
- board text added: "lucy v3-QFP 2023.04.12"

Commit message: replace mx footprint with marbast footprints
Parts:
- MX1, MX10, MX11, MX12, MX13, MX14, MX15, MX16, MX17, MX18, MX19, MX2, MX20, MX21, MX22, MX23, MX24, MX25, MX26, MX27, MX28, MX29, MX3, MX30, MX31, MX32, MX33, MX34, MX35, MX36, MX37, MX38, MX39, MX4, MX40, MX41, MX42, MX43, MX44, MX45, MX46, MX47, MX48, MX49, MX5, MX50, MX51, MX52, MX6, MX7, MX8, MX9: footprint MX_Only:MXOnly-1U-Hotswap -> marbastlib-mx:SW_MX_HS_S_1u; moved to B.Cu
- moved J3 16.9 mm to (221.0, 37.5)
- moved U2 1.49 mm to (44.9, 38.1)
- turned MX1 to 0 degrees
- turned MX10 to 180 degrees
- turned MX11 to 180 degrees
- turned MX12 to 180 degrees
- turned MX13 to 180 degrees
- turned MX14 to 180 degrees
- turned MX15 to 180 degrees
- turned MX16 to 180 degrees
- turned MX17 to 180 degrees
- turned MX18 to 180 degrees
- turned MX19 to 180 degrees
- turned MX2 to 0 degrees
- turned MX20 to 180 degrees
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Routing:
- net col1: track 298.7 -> 273.9 mm, vias 5 -> 1
- net col10/mosi: track 135.8 -> 118.7 mm, vias 5 -> 2
- net col2: track 271.3 -> 255.7 mm, vias 5 -> 1
- net col4: track 219.6 -> 204.0 mm, vias 5 -> 1
- net col3: track 251.6 -> 236.0 mm, vias 5 -> 1
- net col8: track 142.9 -> 127.4 mm, vias 5 -> 1
- net col7: track 161.8 -> 146.3 mm, vias 5 -> 1
- net col9: track 124.0 -> 108.4 mm, vias 5 -> 1
- net col6: track 181.0 -> 165.5 mm, vias 5 -> 1
- net col5: track 200.3 -> 184.8 mm, vias 5 -> 1
- net col11/miso: track 117.3 -> 105.0 mm, vias 4 -> 0
- net col0: track 304.4 -> 293.3 mm, vias 0 -> 1
- net DBUS+: track 238.9 -> 236.4 mm
- net GND: track 464.0 -> 461.9 mm
- net VBUS: track 21.1 -> 22.1 mm
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