File: 01_pcb/3.0_hotswap-QFP-0805/pcb/pcb.kicad_sch (KiCad schematic)
At the start: 126 parts, among them J1 TYPE-C-31-M12_13, J2 AVR-ISP-6_mod, J3 4PIN, J5 Conn_01x08, SW1 SW_PUSH, U1 ATmega32U4-A, U4 USBLC6-2SC6, Y1 16MHz

Commit message: added text
Parts:
- removed U4: USBLC6-2SC6, marbastlib-various:SOT-23-6-routable, symbol Power_Protection:USBLC6-2SC6
- added U2: PRTR5V0U2X, Package_TO_SOT_SMD:SOT-143, symbol Power_Protection:PRTR5V0U2X
- renumbered J1 to USB1
Connections:
- net DBUS+: now also U2.2 (I/O1)
- net DBUS-: now also U2.3 (I/O2)
- net GND: now also U2.1 (GND)
- net VBUS: now also U2.4 (VCC)
- no-connect marks 5 -> 3
Other:
- moved on the sheet: R2, R3

Commit message: replace mx footprint with marbast footprints
Parts:
- MX1, MX10, MX11, MX12, MX13, MX14, MX15, MX16, MX17, MX18, MX19, MX2, MX20, MX21, MX22, MX23, MX24, MX25, MX26, MX27, MX28, MX29, MX3, MX30, MX31, MX32, MX33, MX34, MX35, MX36, MX37, MX38, MX39, MX4, MX40, MX41, MX42, MX43, MX44, MX45, MX46, MX47, MX48, MX49, MX5, MX50, MX51, MX52, MX6, MX7, MX8, MX9: footprint MX_Only:MXOnly-1U-Hotswap -> marbastlib-mx:SW_MX_HS_S_1u
