File: 01_pcb/3.0_hotswap-QFN-0603/pcb.kicad_pcb (KiCad board)
At the start: 2 copper layers, 256 x 75 mm, 126 parts, among them J1 TYPE-C-31-M12_13, J2 AVR-ISP-6_mod, J3 4PIN, J5 Conn_01x08, SW1 SW_PUSH, U1 ATmega32U4-M, U4 USBLC6-2SC6, Y1 16MHz

Commit message: updated QFN, removed some vias
Parts:
- removed F1: .5A, Fuse:Fuse_0805_2012Metric_Pad1.15x1.40mm_HandSolder
- removed J1: TYPE-C-31-M12_13, acheron_Connectors:TYPE-C-31-M-12
- removed RCC1, RCC2: 5.1k, Resistor_SMD:R_0603_1608Metric
- removed U4: USBLC6-2SC6, marbastlib-various:SOT-23-6-routable
- MX1, MX10, MX11, MX12, MX13, MX14, MX15, MX16, MX17, MX18, MX19, MX2, MX20, MX21, MX22, MX23, MX24, MX25, MX26, MX27, MX28, MX29, MX3, MX30, MX31, MX32, MX33, MX34, MX35, MX36, MX37, MX38, MX39, MX4, MX40, MX41, MX42, MX43, MX44, MX45, MX46, MX47, MX48, MX49, MX5, MX50, MX51, MX52, MX6, MX7, MX8, MX9: footprint MX_Only:MXOnly-1U-Hotswap -> marbastlib-mx:SW_MX_HS_S_1u; moved to B.Cu
- U1: value ATmega32U4-M -> ATmega32U4-A
- moved J3 14.5 mm to (223.4, 37.5)
- moved D1 14.0 mm to (44.3, 31.4)
- moved D12 12.4 mm to (239.1, 31.4)
- moved D2 8.63 mm to (63.4, 31.4)
- moved C2 2.86 mm to (250.3, 57.9)
- moved D26 2.81 mm to (277.7, 49.0)
- moved C3 2.65 mm to (261.2, 61.7)
- moved R2 2.45 mm to (254.6, 47.7)
- moved D13 2.38 mm to (277.7, 31.4)
- moved D20 2.38 mm to (158.6, 50.5)
- moved D22 2.38 mm to (196.7, 50.5)
- moved D33 2.38 mm to (158.6, 69.5)
- moved D35 2.38 mm to (196.7, 69.5)
- moved D38 2.38 mm to (253.9, 69.5)
- moved D39 2.38 mm to (277.7, 69.5)
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Connections:
- J3 pad 2: DBUS- -> D-
- J3 pad 3: DBUS+ -> D+
- R2 pad 1: D- -> Net-(U1-D-)
- R2 pad 2: DBUS- -> D-
- R3 pad 1: DBUS+ -> D+
- R3 pad 2: D+ -> Net-(U1-D+)
- U1 pad 3: D- -> Net-(U1-D-)
- U1 pad 4: D+ -> Net-(U1-D+)
Routing:
- net DBUS+: track 242.9 -> 0.00 mm
- net DBUS-: track 240.2 -> 0.00 mm
- net GND: track 484.3 -> 273.8 mm, vias 337 -> 171
- net VCC: track 314.0 -> 127.7 mm, vias 10 -> 7
- net D+: track 4.59 -> 39.6 mm
- net D-: track 4.62 -> 39.6 mm
- net extra8: track 52.6 -> 81.2 mm
- net col1: track 301.3 -> 275.8 mm, vias 5 -> 1
- net VBUS: track 22.0 -> 0.00 mm
- net col10/mosi: track 138.9 -> 118.1 mm, vias 5 -> 2
- net col9: track 126.6 -> 107.7 mm, vias 5 -> 1
- net col8: track 145.7 -> 126.8 mm, vias 5 -> 1
- net col7: track 164.7 -> 145.9 mm, vias 5 -> 1
- net col4: track 221.9 -> 203.2 mm, vias 5 -> 1
- net col6: track 183.7 -> 165.0 mm, vias 5 -> 1
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Other:
- board size 256 x 75 mm -> 251.2 x 75 mm
- board text added: "lucy rev 3.1"
- board text added: "lucy v3.1-QFN 2023.05.18"
- board text removed: "lucy rev 3.0"
- board text removed: "lucy v3-QFN 2023.04.12"
