File: 01_pcb/3.0_hotswap-QFP-0805/pcb.kicad_pcb (KiCad board)
At the start: 2 copper layers, 251.2 x 75 mm, 121 parts, among them J2 AVR-ISP-6_mod, J3 4PIN, J5 Conn_01x08, SW1 SW_PUSH, U1 ATmega32U4-A, Y1 16MHz

Commit message: moved JST connector 20mm
Parts:
- moved J3 20.3 mm to (243.7, 37.5)
Routing:
- net D-: track 32.9 -> 12.7 mm
- net D+: track 33.0 -> 12.7 mm
- net VCC: track 135.5 -> 115.3 mm
- net GND: track 219.0 -> 208.6 mm, vias 151 -> 141
Other:
- board text added: "lucy v3.1-QFP 2023.07.08"
- board text removed: "lucy v3.1-QFP 2023.05.18"
